Commit message: Checkpoint motion diagnostics and sim physics tuning

File: ros2_ws/src/tennis_robot/urdf/components/drivetrain.urdf.xacro (robot description, xacro)
@@ -22,7 +22,13 @@
     </joint>
     <gazebo reference="${side}_wheel_link">
-      <mu1>1.0</mu1>
-      <mu2>0.5</mu2>
-      <fdir1>1 0 0</fdir1>
+      <!-- VER=21: brute-force friction test — mu=5.0 isotropic, no fdir1.
+           VER=20 (mu=1.5) improved rotation from 48° to 73° out of 275° (~73% slip).
+           If mu=5.0 with court mu=2.0 still gives ~73% slip, the URDF <gazebo>
+           friction tags are NOT reaching the physics engine (DART ignoring them)
+           and we need the bullet-featherstone engine or direct SDF injection. -->
+      <mu1>5.0</mu1>
+      <mu2>5.0</mu2>
+      <slip1>0.0</slip1>
+      <slip2>0.0</slip2>
     </gazebo>
   </xacro:macro>
@@ -74,6 +80,5 @@
     <gazebo reference="${name}_caster_wheel_link">
       <mu1>0.8</mu1>
-      <mu2>0.05</mu2>
-      <fdir1>1 0 0</fdir1>
+      <mu2>1.5</mu2>
     </gazebo>
   </xacro:macro>

File: ros2_ws/src/tennis_robot/urdf/components/lidar.urdf.xacro (robot description, xacro)
@@ -24,5 +24,8 @@
     <gazebo reference="${link_name}">
       <sensor name="front_lidar" type="gpu_lidar">
-        <pose>0 0 0 0 0 0</pose>
+        <!-- Raised above head_vis (cylinder r=0.047, z=±0.0225): gpu_lidar
+             renders VISUALS, and a sensor origin inside its own housing makes
+             every ray hit the cylinder interior at ~5 cm (lidar goes blind). -->
+        <pose>0 0 0.035 0 0 0</pose>
         <update_rate>${update_rate}</update_rate>
         <always_on>true</always_on>
@@ -40,5 +43,7 @@
           </scan>
           <range>
-            <min>0.05</min>
+            <!-- RPLIDAR C1 spec min is 0.1 m; 0.15 also rejects any residual
+                 self-hits from the robot's own body. -->
+            <min>0.15</min>
             <max>12.0</max>
             <resolution>0.01</resolution>

File: ros2_ws/src/tennis_robot/urdf/components/oak_d.urdf.xacro (robot description, xacro)
@@ -37,5 +37,5 @@
         <camera>
           <horizontal_fov>1.204</horizontal_fov>
-          <image><width>1920</width><height>1080</height><format>R8G8B8</format></image>
+          <image><width>640</width><height>480</height><format>R8G8B8</format></image>
           <clip><near>0.08</near><far>18</far></clip>
           <noise><type>gaussian</type><mean>0</mean><stddev>0.007</stddev></noise>

File: ros2_ws/src/tennis_robot/urdf/components/ros2_control.urdf.xacro (robot description, xacro)
@@ -57,4 +57,16 @@
         <state_interface name="velocity"/>
       </joint>
+      <!-- ── Passive caster joints: NOT in ros2_control ──────────────────────
+           Previously listed here as state-only so joint_state_broadcaster could
+           publish their positions for RViz TF. However, gz_ros2_control owns any
+           joint it has an interface for, and may zero out state-only joints during
+           initialization or write cycles. Locked caster swivel/wheel joints create
+           ~12 N·m of scrub resistance (mu1=0.8 × caster weight × moment arm) that
+           exceeds the ~7.7 N·m drive torque → 82% rotation slip observed.
+           Fix: remove casters from ros2_control entirely; gz-physics handles them
+           freely via URDF <dynamics damping="0.02" friction="0.001"/> on the swivel.
+           Cost: /joint_states won't include casters → RViz "No transform from
+           front_*_caster_*". Navigation is unaffected (caster TF not used by
+           slam_toolbox or nav2). -->
     </ros2_control>
     <!-- ── gz_ros2_control system plugin (sim only) ─────────────────────────

File: ros2_ws/src/tennis_robot/urdf/tennis_robot.urdf.xacro (robot description, xacro)
@@ -36,5 +36,5 @@
   <xacro:property name="caster_width" value="0.035"/>
   <xacro:property name="caster_trail" value="0.025"/>     <!-- self-aligning offset -->
-  <xacro:property name="caster_z" value="-0.0825"/>       <!-- contact = -0.145 m (coplanar) -->
+  <xacro:property name="caster_z" value="-0.1175"/>       <!-- contact = -0.180 m -->
   <xacro:property name="intake_x" value="0.62"/>
   <xacro:property name="intake_z" value="0.095"/>
@@ -42,5 +42,5 @@
   <xacro:property name="intake_width" value="0.24"/>
   <xacro:property name="lidar_xyz" value="-0.08 0 0.713"/>
-  <xacro:property name="lidar_rpy" value="0 0 0"/>
+  <xacro:property name="lidar_rpy" value="0 -0.053 0"/>  <!-- counter the 3deg chassis pitch so the 360 scan plane stays horizontal -->
   <xacro:property name="camera_xyz" value="0.535 0 0.443"/>
   <xacro:property name="camera_rpy" value="0 0.22 0"/>

Commit message: Add sim-time motion diagnostic and tune casters

File: ros2_ws/src/tennis_robot/urdf/components/drivetrain.urdf.xacro (robot description, xacro)
@@ -80,5 +80,5 @@
     <gazebo reference="${name}_caster_wheel_link">
       <mu1>0.8</mu1>
-      <mu2>1.5</mu2>
+      <mu2>0.05</mu2>
     </gazebo>
   </xacro:macro>

File: ros2_ws/src/tennis_robot/urdf/tennis_robot.urdf.xacro (robot description, xacro)
@@ -36,5 +36,5 @@
   <xacro:property name="caster_width" value="0.035"/>
   <xacro:property name="caster_trail" value="0.025"/>     <!-- self-aligning offset -->
-  <xacro:property name="caster_z" value="-0.1175"/>       <!-- contact = -0.180 m -->
+  <xacro:property name="caster_z" value="-0.0825"/>       <!-- contact = -0.145 m (coplanar with drive wheels under 3deg pitch) -->
   <xacro:property name="intake_x" value="0.62"/>
   <xacro:property name="intake_z" value="0.095"/>
