Commit message: Fix intake capture physics: paddle roller, synced channel geometry, sim instrumentation
Instrumented rosbag testing (8 collect_one runs) traced the capture failure
through four root causes, all fixed:

- Channel/scoop geometry was desynced from the roller tuning offsets
  (hardcoded 0.615/0.112): both generate_curved_scoop_mesh.py and the SDF
  collision patch now follow INTAKE_ROLLER_*_OFFSET_M.
- A rigid fixed-axis cylinder cannot friction-capture a rigid ball
  (interference jams, clearance never grips), and a 1-DOF vertical spring
  carriage only yields vertically while the ball's orbit needs radial
  compliance (every run stalled at fwd=-75mm). Replaced with the original
  paddle-wheel design: hub + 8 sprung paddles (SDF-patched joint springs),
  one contact sensor per paddle on the existing roller_contact_0..7 bridges.
- The near-vertical rear wall left an unpowered 58mm gap above the roller's
  reach: replaced with a concentric guide that keeps the ball driven
  tangentially to the z=155 release edge.
- Contact sensors now bind dynamically to the real (lumped) collision names,
  failing loudly instead of going silently dead.

Test result: ball is now gripped and carried the full arc (z 43->171mm).
Remaining known issue (intake-debug-log #14): basket handoff — the ball
juggles on top of the wheel; deflector/basket-floor geometry needs matching
to the paddle transport.

Also:
- Sim-only intake debug camera + depth (side vantage, point light) with
  bridges and RViz Image display.
- gazebo_extras robot pose from /odom (pose_info child_frame_id is empty in
  this bridge version; ball/contact markers silently never published).
- scripts/sim_debug/: instrumented collect_one orchestrator, gz ground-truth
  pose logger, frame dumper, bag analyzer, live physics probe.
- docs/intake-debug-log-el.md: full change/outcome log of the debugging arc.

Co-Authored-By: Claude Fable 5 <noreply@anthropic.com>

File: ros2_ws/src/tennis_robot/urdf/components/drivetrain.urdf.xacro (robot description, xacro)
@@ -55,44 +55,63 @@
        the drive_wheel macro above). The old swivel-caster macro and its scrub
        resistance are gone. -->
-  <!-- One paddle belonging to the single intake-roller link. `angle` is in the
-       link's x-z plane; rotating the link rotates core and all paddles together. -->
-  <xacro:macro name="intake_flap" params="name angle radius width">
-    <collision name="${name}_col">
-      <origin
-          xyz="${radius * 0.72 * cos(angle)} 0 ${radius * 0.72 * sin(angle)}"
-          rpy="0 ${-angle} 0"/>
-      <geometry><box size="${radius * 0.56} ${width} 0.004"/></geometry>
-    </collision>
-    <visual name="${name}_vis">
-      <origin
-          xyz="${radius * 0.72 * cos(angle)} 0 ${radius * 0.72 * sin(angle)}"
-          rpy="0 ${-angle} 0"/>
-      <geometry><box size="${radius * 0.56} ${width} 0.004"/></geometry>
-      <material name="rubber_black"/>
-    </visual>
+  <!-- One rubber intake paddle: a thin box on its own sprung revolute joint
+       so it bends RADIALLY when squeezing the ball. Spring params are
+       injected into the generated SDF by generate_robot_urdf.py (URDF cannot
+       express joint springs). One contact sensor per paddle, matching the
+       pre-existing /gz/roller_contact_0..7 bridges. -->
+  <xacro:macro name="intake_paddle" params="index angle hub_r paddle_len width thickness">
+    <link name="paddle_${index}_link">
+      <xacro:box_inertial mass="0.012" x="${paddle_len}" y="${width}" z="${thickness}"/>
+      <collision name="paddle_${index}_col">
+        <origin xyz="${paddle_len / 2} 0 0" rpy="0 0 0"/>
+        <geometry><box size="${paddle_len} ${width} ${thickness}"/></geometry>
+      </collision>
+      <visual name="paddle_${index}_vis">
+        <origin xyz="${paddle_len / 2} 0 0" rpy="0 0 0"/>
+        <geometry><box size="${paddle_len} ${width} ${thickness}"/></geometry>
+        <material name="intake_orange"/>
+      </visual>
+    </link>
+    <joint name="paddle_${index}_joint" type="revolute">
+      <parent link="lift_wheel_link"/>
+      <child link="paddle_${index}_link"/>
+      <!-- Root on the hub surface, +x pointing radially outward. -->
+      <origin xyz="${hub_r * cos(angle)} 0 ${hub_r * sin(angle)}" rpy="0 ${-angle} 0"/>
+      <axis xyz="0 1 0"/>
+      <limit lower="-1.2" upper="1.2" effort="10" velocity="60"/>
+      <dynamics damping="0.02"/>
+    </joint>
+    <gazebo reference="paddle_${index}_link">
+      <sensor name="roller_contact_${index}" type="contact">
+        <always_on>true</always_on><update_rate>100</update_rate>
+        <topic>/gz/roller_contact_${index}</topic>
+        <contact><collision>paddle_${index}_col</collision></contact>
+      </sensor>
+    </gazebo>
   </xacro:macro>
   <xacro:macro name="intake_roller" params="x z radius width mass">
+    <!-- Paddle roller: hub + 8 sprung rubber paddles. A rigid fixed-axis
+         cylinder cannot friction-capture a rigid ball, and a 1-DOF sprung
+         carriage only yields VERTICALLY while the ball's orbit around the
+         roller needs ~2 mm of RADIAL compliance at every angle (the vertical
+         travel required blows up to 21+ mm behind the axis — every capture
+         stalled at exactly fwd=-75 mm; intake-debug-log #13). Per-paddle
+         springs give true radial compliance like the real foam surface:
+         paddle tips sweep radius+5 mm and bend back locally around the ball.
+         This restores the project's ORIGINAL paddle-wheel design — the
+         roller_contact_0..7 bridges are its infrastructure. -->
+    <xacro:property name="hub_radius" value="0.025"/>
+    <xacro:property name="paddle_length" value="${radius + 0.005 - hub_radius}"/>
     <link name="lift_wheel_link">
-      <xacro:cylinder_inertial mass="${mass}" radius="${radius}" length="${width}" axis="y"/>
-      <!-- Small rigid hub; the paddles sweep the full `radius` envelope
-           (Ø90 mm with the current intake_radius=0.045). Roller-first design:
-           this envelope is the first hard contact with the ball. -->
-      <collision name="core_col">
+      <xacro:cylinder_inertial mass="${mass}" radius="${hub_radius}" length="${width}" axis="y"/>
+      <collision name="roller_col">
         <origin xyz="0 0 0" rpy="1.5708 0 0"/>
-        <geometry><cylinder radius="${radius * 0.44}" length="${width}"/></geometry>
+        <geometry><cylinder radius="${hub_radius}" length="${width}"/></geometry>
       </collision>
-      <visual name="core_vis">
+      <visual name="roller_vis">
         <origin xyz="0 0 0" rpy="1.5708 0 0"/>
-        <geometry><cylinder radius="${radius * 0.44}" length="${width}"/></geometry>
+        <geometry><cylinder radius="${hub_radius}" length="${width}"/></geometry>
         <material name="rubber_black"/>
       </visual>
-      <xacro:intake_flap name="flap_0" angle="0.0" radius="${radius}" width="${width}"/>
-      <xacro:intake_flap name="flap_1" angle="${pi / 4.0}" radius="${radius}" width="${width}"/>
-      <xacro:intake_flap name="flap_2" angle="${pi / 2.0}" radius="${radius}" width="${width}"/>
-      <xacro:intake_flap name="flap_3" angle="${3.0 * pi / 4.0}" radius="${radius}" width="${width}"/>
-      <xacro:intake_flap name="flap_4" angle="${pi}" radius="${radius}" width="${width}"/>
-      <xacro:intake_flap name="flap_5" angle="${5.0 * pi / 4.0}" radius="${radius}" width="${width}"/>
-      <xacro:intake_flap name="flap_6" angle="${3.0 * pi / 2.0}" radius="${radius}" width="${width}"/>
-      <xacro:intake_flap name="flap_7" angle="${7.0 * pi / 4.0}" radius="${radius}" width="${width}"/>
     </link>
     <joint name="lift_wheel_joint" type="continuous">
@@ -103,50 +122,23 @@
     </joint>
     <gazebo reference="lift_wheel_link">
-      <mu1>1.5</mu1>
-      <mu2>1.5</mu2>
-      <!-- One contact sensor per paddle. Gazebo publishes the real physics
-           contact positions; gazebo_extras_node turns them into short-lived
-           red RViz markers and a /sim/roller_contact heartbeat. -->
-      <sensor name="roller_contact_0" type="contact">
-        <always_on>true</always_on><update_rate>100</update_rate>
-        <topic>/gz/roller_contact_0</topic>
-        <contact><collision>flap_0_col</collision></contact>
-      </sensor>
-      <sensor name="roller_contact_1" type="contact">
-        <always_on>true</always_on><update_rate>100</update_rate>
-        <topic>/gz/roller_contact_1</topic>
-        <contact><collision>flap_1_col</collision></contact>
-      </sensor>
-      <sensor name="roller_contact_2" type="contact">
-        <always_on>true</always_on><update_rate>100</update_rate>
-        <topic>/gz/roller_contact_2</topic>
-        <contact><collision>flap_2_col</collision></contact>
-      </sensor>
-      <sensor name="roller_contact_3" type="contact">
-        <always_on>true</always_on><update_rate>100</update_rate>
-        <topic>/gz/roller_contact_3</topic>
-        <contact><collision>flap_3_col</collision></contact>
-      </sensor>
-      <sensor name="roller_contact_4" type="contact">
-        <always_on>true</always_on><update_rate>100</update_rate>
-        <topic>/gz/roller_contact_4</topic>
-        <contact><collision>flap_4_col</collision></contact>
-      </sensor>
-      <sensor name="roller_contact_5" type="contact">
-        <always_on>true</always_on><update_rate>100</update_rate>
-        <topic>/gz/roller_contact_5</topic>
-        <contact><collision>flap_5_col</collision></contact>
-      </sensor>
-      <sensor name="roller_contact_6" type="contact">
-        <always_on>true</always_on><update_rate>100</update_rate>
-        <topic>/gz/roller_contact_6</topic>
-        <contact><collision>flap_6_col</collision></contact>
-      </sensor>
-      <sensor name="roller_contact_7" type="contact">
-        <always_on>true</always_on><update_rate>100</update_rate>
-        <topic>/gz/roller_contact_7</topic>
-        <contact><collision>flap_7_col</collision></contact>
-      </sensor>
+      <mu1>0.8</mu1>
+      <mu2>0.8</mu2>
     </gazebo>
+    <xacro:intake_paddle index="0" angle="${0 * pi / 4}" hub_r="${hub_radius}"
+        paddle_len="${paddle_length}" width="${width}" thickness="0.004"/>
+    <xacro:intake_paddle index="1" angle="${1 * pi / 4}" hub_r="${hub_radius}"
+        paddle_len="${paddle_length}" width="${width}" thickness="0.004"/>
+    <xacro:intake_paddle index="2" angle="${2 * pi / 4}" hub_r="${hub_radius}"
+        paddle_len="${paddle_length}" width="${width}" thickness="0.004"/>
+    <xacro:intake_paddle index="3" angle="${3 * pi / 4}" hub_r="${hub_radius}"
+        paddle_len="${paddle_length}" width="${width}" thickness="0.004"/>
+    <xacro:intake_paddle index="4" angle="${4 * pi / 4}" hub_r="${hub_radius}"
+        paddle_len="${paddle_length}" width="${width}" thickness="0.004"/>
+    <xacro:intake_paddle index="5" angle="${5 * pi / 4}" hub_r="${hub_radius}"
+        paddle_len="${paddle_length}" width="${width}" thickness="0.004"/>
+    <xacro:intake_paddle index="6" angle="${6 * pi / 4}" hub_r="${hub_radius}"
+        paddle_len="${paddle_length}" width="${width}" thickness="0.004"/>
+    <xacro:intake_paddle index="7" angle="${7 * pi / 4}" hub_r="${hub_radius}"
+        paddle_len="${paddle_length}" width="${width}" thickness="0.004"/>
   </xacro:macro>
   <!--

File: ros2_ws/src/tennis_robot/urdf/tennis_robot.urdf.xacro (robot description, xacro)
@@ -12,4 +12,5 @@
   <xacro:include filename="components/ir_beam.urdf.xacro"/>
   <xacro:include filename="components/body_panels.urdf.xacro"/>
+  <xacro:include filename="components/intake_debug_camera.urdf.xacro"/>
   <!-- ros2_control args. sim_mode swaps the hardware backend (sim vs real).
        controllers_config is the absolute path to controllers.yaml, injected by
@@ -17,4 +18,6 @@
   <xacro:arg name="sim_mode" default="true"/>
   <xacro:arg name="controllers_config" default="config/controllers.yaml"/>
+  <xacro:arg name="intake_roller_x_offset" default="0.0"/>
+  <xacro:arg name="intake_roller_z_offset" default="0.0"/>
   <xacro:property name="chassis_x" value="0.92"/>
   <xacro:property name="chassis_y" value="0.58"/>
@@ -39,14 +42,12 @@
   <xacro:property name="motor_radius" value="0.03"/>
   <xacro:property name="motor_length" value="0.10"/>
-  <!-- Roller-first intake (scripts/generate_curved_scoop_mesh.py): the paddled
+  <!-- Roller-first intake (scripts/generate_curved_scoop_mesh.py): the solid
        roller is the FIRST hard contact with the ball — the entire channel
        sits BEHIND the roller's leading edge. Envelope Ø90 x 180 mm, centre
-       105 mm above ground at x=0.55; the envelope reaches forward to
-       x=0.595 while the effective channel tip is at x=0.540 after the 15 mm
-       rearward tuning offset. A 66 mm ball meets the
-       paddle envelope at centre x=0.580 (contact 63 mm up the ball, above
-       its centre, pulling it in and down) ~14 mm before it could touch the
-       channel tip. The paddles then drive it around the rear-shifted channel
-       arc (nominal radius 105 mm),
+       112 mm above ground at x=0.60; the envelope reaches forward to
+       x=0.645 while the effective channel tip is at x=0.585. A 66 mm ball
+       therefore meets the roller before the rigid central scoop geometry.
+       The roller then drives it around the concentric channel arc
+       (nominal radius 108 mm),
        up the rear wall and over the deflector into the basket
        (funnel.urdf.xacro). The chassis plate has a matching front cutout
@@ -54,7 +55,11 @@
        centre 143.7 mm) never captured: the ball had to climb a passive
        37-degree ramp before the roller could even touch it. -->
-  <xacro:property name="intake_x" value="0.55"/>
-  <!-- base_link origin is 45 mm above ground: 0.105 - 0.045 -->
-  <xacro:property name="intake_z" value="0.060"/>
+  <!-- 50 mm forward of the original x=0.55 position so the roller, rather
+       than the scoop / funnel cheeks, is the first central hard contact. -->
+  <xacro:property name="intake_x" value="${0.60 + float($(arg intake_roller_x_offset))}"/>
+  <!-- base_link origin is 45 mm above ground: 0.112 - 0.045. With a 45 mm
+       roller radius this leaves 67 mm below the roller, so the rigid 66 mm
+       simulation ball can enter without initial interference. -->
+  <xacro:property name="intake_z" value="${0.067 + float($(arg intake_roller_z_offset))}"/>
   <xacro:property name="intake_radius" value="0.045"/>
   <xacro:property name="intake_width" value="0.18"/>
@@ -65,4 +70,18 @@
   <xacro:property name="camera_rpy" value="0 0.273 0"/>  <!-- forward-down tilt ~15.6deg; preserves the old world aim (0.22 cam + 0.053 chassis pitch) now that the chassis is level -->
   <xacro:property name="sensor_update_rate" value="31.25"/>
+  <!-- Sim-only debug camera (intake_debug_camera.urdf.xacro): mounted low and
+       to the LEFT of the intake mouth (base_link 0.5 0.13 -0.02, i.e. 25 mm
+       above ground, just inside the funnel cheek at y=0.145), aimed
+       diagonally inward-up-forward at the roller/lip nip. A head-on underside
+       mount is blocked by the scoop channel itself (verified: its depth
+       camera read a solid surface ~8 cm away filling the whole frame), so the
+       line of sight comes in from the side of the channel where nothing
+       obstructs it. yaw/pitch computed for the roller centre at effective
+       (0.615, 0, 0.107 ground); keep in sync if intake_* offsets change
+       materially. -->
+  <xacro:property name="intake_debug_camera_xyz" value="0.5 0.13 -0.02"/>
+  <!-- Aimed at the nip midpoint (0.607, 0, 0.075 ground) rather than the
+       roller centre, so the ball/roller/lip contact zone is centred. -->
+  <xacro:property name="intake_debug_camera_rpy" value="0 -0.289 -0.882"/>
   <!-- Throat beam crosses the intake mouth at ball-centre height (40 mm
        above ground = -0.005 in base_link), right where the paddles first
@@ -70,5 +89,8 @@
        partial-capture detection). Collection confirmation is the BASKET
        beam pair below — see gazebo_extras_node.py. -->
-  <xacro:property name="ir_x" value="0.575"/>
+  <!-- Trigger just before the ball reaches the roller envelope. The first
+       paddle contact is at ball-centre x≈0.597 m, so a beam behind that point
+       cannot start a stationary roller in time. -->
+  <xacro:property name="ir_x" value="0.620"/>
   <xacro:property name="ir_y" value="0.105"/>
   <xacro:property name="ir_z" value="-0.005"/>
@@ -146,4 +168,13 @@
       rpy="${camera_rpy}"
       update_rate="${sensor_update_rate}"/>
+  <!-- Sim-only: no real-hardware equivalent. -->
+  <xacro:if value="$(arg sim_mode)">
+    <xacro:intake_debug_camera
+        parent="base_link"
+        link_name="intake_debug_camera_link"
+        xyz="${intake_debug_camera_xyz}"
+        rpy="${intake_debug_camera_rpy}"
+        update_rate="${sensor_update_rate}"/>
+  </xacro:if>
   <!-- MPU6050 IMU near the chassis centre, axes aligned with base_link. Mainly
        used for yaw rate, which wheel odometry mis-estimates in skid-steer. -->
