Commit message: feat(mechanics): define fixed-motor compliant-tyre intake

File: ros2_ws/src/tennis_robot/urdf/components/drivetrain.urdf.xacro (robot description, xacro)
@@ -55,9 +55,16 @@
        the drive_wheel macro above). The old swivel-caster macro and its scrub
        resistance are gone. -->
-  <!-- Dual-wheel side-pinch intake (docs/dual-wheel-intake-design-el.md):
+  <!-- NOT_PHYSICAL_INTAKE_ARCHITECTURE:
+       LEGACY SIMULATION_ONLY_TYRE_COMPLIANCE_SURROGATE.
+       Physical architecture: both FIT0186 motors and both wheel centres are
+       fixed to the bridge. Compliance is tennis-ball + Trencher tyre/foam.
+       The prismatic link below moves the motor collision too, so it is not a
+       faithful physical surrogate and is prohibited as validation evidence.
+       It remains temporarily for traceability of older simulation runs.
+       Legacy dual-wheel simulation geometry; physical definition:
+       docs/mechanism/standalone-intake-fixed-motor-compliant-tyre.md.
        two side wheels, one each side of a centre corridor, both inner faces
-       driving rearward (-x). The wheel axis can be pitched slightly toward
-       +x for Phase 3 experiments, adding an upward component as the ball
-       enters the ramp. Each wheel hangs on a passive
+       driving rearward (-x). Both wheel axes share the same longitudinal X-Z
+       tilt and remain parallel in front view. Each wheel hangs on a passive
        prismatic y-carriage whose spring is patched into the generated SDF
        (scripts/generate_robot_urdf.py) — this is the lateral compliance a
@@ -77,6 +84,31 @@
         <material name="mount_gray"/>
       </visual>
-    </link>
-    <!-- Axis points OUTWARD (away from the corridor): rest position 0 is the
+      <!-- Coaxial purchased direct-drive hardware. Local +Z is wheel->motor;
+           common pitch maps both sides to (sin(tilt), 0, cos(tilt)).
+           Wheel centres are mirrored in Y, but the axes stay parallel. -->
+      <collision name="intake_adapter_col">
+        <origin xyz="${sin(tilt_rad) * 0.0435} 0 ${cos(tilt_rad) * 0.0435}"
+                rpy="0 ${tilt_rad} 0"/>
+        <geometry><cylinder radius="0.010" length="0.030"/></geometry>
+      </collision>
+      <visual name="intake_adapter_vis">
+        <origin xyz="${sin(tilt_rad) * 0.0435} 0 ${cos(tilt_rad) * 0.0435}"
+                rpy="0 ${tilt_rad} 0"/>
+        <geometry><cylinder radius="0.010" length="0.030"/></geometry>
+        <material name="safety_orange"/>
+      </visual>
+      <collision name="intake_motor_col">
+        <origin xyz="${sin(tilt_rad) * 0.0935} 0 ${cos(tilt_rad) * 0.0935}"
+                rpy="0 ${tilt_rad} 0"/>
+        <geometry><cylinder radius="0.015" length="0.070"/></geometry>
+      </collision>
+      <visual name="intake_motor_vis">
+        <origin xyz="${sin(tilt_rad) * 0.0935} 0 ${cos(tilt_rad) * 0.0935}"
+                rpy="0 ${tilt_rad} 0"/>
+        <geometry><cylinder radius="0.015" length="0.070"/></geometry>
+        <material name="mount_gray"/>
+      </visual>
+    </link>
+    <!-- LEGACY SURROGATE ONLY. Axis points OUTWARD (away from the corridor): rest position 0 is the
          inner stop (nominal 3 mm interference per side on a 66 mm ball); a
          passing ball compresses the "foam" by pushing the carriage outward

File: ros2_ws/src/tennis_robot/urdf/components/funnel.urdf.xacro (robot description, xacro)
@@ -1,6 +1,7 @@
 <?xml version="1.0" encoding="UTF-8"?>
 <robot xmlns:xacro="http://www.ros.org/wiki/xacro">
-  <!-- Dual-wheel intake support structure. Roles per
-       docs/dual-wheel-intake-design-el.md:
+  <!-- Funnel support for the NOT_PHYSICAL_INTAKE_ARCHITECTURE simulator.
+       Current physical definition:
+       docs/mechanism/standalone-intake-fixed-motor-compliant-tyre.md.
          cheeks -> centering (guide off-centre balls into the wheel throat)
          ramp   -> elevation + guidance toward the basket

File: ros2_ws/src/tennis_robot/urdf/components/ros2_control.urdf.xacro (robot description, xacro)
@@ -2,4 +2,6 @@
 <!--
   ros2_control hardware description for the tennis robot.
+  Intake carriage state is CURRENT_SIMULATION_SURROGATE and
+  NOT_PHYSICAL_INTAKE_ARCHITECTURE. Physical motors/wheel centres are fixed.
   This is the single contract between the high-level stack and the actuators.
   Swapping the <hardware> plugin (sim_mode arg) is the ONLY change required to

File: ros2_ws/src/tennis_robot/urdf/tennis_robot.urdf.xacro (robot description, xacro)
@@ -47,5 +47,6 @@
   <xacro:arg name="basket_floor_thickness" default="0.005"/>
   <xacro:arg name="basket_cad_support_details" default="false"/>
-  <!-- Dual-wheel intake tuning (docs/dual-wheel-intake-design-el.md).
+  <!-- NOT_PHYSICAL_INTAKE_ARCHITECTURE surrogate tuning. Physical definition:
+       docs/mechanism/standalone-intake-fixed-motor-compliant-tyre.md.
        Injected from INTAKE_WHEEL_* envs by scripts/generate_robot_urdf.py. -->
   <xacro:arg name="intake_wheel_radius" default="0.060"/>
@@ -110,5 +111,6 @@
   <xacro:property name="motor_length" value="0.10"/>
   <!-- Dual-wheel side-pinch intake: capture -> transport -> guide -> hopper
-       (docs/dual-wheel-intake-design-el.md). Two vertical-axis wheels flank a
+       (historical rationale archived under docs/archive/mechanism/intake/).
+       Two vertical-axis wheels flank a
        centre corridor at the nip plane; the funnel centres the ball, the
        wheels capture and transport it rearward, the ramp elevates it toward
@@ -130,6 +132,9 @@
   <xacro:property name="intake_wheel_height" value="${float($(arg intake_wheel_width))}"/>
   <xacro:property name="intake_wheel_z" value="${0.070 - base_link_height}"/>
-  <!-- Outward carriage travel: 8 mm absorbs the 3 mm/side nominal
-       interference with margin. Spring k is SDF-patched by the generator. -->
+  <!-- NOT_PHYSICAL_INTAKE_ARCHITECTURE:
+       SIMULATION_ONLY_TYRE_COMPLIANCE_SURROGATE, legacy rigid-wheel model.
+       The physical FIT0186 motors and wheel centres are fixed to the bridge;
+       no carriage exists. This 8 mm DOF must not be used as physical-design
+       or validation evidence and must be replaced by calibrated tyre contact. -->
   <xacro:property name="intake_carriage_travel" value="0.008"/>
   <xacro:property name="intake_assist_x" value="${float($(arg intake_assist_x))}"/>
