Commit message: Survey v2 foundation: LiDAR extraction + coverage (tested offline) — rollback point before replacing dead-reckoning FSM

File: ros2_ws/src/tennis_robot/urdf/components/body_panels.urdf.xacro (robot description, xacro)
@@ -14,5 +14,7 @@
         <origin xyz="0.44 0.18 0.22" rpy="0 0 0"/>
         <geometry><box size="0.04 0.22 0.44"/></geometry>
-        <material name="body_white"/>
+        <material name="body_white">
+          <color rgba="0.92 0.92 0.92 1.0"/>
+        </material>
       </visual>
       <visual name="front_right_housing">
