Commit message: robot refinment

File: ros2_ws/src/tennis_robot/urdf/components/base.urdf.xacro (robot description, xacro)
@@ -12,5 +12,5 @@
   <xacro:macro name="cylinder_inertial" params="mass radius length axis">
     <inertial>
-      <mass value="${mass}"/>
+      <mass value="${mass}"/> [cite: 17]
       <xacro:if value="${axis == 'y'}">
         <inertia
@@ -19,5 +19,5 @@
             izz="${mass * (3.0 * radius * radius + length * length) / 12.0}"/>
       </xacro:if>
-      <xacro:unless value="${axis == 'y'}">
+      <xacro:unless value="${axis == 'y'}"> [cite: 18]
         <inertia
             ixx="${mass * (3.0 * radius * radius + length * length) / 12.0}" ixy="0" ixz="0"
@@ -28,4 +28,10 @@
   </xacro:macro>
   <xacro:macro name="tennis_robot_base" params="chassis_x chassis_y chassis_z chassis_mass">
+    <link name="base_footprint"/>
+    <joint name="base_footprint_joint" type="fixed">
+      <parent link="base_footprint"/>
+      <child link="base_link"/>
+      <origin xyz="0 0 0.09" rpy="0 0.053 0"/>
+    </joint>
     <link name="base_link">
       <xacro:box_inertial mass="${chassis_mass}" x="${chassis_x}" y="${chassis_y}" z="${chassis_z}"/>
@@ -39,48 +45,48 @@
         <material name="plywood"/>
       </visual>
-      <visual name="front_left_cheek_vis">
-        <origin xyz="${chassis_x / 2.0} ${0.30 / 2.0 + (chassis_y - 0.30) / 4.0} 0.17" rpy="0 0 0"/>
-        <geometry><box size="0.025 ${(chassis_y - 0.30) / 2.0} 0.14"/></geometry>
-        <material name="mount_gray"/>
+      <visual name="front_left_cheek_vis"> [cite: 20]
+        <origin xyz="${chassis_x / 2.0} ${0.30 / 2.0 + (chassis_y - 0.30) / 4.0} 0.077" rpy="0 0 0"/> [cite: 20]
+        <geometry><box size="0.025 ${(chassis_y - 0.30) / 2.0} 0.14"/></geometry> [cite: 20]
+        <material name="mount_gray"/> [cite: 20]
       </visual>
-      <visual name="front_right_cheek_vis">
-        <origin xyz="${chassis_x / 2.0} ${-(0.30 / 2.0 + (chassis_y - 0.30) / 4.0)} 0.17" rpy="0 0 0"/>
-        <geometry><box size="0.025 ${(chassis_y - 0.30) / 2.0} 0.14"/></geometry>
-        <material name="mount_gray"/>
+      <visual name="front_right_cheek_vis"> [cite: 20]
+        <origin xyz="${chassis_x / 2.0} ${-(0.30 / 2.0 + (chassis_y - 0.30) / 4.0)} 0.077" rpy="0 0 0"/> [cite: 20]
+        <geometry><box size="0.025 ${(chassis_y - 0.30) / 2.0} 0.14"/></geometry> [cite: 20, 21]
+        <material name="mount_gray"/> [cite: 21]
       </visual>
-      <visual name="rear_wall_vis">
-        <origin xyz="${-chassis_x / 2.0} 0 0.17" rpy="0 0 0"/>
-        <geometry><box size="0.025 ${chassis_y} 0.14"/></geometry>
-        <material name="mount_gray"/>
+      <visual name="rear_wall_vis"> [cite: 21]
+        <origin xyz="${-chassis_x / 2.0} 0 0.077" rpy="0 0 0"/> [cite: 21]
+        <geometry><box size="0.025 ${chassis_y} 0.14"/></geometry> [cite: 21]
+        <material name="mount_gray"/> [cite: 21]
       </visual>
-      <visual name="left_wall_vis">
-        <origin xyz="0 ${chassis_y / 2.0} 0.17" rpy="0 0 0"/>
-        <geometry><box size="${chassis_x} 0.025 0.14"/></geometry>
-        <material name="mount_gray"/>
+      <visual name="left_wall_vis"> [cite: 21]
+        <origin xyz="0 ${chassis_y / 2.0} 0.077" rpy="0 0 0"/> [cite: 21]
+        <geometry><box size="${chassis_x} 0.025 0.14"/></geometry> [cite: 22]
+        <material name="mount_gray"/> [cite: 22]
       </visual>
-      <visual name="right_wall_vis">
-        <origin xyz="0 ${-chassis_y / 2.0} 0.17" rpy="0 0 0"/>
-        <geometry><box size="${chassis_x} 0.025 0.14"/></geometry>
-        <material name="mount_gray"/>
+      <visual name="right_wall_vis"> [cite: 22]
+        <origin xyz="0 ${-chassis_y / 2.0} 0.077" rpy="0 0 0"/> [cite: 22]
+        <geometry><box size="${chassis_x} 0.025 0.14"/></geometry> [cite: 22]
+        <material name="mount_gray"/> [cite: 22]
       </visual>
-      <visual name="elec_vis">
-        <origin xyz="-0.13 0 0.13" rpy="0 0 0"/>
-        <geometry><box size="0.34 0.26 0.12"/></geometry>
-        <material name="anthracite"/>
+      <visual name="left_axle_bracket_vis"> [cite: 22]
+        <origin xyz="-0.35 0.32 0" rpy="0 0 0"/> [cite: 23]
+        <geometry><box size="0.065 0.060 0.018"/></geometry> [cite: 23]
+        <material name="mount_gray"/> [cite: 23]
       </visual>
-      <visual name="intake_left_guide_vis">
-        <origin xyz="0.52 ${0.30 / 2.0 + (0.52 - 0.30) / 4.0} -0.06" rpy="0 0 0"/>
-        <geometry><box size="0.04 ${(0.52 - 0.30) / 2.0} 0.14"/></geometry>
-        <material name="intake_orange"/>
+      <visual name="right_axle_bracket_vis"> [cite: 23]
+        <origin xyz="-0.35 -0.32 0" rpy="0 0 0"/> [cite: 23]
+        <geometry><box size="0.065 0.060 0.018"/></geometry> [cite: 23]
+        <material name="mount_gray"/> [cite: 23]
       </visual>
-      <visual name="intake_right_guide_vis">
-        <origin xyz="0.52 ${-(0.30 / 2.0 + (0.52 - 0.30) / 4.0)} -0.06" rpy="0 0 0"/>
-        <geometry><box size="0.04 ${(0.52 - 0.30) / 2.0} 0.14"/></geometry>
-        <material name="intake_orange"/>
+      <visual name="elec_vis"> [cite: 23]
+        <origin xyz="-0.13 0 0.067" rpy="0 0 0"/> [cite: 23, 24]
+        <geometry><box size="0.34 0.26 0.12"/></geometry> [cite: 24]
+        <material name="anthracite"/> [cite: 24]
       </visual>
-      <visual name="ir_beam_line_vis">
-        <origin xyz="0.54 0 -0.14" rpy="1.5708 0 0"/>
-        <geometry><cylinder radius="0.003" length="0.21"/></geometry>
-        <material name="ir_beam_red"/>
+      <visual name="ir_beam_line_vis"> [cite: 24]
+        <origin xyz="0.54 0 0.053" rpy="1.5708 0 0"/> [cite: 24]
+        <geometry><cylinder radius="0.003" length="0.21"/></geometry> [cite: 24]
+        <material name="ir_beam_red"/> [cite: 24]
       </visual>
     </link>

File: ros2_ws/src/tennis_robot/urdf/components/drivetrain.urdf.xacro (robot description, xacro)
@@ -116,4 +116,8 @@
         <min_linear_acceleration>-${max_linear_acceleration}</min_linear_acceleration>
         <max_angular_acceleration>${max_angular_acceleration}</max_angular_acceleration>
+        <min_angular_acceleration>-${max_angular_acceleration}</min_angular_acceleration>
+      </plugin>
+      <plugin filename="gz-sim-joint-state-publisher-system" name="gz::sim::systems::JointStatePublisher">
+        <topic>/joint_states</topic>
       </plugin>
       <plugin filename="gz-sim-joint-controller-system" name="gz::sim::systems::JointController">

File: ros2_ws/src/tennis_robot/urdf/components/lidar.urdf.xacro (robot description, xacro)
@@ -8,6 +8,6 @@
       </inertial>
       <visual name="mast_vis">
-        <origin xyz="0 0 -0.26" rpy="0 0 0"/>
-        <geometry><box size="0.025 0.025 0.49"/></geometry>
+        <origin xyz="0 0 -0.30" rpy="0 0 0"/>
+        <geometry><box size="0.025 0.025 0.57"/></geometry>
         <material name="anthracite"/>
       </visual>

File: ros2_ws/src/tennis_robot/urdf/components/materials.urdf.xacro (robot description, xacro)
@@ -13,4 +13,7 @@
     <color rgba="0.30 0.32 0.36 1"/>
   </material>
+  <material name="basket_gray">
+    <color rgba="0.42 0.45 0.48 0.65"/>
+  </material>
   <material name="rubber_black">
     <color rgba="0.04 0.04 0.04 1"/>

File: ros2_ws/src/tennis_robot/urdf/tennis_robot.urdf.xacro (robot description, xacro)
@@ -3,16 +3,19 @@
   <xacro:include filename="components/materials.urdf.xacro"/>
   <xacro:include filename="components/base.urdf.xacro"/>
+  <xacro:include filename="components/funnel.urdf.xacro"/>
+  <xacro:include filename="components/basket.urdf.xacro"/>
   <xacro:include filename="components/drivetrain.urdf.xacro"/>
   <xacro:include filename="components/lidar.urdf.xacro"/>
   <xacro:include filename="components/oak_d.urdf.xacro"/>
   <xacro:include filename="components/ir_beam.urdf.xacro"/>
-  <xacro:property name="chassis_x" value="0.92"/>
+  <xacro:include filename="components/body_panels.urdf.xacro"/>
+<xacro:property name="chassis_x" value="0.92"/>
   <xacro:property name="chassis_y" value="0.58"/>
-  <xacro:property name="chassis_z" value="0.20"/>
+  <xacro:property name="chassis_z" value="0.014"/>
   <xacro:property name="chassis_mass" value="7.2"/>
   <xacro:property name="wheel_x" value="-0.35"/>
   <xacro:property name="wheel_y" value="0.35"/>
   <xacro:property name="wheel_z" value="-0.09"/>
-  <xacro:property name="wheel_radius" value="0.11"/>
+  <xacro:property name="wheel_radius" value="0.09"/>
   <xacro:property name="wheel_width" value="0.08"/>
   <xacro:property name="wheel_mass" value="0.25"/>
@@ -20,18 +23,21 @@
   <xacro:property name="caster_x" value="0.31"/>
   <xacro:property name="caster_y" value="0.35"/>
-  <xacro:property name="caster_z" value="-0.145"/>
+  <xacro:property name="caster_z" value="-0.055"/>
   <xacro:property name="caster_radius" value="0.055"/>
   <xacro:property name="intake_x" value="0.62"/>
-  <xacro:property name="intake_z" value="-0.065"/>
-  <xacro:property name="intake_radius" value="0.06"/>
-  <xacro:property name="intake_width" value="0.54"/>
-  <xacro:property name="lidar_xyz" value="-0.08 0 0.52"/>
+  <xacro:property name="intake_z" value="0.095"/>
+  <xacro:property name="intake_radius" value="0.03"/>
+  <xacro:property name="intake_width" value="0.24"/>
+  <xacro:property name="lidar_xyz" value="-0.08 0 0.713"/>
   <xacro:property name="lidar_rpy" value="0 0 0"/>
-  <xacro:property name="camera_xyz" value="0.535 0 0.25"/>
+  <xacro:property name="camera_xyz" value="0.535 0 0.443"/>
   <xacro:property name="camera_rpy" value="0 0.22 0"/>
   <xacro:property name="sensor_update_rate" value="31.25"/>
   <xacro:property name="ir_x" value="0.54"/>
   <xacro:property name="ir_y" value="0.105"/>
-  <xacro:property name="ir_z" value="-0.14"/>
+  <xacro:property name="ir_z" value="0.053"/>
+  <xacro:property name="basket_ir_x" value="0.28"/>
+  <xacro:property name="basket_ir_y" value="0.105"/>
+  <xacro:property name="basket_ir_z" value="0.113"/>
   <xacro:property name="max_linear_acceleration" value="2.0"/>
   <xacro:property name="max_angular_acceleration" value="4.0"/>
@@ -63,6 +69,8 @@
       width="${intake_width}"
       mass="0.20"/>
-  <xacro:caster name="front_left" x="${caster_x}" y="-${caster_y}" z="${caster_z}" radius="${caster_radius}"/>
-  <xacro:caster name="front_right" x="${caster_x}" y="${caster_y}" z="${caster_z}" radius="${caster_radius}"/>
+<xacro:intake_funnel parent="base_link" chassis_z="${chassis_z}"/> [cite: 4]
+  <xacro:ball_basket parent="base_link"/> [cite: 4]
+  <xacro:caster name="front_left" x="${caster_x}" y="-${caster_y}" z="${caster_z}" radius="${caster_radius}"/> [cite: 4]
+  <xacro:caster name="front_right" x="${caster_x}" y="${caster_y}" z="${caster_z}" radius="${caster_radius}"/> [cite: 4]
   <xacro:rplidar_c1_mount
       parent="base_link"
@@ -70,5 +78,5 @@
       xyz="${lidar_xyz}"
       rpy="${lidar_rpy}"
-      update_rate="${sensor_update_rate}"/>
+      update_rate="${sensor_update_rate}"/> [cite: 4]
   <xacro:oak_d_lite_mount
       parent="base_link"
@@ -76,5 +84,5 @@
       xyz="${camera_xyz}"
       rpy="${camera_rpy}"
-      update_rate="${sensor_update_rate}"/>
+      update_rate="${sensor_update_rate}"/> [cite: 4, 5]
   <xacro:ir_beam_sensor
       parent="base_link"
@@ -84,5 +92,5 @@
       rpy="0 0 -1.5708"
       topic="/gz/ir_left"
-      update_rate="${sensor_update_rate}"/>
+      update_rate="${sensor_update_rate}"/> [cite: 5]
   <xacro:ir_beam_sensor
       parent="base_link"
@@ -93,4 +101,20 @@
       topic="/gz/ir_right"
       update_rate="${sensor_update_rate}"/>
+  <xacro:ir_beam_sensor
+      parent="base_link"
+      link_name="basket_ir_left_link"
+      joint_name="basket_ir_left_joint"
+      xyz="${basket_ir_x} -${basket_ir_y} ${basket_ir_z}"
+      rpy="0 0 -1.5708"
+      topic="/gz/basket_ir_left"
+      update_rate="${sensor_update_rate}"/> [cite: 5, 6]
+  <xacro:ir_beam_sensor
+      parent="base_link"
+      link_name="basket_ir_right_link"
+      joint_name="basket_ir_right_joint"
+      xyz="${basket_ir_x} ${basket_ir_y} ${basket_ir_z}"
+      rpy="0 0 1.5708"
+      topic="/gz/basket_ir_right"
+      update_rate="${sensor_update_rate}"/> [cite: 6]
   <xacro:diff_drive_plugin
       wheel_separation="${wheel_separation}"
@@ -98,4 +122,5 @@
       update_rate="${sensor_update_rate}"
       max_linear_acceleration="${max_linear_acceleration}"
-      max_angular_acceleration="${max_angular_acceleration}"/>
+      max_angular_acceleration="${max_angular_acceleration}"/> [cite: 6]
+<xacro:robot_body_panels parent="base_link" chassis_z="${chassis_z}"/>
 </robot>
