Commit message: Adopt ros2_control + Nav2/SLAM stack for autonomous survey
Robot control:
- Migrate from Gazebo plugins to ros2_control (gz_ros2_control sim backend,
  swappable for real hardware); diff_drive_controller + joint_state_broadcaster
  + lift wheel velocity controller; drive_actuator_node + twist_mux arbiter.

Sensors:
- Canonical sensor topic contract (/scan, /camera/*) shared sim/real;
  real_sensors.launch.py for rplidar + OAK-D drivers.

Autonomous survey:
- slam_toolbox mapping + Nav2 (RPP controller, costmaps from /scan) +
  explore_lite frontier exploration; autonomous_survey.launch.py orchestrator.

Fixes:
- Front caster geometry: coplanar contact at design pitch + self-aligning trail.
- CycloneDDS MaxAutoParticipantIndex (free participant index error).
- Strip NUL bytes + stray [cite] markers that broke URDF xacro rendering.

Docker: build gz_ros2_control + explore_lite from source; add nav2/slam deps.

Also sweeps in pre-existing working-tree changes (controller_node.py,
cad/cyber_shell_panels.scad, lidar_survey_v2.py).

File: ros2_ws/src/tennis_robot/urdf/components/base.urdf.xacro (robot description, xacro)
@@ -12,5 +12,5 @@
   <xacro:macro name="cylinder_inertial" params="mass radius length axis">
     <inertial>
-      <mass value="${mass}"/> [cite: 17]
+      <mass value="${mass}"/>
       <xacro:if value="${axis == 'y'}">
         <inertia
@@ -19,5 +19,5 @@
             izz="${mass * (3.0 * radius * radius + length * length) / 12.0}"/>
       </xacro:if>
-      <xacro:unless value="${axis == 'y'}"> [cite: 18]
+      <xacro:unless value="${axis == 'y'}">
         <inertia
             ixx="${mass * (3.0 * radius * radius + length * length) / 12.0}" ixy="0" ixz="0"
@@ -45,48 +45,48 @@
         <material name="plywood"/>
       </visual>
-      <visual name="front_left_cheek_vis"> [cite: 20]
-        <origin xyz="${chassis_x / 2.0} ${0.30 / 2.0 + (chassis_y - 0.30) / 4.0} 0.077" rpy="0 0 0"/> [cite: 20]
-        <geometry><box size="0.025 ${(chassis_y - 0.30) / 2.0} 0.14"/></geometry> [cite: 20]
-        <material name="mount_gray"/> [cite: 20]
+      <visual name="front_left_cheek_vis">
+        <origin xyz="${chassis_x / 2.0} ${0.30 / 2.0 + (chassis_y - 0.30) / 4.0} 0.077" rpy="0 0 0"/>
+        <geometry><box size="0.025 ${(chassis_y - 0.30) / 2.0} 0.14"/></geometry>
+        <material name="mount_gray"/>
       </visual>
-      <visual name="front_right_cheek_vis"> [cite: 20]
-        <origin xyz="${chassis_x / 2.0} ${-(0.30 / 2.0 + (chassis_y - 0.30) / 4.0)} 0.077" rpy="0 0 0"/> [cite: 20]
-        <geometry><box size="0.025 ${(chassis_y - 0.30) / 2.0} 0.14"/></geometry> [cite: 20, 21]
-        <material name="mount_gray"/> [cite: 21]
+      <visual name="front_right_cheek_vis">
+        <origin xyz="${chassis_x / 2.0} ${-(0.30 / 2.0 + (chassis_y - 0.30) / 4.0)} 0.077" rpy="0 0 0"/>
+        <geometry><box size="0.025 ${(chassis_y - 0.30) / 2.0} 0.14"/></geometry>
+        <material name="mount_gray"/>
       </visual>
-      <visual name="rear_wall_vis"> [cite: 21]
-        <origin xyz="${-chassis_x / 2.0} 0 0.077" rpy="0 0 0"/> [cite: 21]
-        <geometry><box size="0.025 ${chassis_y} 0.14"/></geometry> [cite: 21]
-        <material name="mount_gray"/> [cite: 21]
+      <visual name="rear_wall_vis">
+        <origin xyz="${-chassis_x / 2.0} 0 0.077" rpy="0 0 0"/>
+        <geometry><box size="0.025 ${chassis_y} 0.14"/></geometry>
+        <material name="mount_gray"/>
       </visual>
-      <visual name="left_wall_vis"> [cite: 21]
-        <origin xyz="0 ${chassis_y / 2.0} 0.077" rpy="0 0 0"/> [cite: 21]
-        <geometry><box size="${chassis_x} 0.025 0.14"/></geometry> [cite: 22]
-        <material name="mount_gray"/> [cite: 22]
+      <visual name="left_wall_vis">
+        <origin xyz="0 ${chassis_y / 2.0} 0.077" rpy="0 0 0"/>
+        <geometry><box size="${chassis_x} 0.025 0.14"/></geometry>
+        <material name="mount_gray"/>
       </visual>
-      <visual name="right_wall_vis"> [cite: 22]
-        <origin xyz="0 ${-chassis_y / 2.0} 0.077" rpy="0 0 0"/> [cite: 22]
-        <geometry><box size="${chassis_x} 0.025 0.14"/></geometry> [cite: 22]
-        <material name="mount_gray"/> [cite: 22]
+      <visual name="right_wall_vis">
+        <origin xyz="0 ${-chassis_y / 2.0} 0.077" rpy="0 0 0"/>
+        <geometry><box size="${chassis_x} 0.025 0.14"/></geometry>
+        <material name="mount_gray"/>
       </visual>
-      <visual name="left_axle_bracket_vis"> [cite: 22]
-        <origin xyz="-0.35 0.32 0" rpy="0 0 0"/> [cite: 23]
-        <geometry><box size="0.065 0.060 0.018"/></geometry> [cite: 23]
-        <material name="mount_gray"/> [cite: 23]
+      <visual name="left_axle_bracket_vis">
+        <origin xyz="-0.35 0.32 0" rpy="0 0 0"/>
+        <geometry><box size="0.065 0.060 0.018"/></geometry>
+        <material name="mount_gray"/>
       </visual>
-      <visual name="right_axle_bracket_vis"> [cite: 23]
-        <origin xyz="-0.35 -0.32 0" rpy="0 0 0"/> [cite: 23]
-        <geometry><box size="0.065 0.060 0.018"/></geometry> [cite: 23]
-        <material name="mount_gray"/> [cite: 23]
+      <visual name="right_axle_bracket_vis">
+        <origin xyz="-0.35 -0.32 0" rpy="0 0 0"/>
+        <geometry><box size="0.065 0.060 0.018"/></geometry>
+        <material name="mount_gray"/>
       </visual>
-      <visual name="elec_vis"> [cite: 23]
-        <origin xyz="-0.13 0 0.067" rpy="0 0 0"/> [cite: 23, 24]
-        <geometry><box size="0.34 0.26 0.12"/></geometry> [cite: 24]
-        <material name="anthracite"/> [cite: 24]
+      <visual name="elec_vis">
+        <origin xyz="-0.13 0 0.067" rpy="0 0 0"/>
+        <geometry><box size="0.34 0.26 0.12"/></geometry>
+        <material name="anthracite"/>
       </visual>
-      <visual name="ir_beam_line_vis"> [cite: 24]
-        <origin xyz="0.54 0 0.053" rpy="1.5708 0 0"/> [cite: 24]
-        <geometry><cylinder radius="0.003" length="0.21"/></geometry> [cite: 24]
-        <material name="ir_beam_red"/> [cite: 24]
+      <visual name="ir_beam_line_vis">
+        <origin xyz="0.54 0 0.053" rpy="1.5708 0 0"/>
+        <geometry><cylinder radius="0.003" length="0.21"/></geometry>
+        <material name="ir_beam_red"/>
       </visual>
     </link>

File: ros2_ws/src/tennis_robot/urdf/components/drivetrain.urdf.xacro (robot description, xacro)
@@ -27,5 +27,5 @@
     </gazebo>
   </xacro:macro>
-  <xacro:macro name="caster" params="name x y z radius">
+  <xacro:macro name="caster" params="name x y z radius width:=0.030 trail:=0.0">
     <link name="${name}_caster_swivel_link">
       <inertial>
@@ -52,12 +52,12 @@
     </joint>
     <link name="${name}_caster_wheel_link">
-      <xacro:cylinder_inertial mass="0.05" radius="${radius}" length="0.030" axis="y"/>
+      <xacro:cylinder_inertial mass="0.05" radius="${radius}" length="${width}" axis="y"/>
       <collision name="col">
         <origin xyz="0 0 0" rpy="1.5708 0 0"/>
-        <geometry><cylinder radius="${radius}" length="0.030"/></geometry>
+        <geometry><cylinder radius="${radius}" length="${width}"/></geometry>
       </collision>
       <visual name="vis">
         <origin xyz="0 0 0" rpy="1.5708 0 0"/>
-        <geometry><cylinder radius="${radius}" length="0.030"/></geometry>
+        <geometry><cylinder radius="${radius}" length="${width}"/></geometry>
         <material name="rubber_black"/>
       </visual>
@@ -66,5 +66,7 @@
       <parent link="${name}_caster_swivel_link"/>
       <child link="${name}_caster_wheel_link"/>
-      <origin xyz="0 0 -${radius}" rpy="0 0 0"/>
+      <!-- trail: wheel contact sits behind the vertical swivel axis so the
+           caster self-aligns with the direction of travel (no scrub/shimmy). -->
+      <origin xyz="-${trail} 0 -${radius}" rpy="0 0 0"/>
       <axis xyz="0 1 0"/>
       <dynamics damping="0.001" friction="0.0"/>
@@ -100,31 +102,11 @@
     </gazebo>
   </xacro:macro>
-  <xacro:macro name="diff_drive_plugin" params="wheel_separation wheel_radius update_rate max_linear_acceleration max_angular_acceleration">
-    <gazebo>
-      <plugin filename="gz-sim-diff-drive-system" name="gz::sim::systems::DiffDrive">
-        <left_joint>left_wheel_joint</left_joint>
-        <right_joint>right_wheel_joint</right_joint>
-        <wheel_separation>${wheel_separation}</wheel_separation>
-        <wheel_radius>${wheel_radius}</wheel_radius>
-        <odom_publish_frequency>${update_rate}</odom_publish_frequency>
-        <topic>/cmd_vel</topic>
-        <odom_topic>/odom</odom_topic>
-        <tf_topic>/tf</tf_topic>
-        <frame_id>odom</frame_id>
-        <child_frame_id>base_link</child_frame_id>
-        <max_linear_acceleration>${max_linear_acceleration}</max_linear_acceleration>
-        <min_linear_acceleration>-${max_linear_acceleration}</min_linear_acceleration>
-        <max_angular_acceleration>${max_angular_acceleration}</max_angular_acceleration>
-        <min_angular_acceleration>-${max_angular_acceleration}</min_angular_acceleration>
-      </plugin>
-      <plugin filename="gz-sim-joint-state-publisher-system" name="gz::sim::systems::JointStatePublisher">
-        <topic>/joint_states</topic>
-      </plugin>
-      <plugin filename="gz-sim-joint-controller-system" name="gz::sim::systems::JointController">
-        <joint_name>lift_wheel_joint</joint_name>
-        <use_force_commands>false</use_force_commands>
-        <topic>/lift_wheel/cmd</topic>
-      </plugin>
-    </gazebo>
-  </xacro:macro>
+  <!--
+    NOTE: The legacy Gazebo control plugins (gz-sim-diff-drive-system,
+    gz-sim-joint-state-publisher-system, gz-sim-joint-controller-system) were
+    removed during the ros2_control migration. Wheel + intake actuation is now
+    owned by ros2_control via components/ros2_control.urdf.xacro. Odometry,
+    /tf and /joint_states are published by diff_drive_controller +
+    joint_state_broadcaster instead of these plugins.
+  -->
 </robot>

File: ros2_ws/src/tennis_robot/urdf/tennis_robot.urdf.xacro (robot description, xacro)
@@ -6,8 +6,14 @@
   <xacro:include filename="components/basket.urdf.xacro"/>
   <xacro:include filename="components/drivetrain.urdf.xacro"/>
+  <xacro:include filename="components/ros2_control.urdf.xacro"/>
   <xacro:include filename="components/lidar.urdf.xacro"/>
   <xacro:include filename="components/oak_d.urdf.xacro"/>
   <xacro:include filename="components/ir_beam.urdf.xacro"/>
   <xacro:include filename="components/body_panels.urdf.xacro"/>
+  <!-- ros2_control args. sim_mode swaps the hardware backend (sim vs real).
+       controllers_config is the absolute path to controllers.yaml, injected by
+       scripts/generate_robot_urdf.py / the launch file. -->
+  <xacro:arg name="sim_mode" default="true"/>
+  <xacro:arg name="controllers_config" default="config/controllers.yaml"/>
 <xacro:property name="chassis_x" value="0.92"/>
   <xacro:property name="chassis_y" value="0.58"/>
@@ -21,8 +27,14 @@
   <xacro:property name="wheel_mass" value="0.25"/>
   <xacro:property name="wheel_separation" value="${2.0 * wheel_y}"/>
+  <!-- Front swivel casters. Sized for a real clay court (rolling wheel, not a
+       skid/ball). caster_z chosen so the wheel contact is coplanar with the
+       drive wheels at the 3deg design pitch: contact_z = caster_z - caster_radius.
+       Set caster_radius/width/trail to the actual caster hardware you fit. -->
   <xacro:property name="caster_x" value="0.31"/>
   <xacro:property name="caster_y" value="0.35"/>
-  <xacro:property name="caster_z" value="-0.055"/>
-  <xacro:property name="caster_radius" value="0.055"/>
+  <xacro:property name="caster_radius" value="0.0625"/>   <!-- 125 mm wheel dia -->
+  <xacro:property name="caster_width" value="0.035"/>
+  <xacro:property name="caster_trail" value="0.025"/>     <!-- self-aligning offset -->
+  <xacro:property name="caster_z" value="-0.0825"/>       <!-- contact = -0.145 m (coplanar) -->
   <xacro:property name="intake_x" value="0.62"/>
   <xacro:property name="intake_z" value="0.095"/>
@@ -69,8 +81,8 @@
       width="${intake_width}"
       mass="0.20"/>
-<xacro:intake_funnel parent="base_link" chassis_z="${chassis_z}"/> [cite: 4]
-  <xacro:ball_basket parent="base_link"/> [cite: 4]
-  <xacro:caster name="front_left" x="${caster_x}" y="-${caster_y}" z="${caster_z}" radius="${caster_radius}"/> [cite: 4]
-  <xacro:caster name="front_right" x="${caster_x}" y="${caster_y}" z="${caster_z}" radius="${caster_radius}"/> [cite: 4]
+<xacro:intake_funnel parent="base_link" chassis_z="${chassis_z}"/>
+  <xacro:ball_basket parent="base_link"/>
+  <xacro:caster name="front_left" x="${caster_x}" y="-${caster_y}" z="${caster_z}" radius="${caster_radius}" width="${caster_width}" trail="${caster_trail}"/>
+  <xacro:caster name="front_right" x="${caster_x}" y="${caster_y}" z="${caster_z}" radius="${caster_radius}" width="${caster_width}" trail="${caster_trail}"/>
   <xacro:rplidar_c1_mount
       parent="base_link"
@@ -78,5 +90,5 @@
       xyz="${lidar_xyz}"
       rpy="${lidar_rpy}"
-      update_rate="${sensor_update_rate}"/> [cite: 4]
+      update_rate="${sensor_update_rate}"/>
   <xacro:oak_d_lite_mount
       parent="base_link"
@@ -84,5 +96,5 @@
       xyz="${camera_xyz}"
       rpy="${camera_rpy}"
-      update_rate="${sensor_update_rate}"/> [cite: 4, 5]
+      update_rate="${sensor_update_rate}"/>
   <xacro:ir_beam_sensor
       parent="base_link"
@@ -92,5 +104,5 @@
       rpy="0 0 -1.5708"
       topic="/gz/ir_left"
-      update_rate="${sensor_update_rate}"/> [cite: 5]
+      update_rate="${sensor_update_rate}"/>
   <xacro:ir_beam_sensor
       parent="base_link"
@@ -108,5 +120,5 @@
       rpy="0 0 -1.5708"
       topic="/gz/basket_ir_left"
-      update_rate="${sensor_update_rate}"/> [cite: 5, 6]
+      update_rate="${sensor_update_rate}"/>
   <xacro:ir_beam_sensor
       parent="base_link"
@@ -116,11 +128,8 @@
       rpy="0 0 1.5708"
       topic="/gz/basket_ir_right"
-      update_rate="${sensor_update_rate}"/> [cite: 6]
-  <xacro:diff_drive_plugin
-      wheel_separation="${wheel_separation}"
-      wheel_radius="${wheel_radius}"
-      update_rate="${sensor_update_rate}"
-      max_linear_acceleration="${max_linear_acceleration}"
-      max_angular_acceleration="${max_angular_acceleration}"/> [cite: 6]
+      update_rate="${sensor_update_rate}"/>
+  <xacro:tennis_robot_ros2_control
+      sim_mode="$(arg sim_mode)"
+      controllers_config="$(arg controllers_config)"/>
 <xacro:robot_body_panels parent="base_link" chassis_z="${chassis_z}"/>
 </robot>
