Commit message: 4WD skid-steer redesign: level chassis, IMU+EKF fusion, survey net-crossing
- Drivetrain: 2WD+casters -> 4WD skid-steer (4x 180mm driven wheels, 2/side,
  symmetric, no casters); level (un-pitched) chassis; base_footprint on ground
- ros2_control + diff_drive_controller: 4 wheel joints (2 per side);
  wheel_separation 0.70 -> 1.0 (skid-steer odom correction); EKF owns odom TF
- Sensors: lowered LiDAR so the scan plane (world ~0.713m) hits the net again
  (was scanning over it -> drove through); camera tilt preserved; added MPU6050
  IMU + robot_localization EKF fusing wheel vx + IMU yaw-rate
- Survey: net-aware crossing (stop_short flag) so the net is not mistaken for the
  target fence; faster turns (mu 5.0->1.2, TURN_SPEED 0.9, DRIVE_SPEED 0.75);
  return-home waypoint + completion notice
- CAD: 4 motor pods, casters removed; docs + CLAUDE.md updated to 4WD
- Dockerfile: install robot_localization; bump TENNIS_ROBOT_VER

File: ros2_ws/src/tennis_robot/urdf/components/base.urdf.xacro (robot description, xacro)
@@ -32,5 +32,9 @@
       <parent link="base_footprint"/>
       <child link="base_link"/>
-      <origin xyz="0 0 0.09" rpy="0 0.053 0"/>
+      <!-- Level chassis (no pitch). base_link is the chassis plate at axle height
+           + wheel drop: z = wheel_radius - wheel_z = 0.09 - (-0.09) = 0.18, so the
+           four wheel contacts land exactly on the ground plane and base_footprint
+           sits on the ground. -->
+      <origin xyz="0 0 0.18" rpy="0 0 0"/>
     </joint>
     <link name="base_link">
@@ -70,11 +74,21 @@
         <material name="mount_gray"/>
       </visual>
-      <visual name="left_axle_bracket_vis">
-        <origin xyz="-0.35 0.32 0" rpy="0 0 0"/>
+      <visual name="rear_left_axle_bracket_vis">
+        <origin xyz="-0.33 0.32 0" rpy="0 0 0"/>
         <geometry><box size="0.065 0.060 0.018"/></geometry>
         <material name="mount_gray"/>
       </visual>
-      <visual name="right_axle_bracket_vis">
-        <origin xyz="-0.35 -0.32 0" rpy="0 0 0"/>
+      <visual name="rear_right_axle_bracket_vis">
+        <origin xyz="-0.33 -0.32 0" rpy="0 0 0"/>
+        <geometry><box size="0.065 0.060 0.018"/></geometry>
+        <material name="mount_gray"/>
+      </visual>
+      <visual name="front_left_axle_bracket_vis">
+        <origin xyz="0.33 0.32 0" rpy="0 0 0"/>
+        <geometry><box size="0.065 0.060 0.018"/></geometry>
+        <material name="mount_gray"/>
+      </visual>
+      <visual name="front_right_axle_bracket_vis">
+        <origin xyz="0.33 -0.32 0" rpy="0 0 0"/>
         <geometry><box size="0.065 0.060 0.018"/></geometry>
         <material name="mount_gray"/>

File: ros2_ws/src/tennis_robot/urdf/components/drivetrain.urdf.xacro (robot description, xacro)
@@ -22,65 +22,18 @@
     </joint>
     <gazebo reference="${side}_wheel_link">
-      <!-- VER=21: brute-force friction test — mu=5.0 isotropic, no fdir1.
-           VER=20 (mu=1.5) improved rotation from 48° to 73° out of 275° (~73% slip).
-           If mu=5.0 with court mu=2.0 still gives ~73% slip, the URDF <gazebo>
-           friction tags are NOT reaching the physics engine (DART ignoring them)
-           and we need the bullet-featherstone engine or direct SDF injection. -->
-      <mu1>5.0</mu1>
-      <mu2>5.0</mu2>
+      <!-- Moderate friction on all four driven wheels. 4WD skid-steer turning
+           relies on lateral slip; the previous mu=5.0 over-resisted rotation,
+           making in-place turns crawl and survey waypoints time out. mu=1.2
+           keeps enough forward grip (court surface adds more) while letting the
+           robot rotate quickly. -->
+      <mu1>1.2</mu1>
+      <mu2>1.2</mu2>
       <slip1>0.0</slip1>
       <slip2>0.0</slip2>
     </gazebo>
   </xacro:macro>
-  <xacro:macro name="caster" params="name x y z radius width:=0.030 trail:=0.0">
-    <link name="${name}_caster_swivel_link">
-      <inertial>
-        <mass value="0.03"/>
-        <inertia ixx="5e-5" ixy="0" ixz="0" iyy="5e-5" iyz="0" izz="5e-5"/>
-      </inertial>
-      <visual name="swivel_stem_vis">
-        <origin xyz="0 0 0.045" rpy="0 0 0"/>
-        <geometry><cylinder radius="0.014" length="0.09"/></geometry>
-        <material name="mount_gray"/>
-      </visual>
-      <visual name="caster_fork_vis">
-        <origin xyz="0 0 -0.025" rpy="0 0 0"/>
-        <geometry><box size="0.075 0.020 0.055"/></geometry>
-        <material name="mount_gray"/>
-      </visual>
-    </link>
-    <joint name="${name}_caster_swivel_joint" type="continuous">
-      <parent link="base_link"/>
-      <child link="${name}_caster_swivel_link"/>
-      <origin xyz="${x} ${y} ${z + radius}" rpy="0 0 0"/>
-      <axis xyz="0 0 1"/>
-      <dynamics damping="0.02" friction="0.001"/>
-    </joint>
-    <link name="${name}_caster_wheel_link">
-      <xacro:cylinder_inertial mass="0.05" radius="${radius}" length="${width}" axis="y"/>
-      <collision name="col">
-        <origin xyz="0 0 0" rpy="1.5708 0 0"/>
-        <geometry><cylinder radius="${radius}" length="${width}"/></geometry>
-      </collision>
-      <visual name="vis">
-        <origin xyz="0 0 0" rpy="1.5708 0 0"/>
-        <geometry><cylinder radius="${radius}" length="${width}"/></geometry>
-        <material name="rubber_black"/>
-      </visual>
-    </link>
-    <joint name="${name}_caster_wheel_joint" type="continuous">
-      <parent link="${name}_caster_swivel_link"/>
-      <child link="${name}_caster_wheel_link"/>
-      <!-- trail: wheel contact sits behind the vertical swivel axis so the
-           caster self-aligns with the direction of travel (no scrub/shimmy). -->
-      <origin xyz="-${trail} 0 -${radius}" rpy="0 0 0"/>
-      <axis xyz="0 1 0"/>
-      <dynamics damping="0.001" friction="0.0"/>
-    </joint>
-    <gazebo reference="${name}_caster_wheel_link">
-      <mu1>0.8</mu1>
-      <mu2>0.05</mu2>
-    </gazebo>
-  </xacro:macro>
+  <!-- Casters removed: the robot is now 4WD skid-steer (four driven wheels via
+       the drive_wheel macro above). The old swivel-caster macro and its scrub
+       resistance are gone. -->
   <xacro:macro name="intake_roller" params="x z radius width mass">
     <link name="lift_wheel_link">

File: ros2_ws/src/tennis_robot/urdf/components/ros2_control.urdf.xacro (robot description, xacro)
@@ -6,7 +6,8 @@
   move from Gazebo to the real robot: controllers, command topics and the whole
   behavior stack above stay identical.
-  Joints exposed:
-    left_wheel_joint / right_wheel_joint -> velocity command (diff drive)
-    lift_wheel_joint                     -> velocity command (intake roller)
+  Joints exposed (4WD skid-steer):
+    rear_left_wheel_joint  / front_left_wheel_joint  -> velocity command (left side)
+    rear_right_wheel_joint / front_right_wheel_joint -> velocity command (right side)
+    lift_wheel_joint                                 -> velocity command (intake roller)
 -->
 <robot xmlns:xacro="http://www.ros.org/wiki/xacro">
@@ -14,5 +15,5 @@
                params="sim_mode:=true controllers_config wheel_max_vel:=20.0 lift_max_vel:=40.0">
     <ros2_control name="TennisRobotSystem" type="system">
-      <!-- ── Hardware backend (the only sim/real difference) ─────────────── -->
+      <!-- Hardware backend (the only sim/real difference) -->
       <xacro:if value="${sim_mode}">
         <hardware>
@@ -24,13 +25,17 @@
           <!-- TODO(real-robot): replace with the motor-driver hardware interface,
                e.g. a custom tennis_robot_hardware/DiffDriveHardware plugin that
-               talks to the wheel controllers over CAN/serial. Same joint names. -->
+               talks to the BTS7960 drivers over serial/PWM. Same joint names.
+               Real wiring: the two motors on each side are wired in PARALLEL to a
+               single BTS7960 driver, with ONE encoder per side. So the front/rear
+               joints on a side share one velocity command and one feedback source
+               (front mirrors rear). Map both side joints to the same side channel. -->
           <plugin>tennis_robot_hardware/TennisRobotSystem</plugin>
-          <param name="left_wheel_name">left_wheel_joint</param>
-          <param name="right_wheel_name">right_wheel_joint</param>
+          <param name="left_wheel_names">rear_left_wheel_joint,front_left_wheel_joint</param>
+          <param name="right_wheel_names">rear_right_wheel_joint,front_right_wheel_joint</param>
           <param name="lift_wheel_name">lift_wheel_joint</param>
         </hardware>
       </xacro:unless>
-      <!-- ── Drive joints ────────────────────────────────────────────────── -->
-      <joint name="left_wheel_joint">
+      <!-- Drive joints (4WD skid-steer: 2 per side) -->
+      <joint name="rear_left_wheel_joint">
         <command_interface name="velocity">
           <param name="min">-${wheel_max_vel}</param>
@@ -40,5 +45,5 @@
         <state_interface name="velocity"/>
       </joint>
-      <joint name="right_wheel_joint">
+      <joint name="front_left_wheel_joint">
         <command_interface name="velocity">
           <param name="min">-${wheel_max_vel}</param>
@@ -48,5 +53,21 @@
         <state_interface name="velocity"/>
       </joint>
-      <!-- ── Intake roller ───────────────────────────────────────────────── -->
+      <joint name="rear_right_wheel_joint">
+        <command_interface name="velocity">
+          <param name="min">-${wheel_max_vel}</param>
+          <param name="max">${wheel_max_vel}</param>
+        </command_interface>
+        <state_interface name="position"/>
+        <state_interface name="velocity"/>
+      </joint>
+      <joint name="front_right_wheel_joint">
+        <command_interface name="velocity">
+          <param name="min">-${wheel_max_vel}</param>
+          <param name="max">${wheel_max_vel}</param>
+        </command_interface>
+        <state_interface name="position"/>
+        <state_interface name="velocity"/>
+      </joint>
+      <!-- Intake roller -->
       <joint name="lift_wheel_joint">
         <command_interface name="velocity">
@@ -57,21 +78,6 @@
         <state_interface name="velocity"/>
       </joint>
-      <!-- ── Passive caster joints: NOT in ros2_control ──────────────────────
-           Previously listed here as state-only so joint_state_broadcaster could
-           publish their positions for RViz TF. However, gz_ros2_control owns any
-           joint it has an interface for, and may zero out state-only joints during
-           initialization or write cycles. Locked caster swivel/wheel joints create
-           ~12 N·m of scrub resistance (mu1=0.8 × caster weight × moment arm) that
-           exceeds the ~7.7 N·m drive torque → 82% rotation slip observed.
-           Fix: remove casters from ros2_control entirely; gz-physics handles them
-           freely via URDF <dynamics damping="0.02" friction="0.001"/> on the swivel.
-           Cost: /joint_states won't include casters → RViz "No transform from
-           front_*_caster_*". Navigation is unaffected (caster TF not used by
-           slam_toolbox or nav2). -->
     </ros2_control>
-    <!-- ── gz_ros2_control system plugin (sim only) ─────────────────────────
-         Hosts the controller_manager inside the Gazebo process and loads the
-         controllers from controllers.yaml. On the real robot the
-         controller_manager is launched as a normal ROS 2 node instead. -->
+    <!-- gz_ros2_control system plugin (sim only) -->
     <xacro:if value="${sim_mode}">
       <gazebo>

File: ros2_ws/src/tennis_robot/urdf/tennis_robot.urdf.xacro (robot description, xacro)
@@ -9,4 +9,5 @@
   <xacro:include filename="components/lidar.urdf.xacro"/>
   <xacro:include filename="components/oak_d.urdf.xacro"/>
+  <xacro:include filename="components/imu.urdf.xacro"/>
   <xacro:include filename="components/ir_beam.urdf.xacro"/>
   <xacro:include filename="components/body_panels.urdf.xacro"/>
@@ -20,29 +21,24 @@
   <xacro:property name="chassis_z" value="0.014"/>
   <xacro:property name="chassis_mass" value="7.2"/>
-  <xacro:property name="wheel_x" value="-0.35"/>
+  <!-- 4WD skid-steer drivetrain. Four identical 180 mm (radius 0.09) driven
+       wheels, two per side, placed symmetrically about the chassis center
+       (±wheel_base_x). All four share the same wheel_z and radius so their
+       ground contacts are coplanar and the (now level, un-pitched) robot sits
+       flat. Casters removed. -->
+  <xacro:property name="wheel_base_x" value="0.33"/>  <!-- rear at -x, front at +x; wheelbase = 0.66 m -->
   <xacro:property name="wheel_y" value="0.35"/>
   <xacro:property name="wheel_z" value="-0.09"/>
-  <xacro:property name="wheel_radius" value="0.09"/>
+  <xacro:property name="wheel_radius" value="0.09"/>  <!-- 180 mm diameter -->
   <xacro:property name="wheel_width" value="0.08"/>
   <xacro:property name="wheel_mass" value="0.25"/>
   <xacro:property name="wheel_separation" value="${2.0 * wheel_y}"/>
-  <!-- Front swivel casters. Sized for a real clay court (rolling wheel, not a
-       skid/ball). caster_z chosen so the wheel contact is coplanar with the
-       drive wheels at the 3deg design pitch: contact_z = caster_z - caster_radius.
-       Set caster_radius/width/trail to the actual caster hardware you fit. -->
-  <xacro:property name="caster_x" value="0.31"/>
-  <xacro:property name="caster_y" value="0.35"/>
-  <xacro:property name="caster_radius" value="0.0625"/>   <!-- 125 mm wheel dia -->
-  <xacro:property name="caster_width" value="0.035"/>
-  <xacro:property name="caster_trail" value="0.025"/>     <!-- self-aligning offset -->
-  <xacro:property name="caster_z" value="-0.0825"/>       <!-- contact = -0.145 m (coplanar with drive wheels under 3deg pitch) -->
   <xacro:property name="intake_x" value="0.62"/>
   <xacro:property name="intake_z" value="0.095"/>
   <xacro:property name="intake_radius" value="0.03"/>
   <xacro:property name="intake_width" value="0.24"/>
-  <xacro:property name="lidar_xyz" value="-0.08 0 0.713"/>
-  <xacro:property name="lidar_rpy" value="0 -0.053 0"/>  <!-- counter the 3deg chassis pitch so the 360 scan plane stays horizontal -->
+  <xacro:property name="lidar_xyz" value="-0.08 0 0.498"/>  <!-- z chosen so the scan plane sits at world ~0.713 m (the net_lidar_strand height, well below the 0.914 m net-center top) now that base_link is level at 0.18 -->
+  <xacro:property name="lidar_rpy" value="0 0 0"/>  <!-- chassis is now level (no pitch): scan plane is already horizontal -->
   <xacro:property name="camera_xyz" value="0.535 0 0.443"/>
-  <xacro:property name="camera_rpy" value="0 0.22 0"/>
+  <xacro:property name="camera_rpy" value="0 0.273 0"/>  <!-- forward-down tilt ~15.6deg; preserves the old world aim (0.22 cam + 0.053 chassis pitch) now that the chassis is level -->
   <xacro:property name="sensor_update_rate" value="31.25"/>
   <xacro:property name="ir_x" value="0.54"/>
@@ -60,7 +56,7 @@
       chassis_mass="${chassis_mass}"/>
   <xacro:drive_wheel
-      side="left"
+      side="rear_left"
       y="${wheel_y}"
-      wheel_x="${wheel_x}"
+      wheel_x="-${wheel_base_x}"
       wheel_z="${wheel_z}"
       radius="${wheel_radius}"
@@ -68,7 +64,23 @@
       mass="${wheel_mass}"/>
   <xacro:drive_wheel
-      side="right"
+      side="rear_right"
       y="-${wheel_y}"
-      wheel_x="${wheel_x}"
+      wheel_x="-${wheel_base_x}"
+      wheel_z="${wheel_z}"
+      radius="${wheel_radius}"
+      width="${wheel_width}"
+      mass="${wheel_mass}"/>
+  <xacro:drive_wheel
+      side="front_left"
+      y="${wheel_y}"
+      wheel_x="${wheel_base_x}"
+      wheel_z="${wheel_z}"
+      radius="${wheel_radius}"
+      width="${wheel_width}"
+      mass="${wheel_mass}"/>
+  <xacro:drive_wheel
+      side="front_right"
+      y="-${wheel_y}"
+      wheel_x="${wheel_base_x}"
       wheel_z="${wheel_z}"
       radius="${wheel_radius}"
@@ -83,6 +95,4 @@
 <xacro:intake_funnel parent="base_link" chassis_z="${chassis_z}"/>
   <xacro:ball_basket parent="base_link"/>
-  <xacro:caster name="front_left" x="${caster_x}" y="-${caster_y}" z="${caster_z}" radius="${caster_radius}" width="${caster_width}" trail="${caster_trail}"/>
-  <xacro:caster name="front_right" x="${caster_x}" y="${caster_y}" z="${caster_z}" radius="${caster_radius}" width="${caster_width}" trail="${caster_trail}"/>
   <xacro:rplidar_c1_mount
       parent="base_link"
@@ -97,4 +107,13 @@
       rpy="${camera_rpy}"
       update_rate="${sensor_update_rate}"/>
+  <!-- MPU6050 IMU near the chassis centre, axes aligned with base_link. Mainly
+       used for yaw rate, which wheel odometry mis-estimates in skid-steer. -->
+  <xacro:mpu6050_imu
+      parent="base_link"
+      link_name="imu_link"
+      xyz="-0.05 0 0.012"
+      rpy="0 0 0"
+      update_rate="100"
+      topic="/gz/imu"/>
   <xacro:ir_beam_sensor
       parent="base_link"

Commit message: Document motion hardware and 170mm wheel geometry

File: ros2_ws/src/tennis_robot/urdf/components/base.urdf.xacro (robot description, xacro)
@@ -33,8 +33,8 @@
       <child link="base_link"/>
       <!-- Level chassis (no pitch). base_link is the chassis plate at axle height
-           + wheel drop: z = wheel_radius - wheel_z = 0.09 - (-0.09) = 0.18, so the
+           + wheel drop: z = wheel_radius - wheel_z = 0.085 - (-0.09) = 0.175, so the
            four wheel contacts land exactly on the ground plane and base_footprint
            sits on the ground. -->
-      <origin xyz="0 0 0.18" rpy="0 0 0"/>
+      <origin xyz="0 0 0.175" rpy="0 0 0"/>
     </joint>
     <link name="base_link">

File: ros2_ws/src/tennis_robot/urdf/tennis_robot.urdf.xacro (robot description, xacro)
@@ -21,13 +21,13 @@
   <xacro:property name="chassis_z" value="0.014"/>
   <xacro:property name="chassis_mass" value="7.2"/>
-  <!-- 4WD skid-steer drivetrain. Four identical 180 mm (radius 0.09) driven
-       wheels, two per side, placed symmetrically about the chassis center
-       (±wheel_base_x). All four share the same wheel_z and radius so their
-       ground contacts are coplanar and the (now level, un-pitched) robot sits
-       flat. Casters removed. -->
+  <!-- 4WD skid-steer drivetrain. Four identical 170 mm (radius 0.085) driven
+       wheels (HPI Dirt Buster Block, 170x80 mm, Baja 5B), two per side, placed
+       symmetrically about the chassis center (±wheel_base_x). All four share the
+       same wheel_z and radius so their ground contacts are coplanar and the
+       (now level, un-pitched) robot sits flat. Casters removed. -->
   <xacro:property name="wheel_base_x" value="0.33"/>  <!-- rear at -x, front at +x; wheelbase = 0.66 m -->
   <xacro:property name="wheel_y" value="0.35"/>
   <xacro:property name="wheel_z" value="-0.09"/>
-  <xacro:property name="wheel_radius" value="0.09"/>  <!-- 180 mm diameter -->
+  <xacro:property name="wheel_radius" value="0.085"/>  <!-- 170 mm diameter (HPI Dirt Buster Block) -->
   <xacro:property name="wheel_width" value="0.08"/>
   <xacro:property name="wheel_mass" value="0.25"/>
