Commit message: Add physical collector control path and correct intake geometry

File: ros2_ws/src/tennis_robot/urdf/components/base.urdf.xacro (robot description, xacro)
@@ -27,14 +27,12 @@
     </inertial>
   </xacro:macro>
-  <xacro:macro name="tennis_robot_base" params="chassis_x chassis_y chassis_z chassis_mass">
+  <xacro:macro name="tennis_robot_base" params="chassis_x chassis_y chassis_z base_link_height chassis_mass">
     <link name="base_footprint"/>
     <joint name="base_footprint_joint" type="fixed">
       <parent link="base_footprint"/>
       <child link="base_link"/>
-      <!-- Level chassis (no pitch). base_link is the chassis plate at axle height
-           + wheel drop: z = wheel_radius - wheel_z = 0.085 - (-0.09) = 0.175, so the
-           four wheel contacts land exactly on the ground plane and base_footprint
-           sits on the ground. -->
-      <origin xyz="0 0 0.175" rpy="0 0 0"/>
+      <!-- base_footprint is the ground plane. base_link is the centre of the
+           chassis plate, deliberately below the motor/axle centreline. -->
+      <origin xyz="0 0 ${base_link_height}" rpy="0 0 0"/>
     </joint>
     <link name="base_link">
@@ -75,20 +73,20 @@
       </visual>
       <visual name="rear_left_axle_bracket_vis">
-        <origin xyz="-0.33 0.32 0" rpy="0 0 0"/>
+        <origin xyz="-0.33 0.24 ${0.5 * chassis_z + 0.009}" rpy="0 0 0"/>
         <geometry><box size="0.065 0.060 0.018"/></geometry>
         <material name="mount_gray"/>
       </visual>
       <visual name="rear_right_axle_bracket_vis">
-        <origin xyz="-0.33 -0.32 0" rpy="0 0 0"/>
+        <origin xyz="-0.33 -0.24 ${0.5 * chassis_z + 0.009}" rpy="0 0 0"/>
         <geometry><box size="0.065 0.060 0.018"/></geometry>
         <material name="mount_gray"/>
       </visual>
       <visual name="front_left_axle_bracket_vis">
-        <origin xyz="0.33 0.32 0" rpy="0 0 0"/>
+        <origin xyz="0.33 0.24 ${0.5 * chassis_z + 0.009}" rpy="0 0 0"/>
         <geometry><box size="0.065 0.060 0.018"/></geometry>
         <material name="mount_gray"/>
       </visual>
       <visual name="front_right_axle_bracket_vis">
-        <origin xyz="0.33 -0.32 0" rpy="0 0 0"/>
+        <origin xyz="0.33 -0.24 ${0.5 * chassis_z + 0.009}" rpy="0 0 0"/>
         <geometry><box size="0.065 0.060 0.018"/></geometry>
         <material name="mount_gray"/>

File: ros2_ws/src/tennis_robot/urdf/components/drivetrain.urdf.xacro (robot description, xacro)
@@ -1,4 +1,23 @@
 <?xml version="1.0" encoding="UTF-8"?>
 <robot xmlns:xacro="http://www.ros.org/wiki/xacro">
+  <xacro:macro name="drive_motor" params="side y motor_x shaft_z radius length mass">
+    <link name="${side}_motor_link">
+      <xacro:cylinder_inertial mass="${mass}" radius="${radius}" length="${length}" axis="y"/>
+      <collision name="motor_col">
+        <origin xyz="0 0 0" rpy="1.5708 0 0"/>
+        <geometry><cylinder radius="${radius}" length="${length}"/></geometry>
+      </collision>
+      <visual name="motor_vis">
+        <origin xyz="0 0 0" rpy="1.5708 0 0"/>
+        <geometry><cylinder radius="${radius}" length="${length}"/></geometry>
+        <material name="mount_gray"/>
+      </visual>
+    </link>
+    <joint name="${side}_motor_mount_joint" type="fixed">
+      <parent link="base_link"/>
+      <child link="${side}_motor_link"/>
+      <origin xyz="${motor_x} ${y} ${shaft_z}" rpy="0 0 0"/>
+    </joint>
+  </xacro:macro>
   <xacro:macro name="drive_wheel" params="side y wheel_x wheel_z radius width mass">
     <link name="${side}_wheel_link">
@@ -36,16 +55,42 @@
        the drive_wheel macro above). The old swivel-caster macro and its scrub
        resistance are gone. -->
+  <!-- One paddle belonging to the single intake-roller link. `angle` is in the
+       link's x-z plane; rotating the link rotates core and all paddles together. -->
+  <xacro:macro name="intake_flap" params="name angle radius width">
+    <collision name="${name}_col">
+      <origin
+          xyz="${radius * 0.72 * cos(angle)} 0 ${radius * 0.72 * sin(angle)}"
+          rpy="0 ${-angle} 0"/>
+      <geometry><box size="${radius * 0.56} ${width} 0.004"/></geometry>
+    </collision>
+    <visual name="${name}_vis">
+      <origin
+          xyz="${radius * 0.72 * cos(angle)} 0 ${radius * 0.72 * sin(angle)}"
+          rpy="0 ${-angle} 0"/>
+      <geometry><box size="${radius * 0.56} ${width} 0.004"/></geometry>
+      <material name="rubber_black"/>
+    </visual>
+  </xacro:macro>
   <xacro:macro name="intake_roller" params="x z radius width mass">
     <link name="lift_wheel_link">
       <xacro:cylinder_inertial mass="${mass}" radius="${radius}" length="${width}" axis="y"/>
-      <collision name="col">
+      <!-- Small rigid hub; the paddles define the 100 mm swept envelope. -->
+      <collision name="core_col">
         <origin xyz="0 0 0" rpy="1.5708 0 0"/>
-        <geometry><cylinder radius="${radius}" length="${width}"/></geometry>
+        <geometry><cylinder radius="${radius * 0.44}" length="${width}"/></geometry>
       </collision>
-      <visual name="vis">
+      <visual name="core_vis">
         <origin xyz="0 0 0" rpy="1.5708 0 0"/>
-        <geometry><cylinder radius="${radius}" length="${width}"/></geometry>
+        <geometry><cylinder radius="${radius * 0.44}" length="${width}"/></geometry>
         <material name="rubber_black"/>
       </visual>
+      <xacro:intake_flap name="flap_0" angle="0.0" radius="${radius}" width="${width}"/>
+      <xacro:intake_flap name="flap_1" angle="${pi / 4.0}" radius="${radius}" width="${width}"/>
+      <xacro:intake_flap name="flap_2" angle="${pi / 2.0}" radius="${radius}" width="${width}"/>
+      <xacro:intake_flap name="flap_3" angle="${3.0 * pi / 4.0}" radius="${radius}" width="${width}"/>
+      <xacro:intake_flap name="flap_4" angle="${pi}" radius="${radius}" width="${width}"/>
+      <xacro:intake_flap name="flap_5" angle="${5.0 * pi / 4.0}" radius="${radius}" width="${width}"/>
+      <xacro:intake_flap name="flap_6" angle="${3.0 * pi / 2.0}" radius="${radius}" width="${width}"/>
+      <xacro:intake_flap name="flap_7" angle="${7.0 * pi / 4.0}" radius="${radius}" width="${width}"/>
     </link>
     <joint name="lift_wheel_joint" type="continuous">

File: ros2_ws/src/tennis_robot/urdf/components/funnel.urdf.xacro (robot description, xacro)
@@ -1,5 +1,5 @@
 <?xml version="1.0" encoding="UTF-8"?>
 <robot xmlns:xacro="http://www.ros.org/wiki/xacro">
-  <xacro:macro name="intake_funnel" params="parent chassis_z">
+  <xacro:macro name="intake_funnel" params="parent chassis_z pitch">
     <joint name="funnel_joint" type="fixed">
       <parent link="${parent}"/>
@@ -13,20 +13,22 @@
       </inertial>
       <visual name="funnel_left_cheek_vis">
-        <origin xyz="0.54 0.14 0.08" rpy="0 0 0.25"/>
-        <geometry><box size="0.18 0.01 0.14"/></geometry>
+        <origin xyz="0.54 0.14 0.052" rpy="0 ${pitch} 0.25"/>
+        <geometry><box size="0.24 0.01 0.10"/></geometry>
         <material name="intake_orange"/>
       </visual>
       <visual name="funnel_right_cheek_vis">
-        <origin xyz="0.54 -0.14 0.08" rpy="0 0 -0.25"/>
-        <geometry><box size="0.18 0.01 0.14"/></geometry>
+        <origin xyz="0.54 -0.14 0.052" rpy="0 ${pitch} -0.25"/>
+        <geometry><box size="0.24 0.01 0.10"/></geometry>
         <material name="intake_orange"/>
       </visual>
       <collision name="roller_exit_floor_col">
-        <origin xyz="0.54 0 0.01" rpy="0 0 0"/>
-        <geometry><box size="0.16 0.24 0.005"/></geometry>
+        <!-- Closed 2 mm wedge: its front underside is exactly at the ground
+             plane and its 0.32 rad top surface rises toward the roller. -->
+        <origin xyz="0.54 0 0" rpy="0 0 0"/>
+        <geometry><mesh filename="package://tennis_robot/meshes/scooper_wedge.stl"/></geometry>
       </collision>
       <visual name="roller_exit_floor_vis">
-        <origin xyz="0.54 0 0.01" rpy="0 0 0"/>
-        <geometry><box size="0.16 0.24 0.005"/></geometry>
+        <origin xyz="0.54 0 0" rpy="0 0 0"/>
+        <geometry><mesh filename="package://tennis_robot/meshes/scooper_wedge.stl"/></geometry>
         <material name="intake_orange"/>
       </visual>

File: ros2_ws/src/tennis_robot/urdf/components/lidar.urdf.xacro (robot description, xacro)
@@ -8,6 +8,9 @@
       </inertial>
       <visual name="mast_vis">
-        <origin xyz="0 0 -0.30" rpy="0 0 0"/>
-        <geometry><box size="0.025 0.025 0.57"/></geometry>
+        <!-- Runs from just under the LiDAR head down to the chassis top.
+             With lidar_xyz.z=0.498 and a 14 mm plate, the lower end is
+             base_link z=+0.007; it must never protrude below the chassis. -->
+        <origin xyz="0 0 -0.253" rpy="0 0 0"/>
+        <geometry><box size="0.025 0.025 0.476"/></geometry>
         <material name="anthracite"/>
       </visual>

File: ros2_ws/src/tennis_robot/urdf/tennis_robot.urdf.xacro (robot description, xacro)
@@ -17,8 +17,11 @@
   <xacro:arg name="sim_mode" default="true"/>
   <xacro:arg name="controllers_config" default="config/controllers.yaml"/>
-<xacro:property name="chassis_x" value="0.92"/>
+  <xacro:property name="chassis_x" value="0.92"/>
   <xacro:property name="chassis_y" value="0.58"/>
   <xacro:property name="chassis_z" value="0.014"/>
   <xacro:property name="chassis_mass" value="7.2"/>
+  <!-- base_link is the chassis plate centre. The plate top is 52 mm above
+       ground, below the 85 mm motor-shaft/wheel-axle centreline. -->
+  <xacro:property name="base_link_height" value="0.045"/>
   <!-- 4WD skid-steer drivetrain. Four identical 170 mm (radius 0.085) driven
        wheels (HPI Dirt Buster Block, 170x80 mm, Baja 5B), two per side, placed
@@ -28,15 +31,25 @@
   <xacro:property name="wheel_base_x" value="0.33"/>  <!-- rear at -x, front at +x; wheelbase = 0.66 m -->
   <xacro:property name="wheel_y" value="0.35"/>
-  <xacro:property name="wheel_z" value="-0.09"/>
   <xacro:property name="wheel_radius" value="0.085"/>  <!-- 170 mm diameter (HPI Dirt Buster Block) -->
+  <xacro:property name="wheel_z" value="${wheel_radius - base_link_height}"/>
   <xacro:property name="wheel_width" value="0.08"/>
   <xacro:property name="wheel_mass" value="0.25"/>
   <xacro:property name="wheel_separation" value="${2.0 * wheel_y}"/>
-  <xacro:property name="intake_x" value="0.62"/>
-  <xacro:property name="intake_z" value="0.095"/>
-  <xacro:property name="intake_radius" value="0.03"/>
+  <xacro:property name="motor_y" value="${chassis_y / 2.0 - 0.05}"/>
+  <xacro:property name="motor_radius" value="0.03"/>
+  <xacro:property name="motor_length" value="0.10"/>
+  <!-- The 0.66 m scooper lip must meet the ball first. The single roller sits
+       60 mm behind it, over the rising ramp, so the scoop supports the ball
+       while the flaps drive it upward and inward. -->
+  <xacro:property name="intake_x" value="0.60"/>
+  <!-- Single-shaft flap roller: 100 mm swept diameter, with its tip envelope
+       still 64 mm above ground. The rigid core is smaller; eight paddles on
+       the same rotating link provide the compliant-roller approximation. -->
+  <xacro:property name="intake_z" value="0.069"/>
+  <xacro:property name="intake_radius" value="0.05"/>
   <xacro:property name="intake_width" value="0.24"/>
-  <xacro:property name="lidar_xyz" value="-0.08 0 0.498"/>  <!-- z chosen so the scan plane sits at world ~0.713 m (the net_lidar_strand height, well below the 0.914 m net-center top) now that base_link is level at 0.18 -->
-  <xacro:property name="lidar_rpy" value="0 0 0"/>  <!-- chassis is now level (no pitch): scan plane is already horizontal -->
+  <xacro:property name="scooper_pitch" value="0.1745"/>  <!-- 10 degrees -->
+  <xacro:property name="lidar_xyz" value="-0.08 0 0.498"/>
+  <xacro:property name="lidar_rpy" value="0 0 0"/>  <!-- level chassis: horizontal scan plane -->
   <xacro:property name="camera_xyz" value="0.535 0 0.443"/>
   <xacro:property name="camera_rpy" value="0 0.273 0"/>  <!-- forward-down tilt ~15.6deg; preserves the old world aim (0.22 cam + 0.053 chassis pitch) now that the chassis is level -->
@@ -54,5 +67,16 @@
       chassis_y="${chassis_y}"
       chassis_z="${chassis_z}"
+      base_link_height="${base_link_height}"
       chassis_mass="${chassis_mass}"/>
+  <!-- Motors are fixed to the chassis top. Each shaft shares its x/z centre
+       with the corresponding wheel joint; only y differs along the shaft. -->
+  <xacro:drive_motor side="rear_left" y="${motor_y}" motor_x="-${wheel_base_x}"
+      shaft_z="${wheel_z}" radius="${motor_radius}" length="${motor_length}" mass="0.65"/>
+  <xacro:drive_motor side="rear_right" y="-${motor_y}" motor_x="-${wheel_base_x}"
+      shaft_z="${wheel_z}" radius="${motor_radius}" length="${motor_length}" mass="0.65"/>
+  <xacro:drive_motor side="front_left" y="${motor_y}" motor_x="${wheel_base_x}"
+      shaft_z="${wheel_z}" radius="${motor_radius}" length="${motor_length}" mass="0.65"/>
+  <xacro:drive_motor side="front_right" y="-${motor_y}" motor_x="${wheel_base_x}"
+      shaft_z="${wheel_z}" radius="${motor_radius}" length="${motor_length}" mass="0.65"/>
   <xacro:drive_wheel
       side="rear_left"
@@ -93,5 +117,5 @@
       width="${intake_width}"
       mass="0.20"/>
-<xacro:intake_funnel parent="base_link" chassis_z="${chassis_z}"/>
+  <xacro:intake_funnel parent="base_link" chassis_z="${chassis_z}" pitch="${scooper_pitch}"/>
   <xacro:ball_basket parent="base_link"/>
   <xacro:rplidar_c1_mount
@@ -151,4 +175,4 @@
       sim_mode="$(arg sim_mode)"
       controllers_config="$(arg controllers_config)"/>
-<xacro:robot_body_panels parent="base_link" chassis_z="${chassis_z}"/>
+  <xacro:robot_body_panels parent="base_link" chassis_z="${chassis_z}"/>
 </robot>
