Commit message: Basket v2: sunken removable mesh bin, rear battery bay, external lidar mast
Replace the scoop-era basket with the bin designed in
docs/basket-bin-redesign-spec-el.md (user decisions: ~50 balls, removable
wire-mesh bin, sunken floor for retention):

- Bin interior x 0.02-0.42, +-0.14, floor at 0.030 ground through a REAL
  chassis-plate opening (plate is now two side strips + a rear block): a
  ball is retained by 25 mm of depth below the 0.055 jump lip instead of
  the old 3 mm step, and the bin bottom keeps 25 mm of ground clearance.
- Battery pack (user's 19.8x16.6x17 cm, 6.26 kg) modeled with real mass on
  the rear deck as a counterweight to the front intake overhang.
- Lidar mast moves out of the interior to the rear top frame
  (-0.08 -> -0.42; TF-only change) - it used to stand inside the old
  basket footprint.
- Basket IR pair moves to the entry plane (x 0.28 -> 0.40): with the
  sunken floor a rolling ball passes under a 0.085-high beam, so only the
  lip-crossing entry event should cut it (mesh walls let the chassis-
  mounted sensors shine through - the bin lifts out with no connectors).
- Controller basket zone follows the bin (x 0.02..0.42, half width 0.14).
- Bench harness default wheel tilt 0 -> 35 (the one default missed in the
  earlier flip; it silently disabled the vertical kick component).

Validation (debug-log #45): Phase 4 envelope PASS 5/5 with balls resting
ON the sunken floor (z=0.063), and the project's first retention test
PASS 15/15 - fifteen balls aboard through sprints, hard stops, +-2 rad/s
spins and hard reverse, zero escapes.

Co-Authored-By: Claude Fable 5 <noreply@anthropic.com>

File: ros2_ws/src/tennis_robot/urdf/components/base.urdf.xacro (robot description, xacro)
@@ -38,32 +38,34 @@
     <link name="base_link">
       <xacro:box_inertial mass="${chassis_mass}" x="${chassis_x}" y="${chassis_y}" z="${chassis_z}"/>
-      <!-- Front-centre cutout (0.20 wide x 0.04 deep): leaves clearance for
-           the launcher scoop/ramp path into the basket. Plate = two
-           full-length side strips + one centre strip ending at x=0.42. -->
+      <!-- Bin v2 opening (docs/basket-bin-redesign-spec-el.md §3): the plate
+           is REALLY open at x 0.01..0.46, y ±0.15 so the sunken bin floor
+           (0.030 ground) is the surface balls actually rest on — a solid
+           plate here would bury the bin's 25 mm retention depth. Plate =
+           two full-length side strips (|y| 0.15..0.29) + rear block. -->
       <collision name="chassis_left_col">
-        <origin xyz="0 ${0.10 + (chassis_y / 2.0 - 0.10) / 2.0} 0" rpy="0 0 0"/>
-        <geometry><box size="${chassis_x} ${chassis_y / 2.0 - 0.10} ${chassis_z}"/></geometry>
+        <origin xyz="0 0.22 0" rpy="0 0 0"/>
+        <geometry><box size="${chassis_x} 0.14 ${chassis_z}"/></geometry>
       </collision>
       <collision name="chassis_right_col">
-        <origin xyz="0 ${-(0.10 + (chassis_y / 2.0 - 0.10) / 2.0)} 0" rpy="0 0 0"/>
-        <geometry><box size="${chassis_x} ${chassis_y / 2.0 - 0.10} ${chassis_z}"/></geometry>
+        <origin xyz="0 -0.22 0" rpy="0 0 0"/>
+        <geometry><box size="${chassis_x} 0.14 ${chassis_z}"/></geometry>
       </collision>
-      <collision name="chassis_centre_col">
-        <origin xyz="-0.02 0 0" rpy="0 0 0"/>
-        <geometry><box size="${chassis_x - 0.04} 0.20 ${chassis_z}"/></geometry>
+      <collision name="chassis_rear_col">
+        <origin xyz="-0.225 0 0" rpy="0 0 0"/>
+        <geometry><box size="0.47 0.30 ${chassis_z}"/></geometry>
       </collision>
       <visual name="chassis_left_vis">
-        <origin xyz="0 ${0.10 + (chassis_y / 2.0 - 0.10) / 2.0} 0" rpy="0 0 0"/>
-        <geometry><box size="${chassis_x} ${chassis_y / 2.0 - 0.10} ${chassis_z}"/></geometry>
+        <origin xyz="0 0.22 0" rpy="0 0 0"/>
+        <geometry><box size="${chassis_x} 0.14 ${chassis_z}"/></geometry>
         <material name="plywood"/>
       </visual>
       <visual name="chassis_right_vis">
-        <origin xyz="0 ${-(0.10 + (chassis_y / 2.0 - 0.10) / 2.0)} 0" rpy="0 0 0"/>
-        <geometry><box size="${chassis_x} ${chassis_y / 2.0 - 0.10} ${chassis_z}"/></geometry>
+        <origin xyz="0 -0.22 0" rpy="0 0 0"/>
+        <geometry><box size="${chassis_x} 0.14 ${chassis_z}"/></geometry>
         <material name="plywood"/>
       </visual>
-      <visual name="chassis_centre_vis">
-        <origin xyz="-0.02 0 0" rpy="0 0 0"/>
-        <geometry><box size="${chassis_x - 0.04} 0.20 ${chassis_z}"/></geometry>
+      <visual name="chassis_rear_vis">
+        <origin xyz="-0.225 0 0" rpy="0 0 0"/>
+        <geometry><box size="0.47 0.30 ${chassis_z}"/></geometry>
         <material name="plywood"/>
       </visual>
@@ -114,6 +116,6 @@
       </visual>
       <visual name="elec_vis">
-        <origin xyz="-0.13 0 0.067" rpy="0 0 0"/>
-        <geometry><box size="0.34 0.26 0.12"/></geometry>
+        <origin xyz="-0.36 0 0.067" rpy="0 0 0"/>
+        <geometry><box size="0.18 0.26 0.12"/></geometry>
         <material name="anthracite"/>
       </visual>

File: ros2_ws/src/tennis_robot/urdf/components/basket.urdf.xacro (robot description, xacro)
@@ -1,17 +1,22 @@
 <?xml version="1.0" encoding="UTF-8"?>
 <robot xmlns:xacro="http://www.ros.org/wiki/xacro">
-  <!-- Ball collection basket (floor + three walls), fixed to parent link.
-       floor_front_x: forward edge of the floor (base_link x). Must stay clear
-         of the intake wheel span (nip_x - wheel radius) or it overhangs the
-         wheel-to-hopper handoff and caps the ball's climb (debug-log #41).
-       floor_top_z_ground: floor top height in the GROUND frame. The scoop-era
-         launch design used 0.128; the dual-wheel transport concept wants a low
-         hopper entry just above the chassis plate (~0.058). -->
-  <xacro:macro name="ball_basket" params="parent floor_front_x floor_top_z_ground">
-    <!-- basket_link shares base_link's origin (45 mm above ground). -->
+  <!-- Bin v2 (docs/basket-bin-redesign-spec-el.md): sunken removable
+       wire-mesh bin. The floor drops through a chassis-plate opening so the
+       ball is retained by real depth below the jump lip (25 mm) instead of
+       the old 3 mm step. Collisions are solid boxes: a 66 mm ball cannot
+       pass the <=40 mm mesh openings, so mesh vs solid is visual only.
+       All *_ground params are in the GROUND frame; basket_link shares
+       base_link's origin (base_link_height above ground). -->
+  <xacro:macro name="ball_basket"
+      params="parent floor_front_x floor_top_z_ground rear_x half_width wall_top_z_ground">
     <xacro:property name="floor_top" value="${floor_top_z_ground - base_link_height}"/>
-    <xacro:property name="floor_thickness" value="0.020"/>
-    <xacro:property name="floor_rear_x" value="-0.12"/>
-    <xacro:property name="wall_top" value="0.353"/>
+    <xacro:property name="wall_top" value="${wall_top_z_ground - base_link_height}"/>
+    <!-- Thin skinned bin: 5 mm floor (exterior bottom = floor_top - 0.005,
+         the robot's lowest point), 10 mm wall frames. -->
+    <xacro:property name="floor_thickness" value="0.005"/>
+    <xacro:property name="wall_thickness" value="0.010"/>
+    <xacro:property name="bin_length" value="${floor_front_x - rear_x}"/>
+    <xacro:property name="wall_height" value="${wall_top - floor_top}"/>
+    <xacro:property name="wall_centre_z" value="${(wall_top + floor_top) / 2.0}"/>
     <joint name="basket_joint" type="fixed">
       <parent link="${parent}"/>
@@ -25,45 +30,46 @@
       </inertial>
       <collision name="basket_floor_col">
-        <origin xyz="${(floor_front_x + floor_rear_x) / 2.0} 0 ${floor_top - floor_thickness / 2.0}" rpy="0 0 0"/>
-        <geometry><box size="${floor_front_x - floor_rear_x} 0.34 ${floor_thickness}"/></geometry>
+        <origin xyz="${(floor_front_x + rear_x) / 2.0} 0 ${floor_top - floor_thickness / 2.0}" rpy="0 0 0"/>
+        <geometry><box size="${bin_length} ${2.0 * half_width} ${floor_thickness}"/></geometry>
       </collision>
       <visual name="basket_floor_vis">
-        <origin xyz="${(floor_front_x + floor_rear_x) / 2.0} 0 ${floor_top - floor_thickness / 2.0}" rpy="0 0 0"/>
-        <geometry><box size="${floor_front_x - floor_rear_x} 0.34 ${floor_thickness}"/></geometry>
+        <origin xyz="${(floor_front_x + rear_x) / 2.0} 0 ${floor_top - floor_thickness / 2.0}" rpy="0 0 0"/>
+        <geometry><box size="${bin_length} ${2.0 * half_width} ${floor_thickness}"/></geometry>
         <material name="basket_gray"/>
       </visual>
-      <!-- Walls run from the floor top up to a fixed rim so lowering the
-           floor cannot open a gap balls could escape through. -->
+      <!-- Side walls run the full bin length from floor to rim. -->
       <collision name="basket_left_wall_col">
-        <origin xyz="0.15 0.17 ${(wall_top + floor_top - floor_thickness) / 2.0}" rpy="0 0 0"/>
-        <geometry><box size="0.54 0.020 ${wall_top - floor_top + floor_thickness}"/></geometry>
+        <origin xyz="${(floor_front_x + rear_x) / 2.0} ${half_width + wall_thickness / 2.0} ${wall_centre_z}" rpy="0 0 0"/>
+        <geometry><box size="${bin_length} ${wall_thickness} ${wall_height}"/></geometry>
       </collision>
       <visual name="basket_left_wall_vis">
-        <origin xyz="0.15 0.17 ${(wall_top + floor_top - floor_thickness) / 2.0}" rpy="0 0 0"/>
-        <geometry><box size="0.54 0.020 ${wall_top - floor_top + floor_thickness}"/></geometry>
+        <origin xyz="${(floor_front_x + rear_x) / 2.0} ${half_width + wall_thickness / 2.0} ${wall_centre_z}" rpy="0 0 0"/>
+        <geometry><box size="${bin_length} ${wall_thickness} ${wall_height}"/></geometry>
         <material name="basket_gray"/>
       </visual>
       <collision name="basket_right_wall_col">
-        <origin xyz="0.15 -0.17 ${(wall_top + floor_top - floor_thickness) / 2.0}" rpy="0 0 0"/>
-        <geometry><box size="0.54 0.020 ${wall_top - floor_top + floor_thickness}"/></geometry>
+        <origin xyz="${(floor_front_x + rear_x) / 2.0} ${-(half_width + wall_thickness / 2.0)} ${wall_centre_z}" rpy="0 0 0"/>
+        <geometry><box size="${bin_length} ${wall_thickness} ${wall_height}"/></geometry>
       </collision>
       <visual name="basket_right_wall_vis">
-        <origin xyz="0.15 -0.17 ${(wall_top + floor_top - floor_thickness) / 2.0}" rpy="0 0 0"/>
-        <geometry><box size="0.54 0.020 ${wall_top - floor_top + floor_thickness}"/></geometry>
+        <origin xyz="${(floor_front_x + rear_x) / 2.0} ${-(half_width + wall_thickness / 2.0)} ${wall_centre_z}" rpy="0 0 0"/>
+        <geometry><box size="${bin_length} ${wall_thickness} ${wall_height}"/></geometry>
         <material name="basket_gray"/>
       </visual>
       <collision name="basket_rear_wall_col">
-        <origin xyz="-0.12 0 ${(wall_top + floor_top - floor_thickness) / 2.0}" rpy="0 0 0"/>
-        <geometry><box size="0.020 0.34 ${wall_top - floor_top + floor_thickness}"/></geometry>
+        <origin xyz="${rear_x - wall_thickness / 2.0} 0 ${wall_centre_z}" rpy="0 0 0"/>
+        <geometry><box size="${wall_thickness} ${2.0 * (half_width + wall_thickness)} ${wall_height}"/></geometry>
       </collision>
       <visual name="basket_rear_wall_vis">
-        <origin xyz="-0.12 0 ${(wall_top + floor_top - floor_thickness) / 2.0}" rpy="0 0 0"/>
-        <geometry><box size="0.020 0.34 ${wall_top - floor_top + floor_thickness}"/></geometry>
+        <origin xyz="${rear_x - wall_thickness / 2.0} 0 ${wall_centre_z}" rpy="0 0 0"/>
+        <geometry><box size="${wall_thickness} ${2.0 * (half_width + wall_thickness)} ${wall_height}"/></geometry>
         <material name="basket_gray"/>
       </visual>
-      <!-- Matches basket_ir_z in tennis_robot.urdf.xacro: beam at rolling
-           ball equator height in the low hopper (0.085 ground). -->
+      <!-- No front wall: the jump sheet's back face closes the front; the
+           entry lip at (0.425, 0.055) is the only way in or out. -->
+      <!-- IR beam pair line (sensors mount on the chassis and shine through
+           the mesh — see spec §2). Height = rolling-ball equator. -->
       <visual name="basket_ir_beam_line_vis">
-        <origin xyz="0.28 0 0.040" rpy="1.5708 0 0"/>
+        <origin xyz="0.40 0 0.040" rpy="1.5708 0 0"/>
         <geometry><cylinder radius="0.003" length="0.21"/></geometry>
         <material name="ir_beam_red"/>

File: ros2_ws/src/tennis_robot/urdf/tennis_robot.urdf.xacro (robot description, xacro)
@@ -5,4 +5,5 @@
   <xacro:include filename="components/funnel.urdf.xacro"/>
   <xacro:include filename="components/basket.urdf.xacro"/>
+  <xacro:include filename="components/battery.urdf.xacro"/>
   <xacro:include filename="components/drivetrain.urdf.xacro"/>
   <xacro:include filename="components/ros2_control.urdf.xacro"/>
@@ -38,9 +39,11 @@
   <xacro:arg name="intake_conveyor_x_bias" default="0.000"/>
   <xacro:arg name="intake_conveyor_z_bias" default="0.000"/>
-  <!-- Basket handoff geometry (ground frame for the floor top). Defaults are
-       the scoop-era launch design; the dual-wheel bench lowers these to make
-       the basket a low hopper behind the intake wheels (debug-log #41). -->
+  <!-- Bin v2 (docs/basket-bin-redesign-spec-el.md): sunken removable bin.
+       Ground-frame heights; front edge is pinned to the jump lip (0.425). -->
   <xacro:arg name="basket_floor_front_x" default="0.42"/>
-  <xacro:arg name="basket_floor_top_z" default="0.052"/>
+  <xacro:arg name="basket_floor_top_z" default="0.030"/>
+  <xacro:arg name="basket_rear_x" default="0.02"/>
+  <xacro:arg name="basket_half_width" default="0.14"/>
+  <xacro:arg name="basket_wall_top_z" default="0.25"/>
   <xacro:property name="chassis_x" value="0.92"/>
   <xacro:property name="chassis_y" value="0.58"/>
@@ -98,5 +101,5 @@
   <xacro:property name="intake_conveyor_length" value="0.200"/>
   <xacro:property name="scooper_pitch" value="0.1745"/>  <!-- 10 degrees; funnel-cheek tilt -->
-  <xacro:property name="lidar_xyz" value="-0.08 0 0.498"/>
+  <xacro:property name="lidar_xyz" value="-0.42 0 0.498"/>
   <xacro:property name="lidar_rpy" value="0 0 0"/>  <!-- level chassis: horizontal scan plane -->
   <xacro:property name="camera_xyz" value="0.535 0 0.443"/>
@@ -122,5 +125,5 @@
   <xacro:property name="ir_y" value="0.105"/>
   <xacro:property name="ir_z" value="-0.005"/>
-  <xacro:property name="basket_ir_x" value="0.28"/>
+  <xacro:property name="basket_ir_x" value="0.40"/>
   <xacro:property name="basket_ir_y" value="0.105"/>
   <xacro:property name="basket_ir_z" value="0.040"/>
@@ -243,5 +246,9 @@
       parent="base_link"
       floor_front_x="${float($(arg basket_floor_front_x))}"
-      floor_top_z_ground="${float($(arg basket_floor_top_z))}"/>
+      floor_top_z_ground="${float($(arg basket_floor_top_z))}"
+      rear_x="${float($(arg basket_rear_x))}"
+      half_width="${float($(arg basket_half_width))}"
+      wall_top_z_ground="${float($(arg basket_wall_top_z))}"/>
+  <xacro:battery_pack parent="base_link"/>
   <xacro:rplidar_c1_mount
       parent="base_link"
