Commit message: new form

File: ros2_ws/src/tennis_robot/urdf/components/base.urdf.xacro (robot description, xacro)
@@ -38,11 +38,34 @@
     <link name="base_link">
       <xacro:box_inertial mass="${chassis_mass}" x="${chassis_x}" y="${chassis_y}" z="${chassis_z}"/>
-      <collision name="chassis_col">
-        <origin xyz="0 0 0" rpy="0 0 0"/>
-        <geometry><box size="${chassis_x} ${chassis_y} ${chassis_z}"/></geometry>
+      <!-- Front-centre cutout (0.20 wide x 0.04 deep): the roller-first
+           intake channel wraps the ball around behind the roller close to
+           the chassis front edge (x=0.46); without the notch the plate
+           corner clips the rising ball by ~1 mm. Plate = two full-length
+           side strips + one centre strip ending at x=0.42. -->
+      <collision name="chassis_left_col">
+        <origin xyz="0 ${0.10 + (chassis_y / 2.0 - 0.10) / 2.0} 0" rpy="0 0 0"/>
+        <geometry><box size="${chassis_x} ${chassis_y / 2.0 - 0.10} ${chassis_z}"/></geometry>
       </collision>
-      <visual name="chassis_vis">
-        <origin xyz="0 0 0" rpy="0 0 0"/>
-        <geometry><box size="${chassis_x} ${chassis_y} ${chassis_z}"/></geometry>
+      <collision name="chassis_right_col">
+        <origin xyz="0 ${-(0.10 + (chassis_y / 2.0 - 0.10) / 2.0)} 0" rpy="0 0 0"/>
+        <geometry><box size="${chassis_x} ${chassis_y / 2.0 - 0.10} ${chassis_z}"/></geometry>
+      </collision>
+      <collision name="chassis_centre_col">
+        <origin xyz="-0.02 0 0" rpy="0 0 0"/>
+        <geometry><box size="${chassis_x - 0.04} 0.20 ${chassis_z}"/></geometry>
+      </collision>
+      <visual name="chassis_left_vis">
+        <origin xyz="0 ${0.10 + (chassis_y / 2.0 - 0.10) / 2.0} 0" rpy="0 0 0"/>
+        <geometry><box size="${chassis_x} ${chassis_y / 2.0 - 0.10} ${chassis_z}"/></geometry>
+        <material name="plywood"/>
+      </visual>
+      <visual name="chassis_right_vis">
+        <origin xyz="0 ${-(0.10 + (chassis_y / 2.0 - 0.10) / 2.0)} 0" rpy="0 0 0"/>
+        <geometry><box size="${chassis_x} ${chassis_y / 2.0 - 0.10} ${chassis_z}"/></geometry>
+        <material name="plywood"/>
+      </visual>
+      <visual name="chassis_centre_vis">
+        <origin xyz="-0.02 0 0" rpy="0 0 0"/>
+        <geometry><box size="${chassis_x - 0.04} 0.20 ${chassis_z}"/></geometry>
         <material name="plywood"/>
       </visual>
@@ -97,6 +120,8 @@
         <material name="anthracite"/>
       </visual>
+      <!-- Throat beam-line visual: matches ir_x/ir_z in tennis_robot.urdf.xacro
+           (nip jam detection, 40 mm above ground just behind the lip). -->
       <visual name="ir_beam_line_vis">
-        <origin xyz="0.54 0 0.053" rpy="1.5708 0 0"/>
+        <origin xyz="0.575 0 -0.005" rpy="1.5708 0 0"/>
         <geometry><cylinder radius="0.003" length="0.21"/></geometry>
         <material name="ir_beam_red"/>

File: ros2_ws/src/tennis_robot/urdf/components/basket.urdf.xacro (robot description, xacro)
@@ -13,29 +13,33 @@
         <inertia ixx="0.0001" ixy="0" ixz="0" iyy="0.0001" iyz="0" izz="0.0001"/>
       </inertial>
+      <!-- Floor + side walls extended forward to x=0.42 (base_link frame) so
+           the ball deflected off the intake deflector plate (lands ~x
+           0.32-0.42) drops onto the floor instead of falling back into the
+           channel. Floor top is 0.128 above ground. -->
       <collision name="basket_floor_col">
-        <origin xyz="0.10 0 0.073" rpy="0 0 0"/>
-        <geometry><box size="0.44 0.34 0.020"/></geometry>
+        <origin xyz="0.15 0 0.073" rpy="0 0 0"/>
+        <geometry><box size="0.54 0.34 0.020"/></geometry>
       </collision>
       <visual name="basket_floor_vis">
-        <origin xyz="0.10 0 0.073" rpy="0 0 0"/>
-        <geometry><box size="0.44 0.34 0.020"/></geometry>
+        <origin xyz="0.15 0 0.073" rpy="0 0 0"/>
+        <geometry><box size="0.54 0.34 0.020"/></geometry>
         <material name="basket_gray"/>
       </visual>
       <collision name="basket_left_wall_col">
-        <origin xyz="0.10 0.17 0.213" rpy="0 0 0"/>
-        <geometry><box size="0.44 0.020 0.28"/></geometry>
+        <origin xyz="0.15 0.17 0.213" rpy="0 0 0"/>
+        <geometry><box size="0.54 0.020 0.28"/></geometry>
       </collision>
       <visual name="basket_left_wall_vis">
-        <origin xyz="0.10 0.17 0.213" rpy="0 0 0"/>
-        <geometry><box size="0.44 0.020 0.28"/></geometry>
+        <origin xyz="0.15 0.17 0.213" rpy="0 0 0"/>
+        <geometry><box size="0.54 0.020 0.28"/></geometry>
         <material name="basket_gray"/>
       </visual>
       <collision name="basket_right_wall_col">
-        <origin xyz="0.10 -0.17 0.213" rpy="0 0 0"/>
-        <geometry><box size="0.44 0.020 0.28"/></geometry>
+        <origin xyz="0.15 -0.17 0.213" rpy="0 0 0"/>
+        <geometry><box size="0.54 0.020 0.28"/></geometry>
       </collision>
       <visual name="basket_right_wall_vis">
-        <origin xyz="0.10 -0.17 0.213" rpy="0 0 0"/>
-        <geometry><box size="0.44 0.020 0.28"/></geometry>
+        <origin xyz="0.15 -0.17 0.213" rpy="0 0 0"/>
+        <geometry><box size="0.54 0.020 0.28"/></geometry>
         <material name="basket_gray"/>
       </visual>

File: ros2_ws/src/tennis_robot/urdf/components/drivetrain.urdf.xacro (robot description, xacro)
@@ -75,5 +75,7 @@
     <link name="lift_wheel_link">
       <xacro:cylinder_inertial mass="${mass}" radius="${radius}" length="${width}" axis="y"/>
-      <!-- Small rigid hub; the paddles define the 100 mm swept envelope. -->
+      <!-- Small rigid hub; the paddles sweep the full `radius` envelope
+           (Ø90 mm with the current intake_radius=0.045). Roller-first design:
+           this envelope is the first hard contact with the ball. -->
       <collision name="core_col">
         <origin xyz="0 0 0" rpy="1.5708 0 0"/>
@@ -103,4 +105,47 @@
       <mu1>1.5</mu1>
       <mu2>1.5</mu2>
+      <!-- One contact sensor per paddle. Gazebo publishes the real physics
+           contact positions; gazebo_extras_node turns them into short-lived
+           red RViz markers and a /sim/roller_contact heartbeat. -->
+      <sensor name="roller_contact_0" type="contact">
+        <always_on>true</always_on><update_rate>100</update_rate>
+        <topic>/gz/roller_contact_0</topic>
+        <contact><collision>flap_0_col</collision></contact>
+      </sensor>
+      <sensor name="roller_contact_1" type="contact">
+        <always_on>true</always_on><update_rate>100</update_rate>
+        <topic>/gz/roller_contact_1</topic>
+        <contact><collision>flap_1_col</collision></contact>
+      </sensor>
+      <sensor name="roller_contact_2" type="contact">
+        <always_on>true</always_on><update_rate>100</update_rate>
+        <topic>/gz/roller_contact_2</topic>
+        <contact><collision>flap_2_col</collision></contact>
+      </sensor>
+      <sensor name="roller_contact_3" type="contact">
+        <always_on>true</always_on><update_rate>100</update_rate>
+        <topic>/gz/roller_contact_3</topic>
+        <contact><collision>flap_3_col</collision></contact>
+      </sensor>
+      <sensor name="roller_contact_4" type="contact">
+        <always_on>true</always_on><update_rate>100</update_rate>
+        <topic>/gz/roller_contact_4</topic>
+        <contact><collision>flap_4_col</collision></contact>
+      </sensor>
+      <sensor name="roller_contact_5" type="contact">
+        <always_on>true</always_on><update_rate>100</update_rate>
+        <topic>/gz/roller_contact_5</topic>
+        <contact><collision>flap_5_col</collision></contact>
+      </sensor>
+      <sensor name="roller_contact_6" type="contact">
+        <always_on>true</always_on><update_rate>100</update_rate>
+        <topic>/gz/roller_contact_6</topic>
+        <contact><collision>flap_6_col</collision></contact>
+      </sensor>
+      <sensor name="roller_contact_7" type="contact">
+        <always_on>true</always_on><update_rate>100</update_rate>
+        <topic>/gz/roller_contact_7</topic>
+        <contact><collision>flap_7_col</collision></contact>
+      </sensor>
     </gazebo>
   </xacro:macro>

File: ros2_ws/src/tennis_robot/urdf/components/funnel.urdf.xacro (robot description, xacro)
@@ -13,27 +13,60 @@
       </inertial>
       <visual name="funnel_left_cheek_vis">
-        <origin xyz="0.54 0.14 0.052" rpy="0 ${pitch} 0.25"/>
+        <origin xyz="0.60 0.145 0.052" rpy="0 ${pitch} 0.25"/>
         <geometry><box size="0.24 0.01 0.10"/></geometry>
         <material name="intake_orange"/>
       </visual>
+      <!-- Cheek collisions so the funnel physically guides off-centre balls
+           into the (narrower, scoop-width) intake instead of only looking
+           like it does. Mouth is ~0.35 m wide at the front tips, converging
+           to the 0.18 m roller/channel width at the intake mouth. -->
+      <collision name="funnel_left_cheek_col">
+        <origin xyz="0.60 0.145 0.052" rpy="0 ${pitch} 0.25"/>
+        <geometry><box size="0.24 0.01 0.10"/></geometry>
+      </collision>
       <visual name="funnel_right_cheek_vis">
-        <origin xyz="0.54 -0.14 0.052" rpy="0 ${pitch} -0.25"/>
+        <origin xyz="0.60 -0.145 0.052" rpy="0 ${pitch} -0.25"/>
         <geometry><box size="0.24 0.01 0.10"/></geometry>
         <material name="intake_orange"/>
       </visual>
-      <collision name="roller_exit_floor_col">
-        <!-- Closed 2 mm wedge: its front underside is exactly at the ground
-             plane and its 0.32 rad top surface rises toward the roller. -->
-        <origin xyz="0.54 0 0" rpy="0 0 0"/>
-        <geometry><mesh filename="package://tennis_robot/meshes/scooper_wedge.stl"/></geometry>
+      <collision name="funnel_right_cheek_col">
+        <origin xyz="0.60 -0.145 0.052" rpy="0 ${pitch} -0.25"/>
+        <geometry><box size="0.24 0.01 0.10"/></geometry>
       </collision>
-      <visual name="roller_exit_floor_vis">
-        <origin xyz="0.54 0 0" rpy="0 0 0"/>
-        <geometry><mesh filename="package://tennis_robot/meshes/scooper_wedge.stl"/></geometry>
+      <collision name="intake_channel_col">
+        <!-- Roller-first intake channel, entirely BEHIND the roller's
+             leading edge (envelope reaches x=0.595, effective channel tip at
+             x=0.540 after the rearward tuning offset):
+             2 mm tip on the ground plane, then a circular arc of radius
+             105 mm around the roller centre (0.55, 0.105 above ground) up to
+             a near-vertical rear wall ending at z=0.155. The paddled roller
+             (tennis_robot.urdf.xacro intake_*) is the first hard contact and
+             drives the ball around the channel. Mesh is generated in
+             funnel-frame coords by scripts/generate_curved_scoop_mesh.py —
+             keep the two in sync. -->
+        <!-- Shifted 15 mm rearward after the first mechanical-capture test:
+             this gives the paddle envelope more room to engage the ball
+             before the rigid channel can support / block it. -->
+        <origin xyz="-0.015 0 0" rpy="0 0 0"/>
+        <geometry><mesh filename="package://tennis_robot/meshes/curved_scoop.stl"/></geometry>
+      </collision>
+      <visual name="intake_channel_vis">
+        <origin xyz="-0.015 0 0" rpy="0 0 0"/>
+        <geometry><mesh filename="package://tennis_robot/meshes/curved_scoop.stl"/></geometry>
         <material name="intake_orange"/>
       </visual>
-      <visual name="internal_slide_vis">
-        <origin xyz="0.40 0 0.03" rpy="0 -0.12 0"/>
-        <geometry><box size="0.14 0.24 0.005"/></geometry>
+      <!-- Deflector plate above/behind the roller: catches the ball flung up
+           the rear wall (rising at x~0.48) and deflects it backward onto the
+           basket floor (top at 0.128 above ground, extended to x=0.42 —
+           basket.urdf.xacro). Ground-frame edges: front-high (0.49, 0.266),
+           rear-low (0.36, 0.204) — 76 mm above the basket floor so a 66 mm
+           ball can't jam under it; clears the roller envelope top (0.15). -->
+      <collision name="intake_deflector_col">
+        <origin xyz="0.425 0 0.197" rpy="0 -0.43 0"/>
+        <geometry><box size="0.15 0.20 0.006"/></geometry>
+      </collision>
+      <visual name="intake_deflector_vis">
+        <origin xyz="0.425 0 0.197" rpy="0 -0.43 0"/>
+        <geometry><box size="0.15 0.20 0.006"/></geometry>
         <material name="intake_orange"/>
       </visual>

File: ros2_ws/src/tennis_robot/urdf/tennis_robot.urdf.xacro (robot description, xacro)
@@ -39,15 +39,25 @@
   <xacro:property name="motor_radius" value="0.03"/>
   <xacro:property name="motor_length" value="0.10"/>
-  <!-- The 0.66 m scooper lip must meet the ball first. The single roller sits
-       60 mm behind it, over the rising ramp, so the scoop supports the ball
-       while the flaps drive it upward and inward. -->
-  <xacro:property name="intake_x" value="0.60"/>
-  <!-- Single-shaft flap roller: 100 mm swept diameter, with its tip envelope
-       still 64 mm above ground. The rigid core is smaller; eight paddles on
-       the same rotating link provide the compliant-roller approximation. -->
-  <xacro:property name="intake_z" value="0.069"/>
-  <xacro:property name="intake_radius" value="0.05"/>
-  <xacro:property name="intake_width" value="0.24"/>
-  <xacro:property name="scooper_pitch" value="0.1745"/>  <!-- 10 degrees -->
+  <!-- Roller-first intake (scripts/generate_curved_scoop_mesh.py): the paddled
+       roller is the FIRST hard contact with the ball — the entire channel
+       sits BEHIND the roller's leading edge. Envelope Ø90 x 180 mm, centre
+       105 mm above ground at x=0.55; the envelope reaches forward to
+       x=0.595 while the effective channel tip is at x=0.540 after the 15 mm
+       rearward tuning offset. A 66 mm ball meets the
+       paddle envelope at centre x=0.580 (contact 63 mm up the ball, above
+       its centre, pulling it in and down) ~14 mm before it could touch the
+       channel tip. The paddles then drive it around the rear-shifted channel
+       arc (nominal radius 105 mm),
+       up the rear wall and over the deflector into the basket
+       (funnel.urdf.xacro). The chassis plate has a matching front cutout
+       (base.urdf.xacro). The old push-ramp design (lip at 0.66, roller
+       centre 143.7 mm) never captured: the ball had to climb a passive
+       37-degree ramp before the roller could even touch it. -->
+  <xacro:property name="intake_x" value="0.55"/>
+  <!-- base_link origin is 45 mm above ground: 0.105 - 0.045 -->
+  <xacro:property name="intake_z" value="0.060"/>
+  <xacro:property name="intake_radius" value="0.045"/>
+  <xacro:property name="intake_width" value="0.18"/>
+  <xacro:property name="scooper_pitch" value="0.1745"/>  <!-- 10 degrees; funnel-cheek tilt -->
   <xacro:property name="lidar_xyz" value="-0.08 0 0.498"/>
   <xacro:property name="lidar_rpy" value="0 0 0"/>  <!-- level chassis: horizontal scan plane -->
@@ -55,7 +65,12 @@
   <xacro:property name="camera_rpy" value="0 0.273 0"/>  <!-- forward-down tilt ~15.6deg; preserves the old world aim (0.22 cam + 0.053 chassis pitch) now that the chassis is level -->
   <xacro:property name="sensor_update_rate" value="31.25"/>
-  <xacro:property name="ir_x" value="0.54"/>
+  <!-- Throat beam crosses the intake mouth at ball-centre height (40 mm
+       above ground = -0.005 in base_link), right where the paddles first
+       grab the ball (centre x~0.58): detects a ball at the nip (jam /
+       partial-capture detection). Collection confirmation is the BASKET
+       beam pair below — see gazebo_extras_node.py. -->
+  <xacro:property name="ir_x" value="0.575"/>
   <xacro:property name="ir_y" value="0.105"/>
-  <xacro:property name="ir_z" value="0.053"/>
+  <xacro:property name="ir_z" value="-0.005"/>
   <xacro:property name="basket_ir_x" value="0.28"/>
   <xacro:property name="basket_ir_y" value="0.105"/>
@@ -145,5 +160,5 @@
       joint_name="ir_left_joint"
       xyz="${ir_x} -${ir_y} ${ir_z}"
-      rpy="0 0 -1.5708"
+      rpy="0 0 1.5708"
       topic="/gz/ir_left"
       update_rate="${sensor_update_rate}"/>
@@ -153,5 +168,5 @@
       joint_name="ir_right_joint"
       xyz="${ir_x} ${ir_y} ${ir_z}"
-      rpy="0 0 1.5708"
+      rpy="0 0 -1.5708"
       topic="/gz/ir_right"
       update_rate="${sensor_update_rate}"/>
@@ -161,5 +176,5 @@
       joint_name="basket_ir_left_joint"
       xyz="${basket_ir_x} -${basket_ir_y} ${basket_ir_z}"
-      rpy="0 0 -1.5708"
+      rpy="0 0 1.5708"
       topic="/gz/basket_ir_left"
       update_rate="${sensor_update_rate}"/>
@@ -169,5 +184,5 @@
       joint_name="basket_ir_right_joint"
       xyz="${basket_ir_x} ${basket_ir_y} ${basket_ir_z}"
-      rpy="0 0 1.5708"
+      rpy="0 0 -1.5708"
       topic="/gz/basket_ir_right"
       update_rate="${sensor_update_rate}"/>
