Commit message: Document intake bench decision and tooling

File: ros2_ws/src/tennis_robot/urdf/components/base.urdf.xacro (robot description, xacro)
@@ -38,9 +38,7 @@
     <link name="base_link">
       <xacro:box_inertial mass="${chassis_mass}" x="${chassis_x}" y="${chassis_y}" z="${chassis_z}"/>
-      <!-- Front-centre cutout (0.20 wide x 0.04 deep): the roller-first
-           intake channel wraps the ball around behind the roller close to
-           the chassis front edge (x=0.46); without the notch the plate
-           corner clips the rising ball by ~1 mm. Plate = two full-length
-           side strips + one centre strip ending at x=0.42. -->
+      <!-- Front-centre cutout (0.20 wide x 0.04 deep): leaves clearance for
+           the launcher scoop/ramp path into the basket. Plate = two
+           full-length side strips + one centre strip ending at x=0.42. -->
       <collision name="chassis_left_col">
         <origin xyz="0 ${0.10 + (chassis_y / 2.0 - 0.10) / 2.0} 0" rpy="0 0 0"/>

File: ros2_ws/src/tennis_robot/urdf/components/basket.urdf.xacro (robot description, xacro)
@@ -13,10 +13,7 @@
         <inertia ixx="0.0001" ixy="0" ixz="0" iyy="0.0001" iyz="0" izz="0.0001"/>
       </inertial>
-      <!-- Floor extended forward to x=0.50 (base_link frame), 4.5 mm behind
-           the intake guide sheet, so the ball spin-walked backward off the
-           wheel top (intake-debug-log #15) lands on floor instead of falling
-           through the old x 0.42-0.50 gap to the court. Floor top is 0.128
-           above ground; the front corner stays 116 mm from the paddle axis
-           (sweep 50 mm). -->
+      <!-- Floor extended forward to x=0.50 (base_link frame) so a ball
+           launched up the scoop has a continuous landing surface into the
+           basket. Floor top is 0.128 m above ground. -->
       <collision name="basket_floor_col">
         <origin xyz="0.19 0 0.073" rpy="0 0 0"/>

File: ros2_ws/src/tennis_robot/urdf/components/drivetrain.urdf.xacro (robot description, xacro)
@@ -55,62 +55,25 @@
        the drive_wheel macro above). The old swivel-caster macro and its scrub
        resistance are gone. -->
-  <!-- One rubber intake paddle: a thin box on its own sprung revolute joint
-       so it bends RADIALLY when squeezing the ball. Spring params are
-       injected into the generated SDF by generate_robot_urdf.py (URDF cannot
-       express joint springs). One contact sensor per paddle, matching the
-       pre-existing /gz/roller_contact_0..7 bridges. -->
-  <xacro:macro name="intake_paddle" params="index angle hub_r paddle_len width thickness">
-    <link name="paddle_${index}_link">
-      <xacro:box_inertial mass="0.012" x="${paddle_len}" y="${width}" z="${thickness}"/>
-      <collision name="paddle_${index}_col">
-        <origin xyz="${paddle_len / 2} 0 0" rpy="0 0 0"/>
-        <geometry><box size="${paddle_len} ${width} ${thickness}"/></geometry>
-      </collision>
-      <visual name="paddle_${index}_vis">
-        <origin xyz="${paddle_len / 2} 0 0" rpy="0 0 0"/>
-        <geometry><box size="${paddle_len} ${width} ${thickness}"/></geometry>
-        <material name="intake_orange"/>
-      </visual>
-    </link>
-    <joint name="paddle_${index}_joint" type="revolute">
-      <parent link="lift_wheel_link"/>
-      <child link="paddle_${index}_link"/>
-      <!-- Root on the hub surface, +x pointing radially outward. -->
-      <origin xyz="${hub_r * cos(angle)} 0 ${hub_r * sin(angle)}" rpy="0 ${-angle} 0"/>
-      <axis xyz="0 1 0"/>
-      <limit lower="-1.2" upper="1.2" effort="10" velocity="60"/>
-      <dynamics damping="0.02"/>
-    </joint>
-    <gazebo reference="paddle_${index}_link">
-      <sensor name="roller_contact_${index}" type="contact">
-        <always_on>true</always_on><update_rate>100</update_rate>
-        <topic>/gz/roller_contact_${index}</topic>
-        <contact><collision>paddle_${index}_col</collision></contact>
-      </sensor>
-    </gazebo>
-  </xacro:macro>
   <xacro:macro name="intake_roller" params="x z radius width mass">
-    <!-- Paddle roller: hub + 8 sprung rubber paddles. A rigid fixed-axis
-         cylinder cannot friction-capture a rigid ball, and a 1-DOF sprung
-         carriage only yields VERTICALLY while the ball's orbit around the
-         roller needs ~2 mm of RADIAL compliance at every angle (the vertical
-         travel required blows up to 21+ mm behind the axis — every capture
-         stalled at exactly fwd=-75 mm; intake-debug-log #13). Per-paddle
-         springs give true radial compliance like the real foam surface:
-         paddle tips sweep radius+5 mm and bend back locally around the ball.
-         This restores the project's ORIGINAL paddle-wheel design — the
-         roller_contact_0..7 bridges are its infrastructure. -->
-    <xacro:property name="hub_radius" value="0.025"/>
-    <xacro:property name="paddle_length" value="${radius + 0.005 - hub_radius}"/>
+    <!-- Top intake roller: one continuous foam/rubber cylinder. The simulated
+         collision is rigid, but its outer radius and high friction represent
+         a lightly compressible foam sleeve that gives a short launch impulse
+         at the 2 mm scoop lip. It should not transport the ball along the
+         whole ramp. -->
     <link name="lift_wheel_link">
-      <xacro:cylinder_inertial mass="${mass}" radius="${hub_radius}" length="${width}" axis="y"/>
+      <xacro:cylinder_inertial mass="${mass}" radius="${radius}" length="${width}" axis="y"/>
       <collision name="roller_col">
         <origin xyz="0 0 0" rpy="1.5708 0 0"/>
-        <geometry><cylinder radius="${hub_radius}" length="${width}"/></geometry>
+        <geometry><cylinder radius="${radius}" length="${width}"/></geometry>
       </collision>
       <visual name="roller_vis">
         <origin xyz="0 0 0" rpy="1.5708 0 0"/>
-        <geometry><cylinder radius="${hub_radius}" length="${width}"/></geometry>
+        <geometry><cylinder radius="${radius}" length="${width}"/></geometry>
         <material name="rubber_black"/>
+      </visual>
+      <visual name="roller_spin_marker_vis">
+        <origin xyz="${radius} 0 0" rpy="0 0 0"/>
+        <geometry><box size="0.004 ${width + 0.004} 0.018"/></geometry>
+        <material name="safety_orange"/>
       </visual>
     </link>
@@ -124,21 +87,10 @@
       <mu1>0.8</mu1>
       <mu2>0.8</mu2>
+      <sensor name="roller_contact_0" type="contact">
+        <always_on>true</always_on><update_rate>100</update_rate>
+        <topic>/gz/roller_contact_0</topic>
+        <contact><collision>roller_col</collision></contact>
+      </sensor>
     </gazebo>
-    <xacro:intake_paddle index="0" angle="${0 * pi / 4}" hub_r="${hub_radius}"
-        paddle_len="${paddle_length}" width="${width}" thickness="0.004"/>
-    <xacro:intake_paddle index="1" angle="${1 * pi / 4}" hub_r="${hub_radius}"
-        paddle_len="${paddle_length}" width="${width}" thickness="0.004"/>
-    <xacro:intake_paddle index="2" angle="${2 * pi / 4}" hub_r="${hub_radius}"
-        paddle_len="${paddle_length}" width="${width}" thickness="0.004"/>
-    <xacro:intake_paddle index="3" angle="${3 * pi / 4}" hub_r="${hub_radius}"
-        paddle_len="${paddle_length}" width="${width}" thickness="0.004"/>
-    <xacro:intake_paddle index="4" angle="${4 * pi / 4}" hub_r="${hub_radius}"
-        paddle_len="${paddle_length}" width="${width}" thickness="0.004"/>
-    <xacro:intake_paddle index="5" angle="${5 * pi / 4}" hub_r="${hub_radius}"
-        paddle_len="${paddle_length}" width="${width}" thickness="0.004"/>
-    <xacro:intake_paddle index="6" angle="${6 * pi / 4}" hub_r="${hub_radius}"
-        paddle_len="${paddle_length}" width="${width}" thickness="0.004"/>
-    <xacro:intake_paddle index="7" angle="${7 * pi / 4}" hub_r="${hub_radius}"
-        paddle_len="${paddle_length}" width="${width}" thickness="0.004"/>
   </xacro:macro>
   <!--

File: ros2_ws/src/tennis_robot/urdf/components/funnel.urdf.xacro (robot description, xacro)
@@ -35,17 +35,10 @@
       </collision>
       <collision name="intake_channel_col">
-        <!-- Roller-first intake channel, entirely BEHIND the roller's
-             leading edge (envelope reaches x=0.595, effective channel tip at
-             x=0.540 after the rearward tuning offset):
-             2 mm tip on the ground plane, then a circular arc of radius
-             105 mm around the roller centre (0.55, 0.105 above ground) up to
-             a near-vertical rear wall ending at z=0.155. The paddled roller
-             (tennis_robot.urdf.xacro intake_*) is the first hard contact and
-             drives the ball around the channel. Mesh is generated in
+        <!-- Launcher scoop: a 2 mm entry lip creates the initial resistance
+             needed for roller bite, then the ramp quickly opens away from
+             the roller and rises toward the basket. This is a guide/launch
+             ramp, not a curved conveyor channel. Mesh is generated in
              funnel-frame coords by scripts/generate_curved_scoop_mesh.py —
              keep the two in sync. -->
-        <!-- Shifted 15 mm rearward after the first mechanical-capture test:
-             this gives the paddle envelope more room to engage the ball
-             before the rigid channel can support / block it. -->
         <origin xyz="-0.015 0 0" rpy="0 0 0"/>
         <geometry><mesh filename="package://tennis_robot/meshes/curved_scoop.stl"/></geometry>
@@ -56,18 +49,7 @@
         <material name="intake_orange"/>
       </visual>
-      <!-- Spin-walk ceiling over the paddle-wheel top: the paddles carry the
-           ball around the guide and juggle it at the wheel top (ground z
-           ~162-171 centre) with BACKSPIN. This front-LOW / rear-HIGH plate
-           sits just inside the juggle band so the spinning ball presses its
-           top against the underside and friction walks it BACKWARD over the
-           guide edge onto the (forward-extended) basket floor. Ground-frame
-           edges: front-low (0.593, 0.172) — 15.8 mm from the paddle tips so
-           the ball cannot escape forward — rear-high (0.447, 0.238). The old
-           front-high plate assumed a ballistic fling to z 204+ that the
-           paddle transport never reaches (intake-debug-log #15). -->
-      <!-- Raised +40 mm after the spiral-guide exit (intake-debug-log #17):
-           the paddles now push the ball positively over the spiral edge at
-           (0.554, 0.183), so this plate is only a safety net for wild
-           bounces, out of the exit trajectory. -->
+      <!-- High safety deflector only. The launcher path should not depend on
+           this ceiling for transport; it is kept above the expected ramp
+           trajectory to catch wild rebounds. -->
       <collision name="intake_deflector_col">
         <origin xyz="0.52 0 0.207" rpy="0 0.43 0"/>

File: ros2_ws/src/tennis_robot/urdf/components/materials.urdf.xacro (robot description, xacro)
@@ -9,4 +9,7 @@
   <material name="intake_orange">
     <color rgba="0.96 0.52 0.10 1"/>
+  </material>
+  <material name="safety_orange">
+    <color rgba="1.0 0.24 0.02 1"/>
   </material>
   <material name="mount_gray">

File: ros2_ws/src/tennis_robot/urdf/tennis_robot.urdf.xacro (robot description, xacro)
@@ -42,19 +42,13 @@
   <xacro:property name="motor_radius" value="0.03"/>
   <xacro:property name="motor_length" value="0.10"/>
-  <!-- Roller-first intake (scripts/generate_curved_scoop_mesh.py): the solid
-       roller is the FIRST hard contact with the ball — the entire channel
-       sits BEHIND the roller's leading edge. Envelope Ø90 x 180 mm, centre
-       112 mm above ground at x=0.60; the envelope reaches forward to
-       x=0.645 while the effective channel tip is at x=0.585. A 66 mm ball
-       therefore meets the roller before the rigid central scoop geometry.
-       The roller then drives it around the concentric channel arc
-       (nominal radius 108 mm),
-       up the rear wall and over the deflector into the basket
-       (funnel.urdf.xacro). The chassis plate has a matching front cutout
-       (base.urdf.xacro). The old push-ramp design (lip at 0.66, roller
-       centre 143.7 mm) never captured: the ball had to climb a passive
-       37-degree ramp before the roller could even touch it. -->
-  <!-- 50 mm forward of the original x=0.55 position so the roller, rather
-       than the scoop / funnel cheeks, is the first central hard contact. -->
+  <!-- Top-roller launcher intake (scripts/generate_curved_scoop_mesh.py):
+       the scoop is NOT a transport channel. Its front lip sits about 2 mm
+       above the court to give the ball a short, controlled resistance point
+       against the top roller. The roller should impart a brief launch impulse;
+       after that bite zone the ramp opens away from the roller so the ball
+       rides up by momentum and drops into the basket. Avoid tuning this back
+       into a continuous pinch path between roller and scoop. -->
+  <!-- Kept forward so the roller/lip bite happens before the funnel cheeks or
+       the main ramp can shove the ball sideways. -->
   <xacro:property name="intake_x" value="${0.60 + float($(arg intake_roller_x_offset))}"/>
   <!-- base_link origin is 45 mm above ground: 0.112 - 0.045. With a 45 mm
@@ -74,5 +68,5 @@
        above ground, just inside the funnel cheek at y=0.145), aimed
        diagonally inward-up-forward at the roller/lip nip. A head-on underside
-       mount is blocked by the scoop channel itself (verified: its depth
+       mount is blocked by the scoop/ramp itself (verified: its depth
        camera read a solid surface ~8 cm away filling the whole frame), so the
        line of sight comes in from the side of the channel where nothing
@@ -85,10 +79,10 @@
   <xacro:property name="intake_debug_camera_rpy" value="0 -0.289 -0.882"/>
   <!-- Throat beam crosses the intake mouth at ball-centre height (40 mm
-       above ground = -0.005 in base_link), right where the paddles first
-       grab the ball (centre x~0.58): detects a ball at the nip (jam /
+       above ground = -0.005 in base_link), right where the foam roller first
+       bites the ball (centre x~0.58): detects a ball at the nip (jam /
        partial-capture detection). Collection confirmation is the BASKET
        beam pair below — see gazebo_extras_node.py. -->
   <!-- Trigger just before the ball reaches the roller envelope. The first
-       paddle contact is at ball-centre x≈0.597 m, so a beam behind that point
+       roller contact is at ball-centre x≈0.597 m, so a beam behind that point
        cannot start a stationary roller in time. -->
   <xacro:property name="ir_x" value="0.620"/>

Commit message: feat(collection): harden intake and recovery runs

File: ros2_ws/src/tennis_robot/urdf/components/base.urdf.xacro (robot description, xacro)
@@ -27,5 +27,6 @@
     </inertial>
   </xacro:macro>
-  <xacro:macro name="tennis_robot_base" params="chassis_x chassis_y chassis_z base_link_height chassis_mass">
+  <xacro:macro name="tennis_robot_base"
+               params="chassis_x chassis_y chassis_z base_link_height chassis_mass entry_beam_x entry_beam_z entry_beam_width">
     <link name="base_footprint"/>
     <joint name="base_footprint_joint" type="fixed">
@@ -120,9 +121,10 @@
         <material name="anthracite"/>
       </visual>
-      <!-- Throat beam-line visual: matches ir_x/ir_z in tennis_robot.urdf.xacro
-           (nip jam detection, 40 mm above ground just behind the lip). -->
+      <!-- Entry beam-line visual. Its position and width are injected from the
+           same properties that place the two Gazebo rays, so diagnostics can
+           never drift away from the actual sensing geometry. -->
       <visual name="ir_beam_line_vis">
-        <origin xyz="0.575 0 -0.005" rpy="1.5708 0 0"/>
-        <geometry><cylinder radius="0.003" length="0.21"/></geometry>
+        <origin xyz="${entry_beam_x} 0 ${entry_beam_z}" rpy="1.5708 0 0"/>
+        <geometry><cylinder radius="0.003" length="${entry_beam_width}"/></geometry>
         <material name="ir_beam_red"/>
       </visual>

File: ros2_ws/src/tennis_robot/urdf/tennis_robot.urdf.xacro (robot description, xacro)
@@ -128,7 +128,7 @@
        wheel cylinders span x = nip_x ± Rw = 0.53..0.65, so a beam inside
        that band would stare at the wheels and read permanently broken.
-       At x=0.670 it fires when the ball centre is ~57 mm before first wheel
-       contact (ball-centre x≈0.613). Collection confirmation is the BASKET
-       beam pair below — see gazebo_extras_node.py. -->
+       At x=0.720 it fires before first wheel contact, leaving time to start
+       or maintain the rollers. Collection confirmation is the BASKET beam
+       pair below — see gazebo_extras_node.py. -->
   <xacro:property name="ir_x" value="0.720"/>
   <xacro:property name="ir_y" value="0.105"/>
@@ -151,5 +151,8 @@
       chassis_z="${chassis_z}"
       base_link_height="${base_link_height}"
-      chassis_mass="${chassis_mass}"/>
+      chassis_mass="${chassis_mass}"
+      entry_beam_x="${ir_x}"
+      entry_beam_z="${ir_z}"
+      entry_beam_width="${2.0 * ir_y}"/>
   <!-- Motors are fixed to the chassis top. Each shaft shares its x/z centre
        with the corresponding wheel joint; only y differs along the shaft. -->
