Commit message: Add spiral guide exit, align court visual/collision, log tests 10-12
- Spiral guide (R 109->101 over 50deg wrap): a concentric guide can never
  end inside the paddles' 83mm drive circle, so the ball always parked just
  out of reach (tests 9-10). With the taper the exit edge sits deep in the
  drive zone; 14mm taper was too aggressive (ball slipped between fully
  bent paddles, test11), 8mm transports cleanly (test12).
- Court ground collision aligned to its visual (-0.01 pose): the physics
  surface sat 10mm above the visible court, making balls/robot appear to
  float and offsetting all ground-truth z by +10mm.
- Deflector raised to a safety-net position out of the exit trajectory.
- Remaining (intake-debug-log #19): test12 shows perfect transport but the
  ball now rides over the wheel top and launches forward — needs a stripper
  plate at the spiral exit (specified with numbers in the log).

Co-Authored-By: Claude Fable 5 <noreply@anthropic.com>

File: ros2_ws/src/tennis_robot/urdf/components/funnel.urdf.xacro (robot description, xacro)
@@ -66,10 +66,14 @@
            front-high plate assumed a ballistic fling to z 204+ that the
            paddle transport never reaches (intake-debug-log #15). -->
+      <!-- Raised +40 mm after the spiral-guide exit (intake-debug-log #17):
+           the paddles now push the ball positively over the spiral edge at
+           (0.554, 0.183), so this plate is only a safety net for wild
+           bounces, out of the exit trajectory. -->
       <collision name="intake_deflector_col">
-        <origin xyz="0.52 0 0.167" rpy="0 0.43 0"/>
+        <origin xyz="0.52 0 0.207" rpy="0 0.43 0"/>
         <geometry><box size="0.16 0.20 0.006"/></geometry>
       </collision>
       <visual name="intake_deflector_vis">
-        <origin xyz="0.52 0 0.167" rpy="0 0.43 0"/>
+        <origin xyz="0.52 0 0.207" rpy="0 0.43 0"/>
         <geometry><box size="0.16 0.20 0.006"/></geometry>
         <material name="intake_orange"/>

Commit message: Net-collision fixes: timeout-first approach, phantom gate, LiDAR guard, real net line, narrower funnel exit
Run 3 drove into the net chasing a phantom map entry for 78 s
(collection-route-debug-log-el #6). Four roots, four fixes:
- The approach gave_up/timeout check now runs BEFORE every early-return
  branch (the turn-toward-target branch used to starve it).
- Phantom gate: no live sighting within the relock gate by MISSING_SCAN_S
  from the 1.3 m standoff marks the stop missing instead of dead-reckoning
  a capture into whatever stands there.
- LiDAR forward guard during fine approach (COLLECT_ROUTE_FRONT_BLOCK_M,
  1.45 m from the mast = ~15 cm before funnel contact): the capture stream
  has no costmap and the lidar plane cannot see balls, so anything solid
  ahead is net/fence.
- Side classification now uses the surveyed net line (CourtModel.same_side/
  contains) in the plan, insertions and the collect_route observation
  filter; across_net(net_x=0) only holds in net-centred frames — this map
  has the net at x~8.

Also (intake debug-log #59, user-approved): funnel cheek rear tips pulled
in from (0.647,±0.146) to (0.680,±0.104) so the exit corridor caps the
ball centre at ±0.066 — inside the bench-validated ±0.08 nip envelope;
front opening unchanged, 91 mm wheel clearance. Bench sweep pending.

Co-Authored-By: Claude Fable 5 <noreply@anthropic.com>

File: ros2_ws/src/tennis_robot/urdf/components/funnel.urdf.xacro (robot description, xacro)
@@ -19,28 +19,31 @@
       </inertial>
       <xacro:if value="${enable_cheeks}">
-        <!-- Cheeks hand the ball off to the intake wheels' front quadrants:
-             rear tips at ~(0.647, ±0.146), a clear 81 mm from the wheel
-             centres (0.590, ±0.090, r=0.060+carriage travel). The spinning
-             wheel fronts continue the convergence (their front surfaces
-             sweep toward the centreline), so the cheeks only need to bring
-             the ball inside |y| < ~0.14. The old cheeks at x=0.60 would
-             intersect the wheel cylinders (51 mm < 65 mm clearance). -->
+        <!-- Cheeks guide the ball INTO the wheel nip, not just near it
+             (intake debug-log #59): front tips unchanged at ~(0.876, ±0.205)
+             (mouth 410 mm), rear tips pulled in to ~(0.680, ±0.104) so the
+             exit corridor caps the ball centre at |y| ≤ ~0.066 — inside the
+             bench-validated ±0.08 envelope. The old rear tips at ±0.146 let
+             the ball exit at |y| ≤ 0.108 and meet the wheel's OUTER front
+             quadrant (surface sweeping outward), deflecting it sideways
+             (collection-route-debug-log-el #3). Rear tips clear the wheel
+             centres (0.590, ±0.090) by 91 mm — rule is ≥65 mm (cylinder
+             r=0.060 + carriage travel). -->
         <visual name="funnel_left_cheek_vis">
-          <origin xyz="0.76 0.175 0.052" rpy="0 ${pitch} 0.25"/>
-          <geometry><box size="0.24 0.01 0.10"/></geometry>
+          <origin xyz="0.778 0.1545 0.052" rpy="0 ${pitch} 0.476"/>
+          <geometry><box size="0.2205 0.01 0.10"/></geometry>
           <material name="intake_orange"/>
         </visual>
         <collision name="funnel_left_cheek_col">
-          <origin xyz="0.76 0.175 0.052" rpy="0 ${pitch} 0.25"/>
-          <geometry><box size="0.24 0.01 0.10"/></geometry>
+          <origin xyz="0.778 0.1545 0.052" rpy="0 ${pitch} 0.476"/>
+          <geometry><box size="0.2205 0.01 0.10"/></geometry>
         </collision>
         <visual name="funnel_right_cheek_vis">
-          <origin xyz="0.76 -0.175 0.052" rpy="0 ${pitch} -0.25"/>
-          <geometry><box size="0.24 0.01 0.10"/></geometry>
+          <origin xyz="0.778 -0.1545 0.052" rpy="0 ${pitch} -0.476"/>
+          <geometry><box size="0.2205 0.01 0.10"/></geometry>
           <material name="intake_orange"/>
         </visual>
         <collision name="funnel_right_cheek_col">
-          <origin xyz="0.76 -0.175 0.052" rpy="0 ${pitch} -0.25"/>
-          <geometry><box size="0.24 0.01 0.10"/></geometry>
+          <origin xyz="0.778 -0.1545 0.052" rpy="0 ${pitch} -0.476"/>
+          <geometry><box size="0.2205 0.01 0.10"/></geometry>
         </collision>
       </xacro:if>
