Commit message: Add basket handoff package: spin-walk ceiling and forward-extended floor
The paddle wheel carries the ball to its top and juggles it there with
backspin — the wheel top always drives forward, so the ball can never be
pushed backward into the basket by the wheel itself (collect_test8,
intake-debug-log #15).

- Deflector plate repositioned from a ballistic front-high catcher (which
  the paddle transport never reaches) to a front-low/rear-high ceiling just
  inside the juggle band: the backspinning ball presses its top against the
  underside and friction (new mu 1.2 patch) walks it backward over the
  guide edge. Its front edge also closes the forward escape (15.8 mm to the
  paddle tips).
- Basket floor extended forward to x=0.50, closing the x 0.42-0.50 gap the
  descending ball would otherwise fall through to the court.

Co-Authored-By: Claude Fable 5 <noreply@anthropic.com>

File: ros2_ws/src/tennis_robot/urdf/components/basket.urdf.xacro (robot description, xacro)
@@ -13,15 +13,17 @@
         <inertia ixx="0.0001" ixy="0" ixz="0" iyy="0.0001" iyz="0" izz="0.0001"/>
       </inertial>
-      <!-- Floor + side walls extended forward to x=0.42 (base_link frame) so
-           the ball deflected off the intake deflector plate (lands ~x
-           0.32-0.42) drops onto the floor instead of falling back into the
-           channel. Floor top is 0.128 above ground. -->
+      <!-- Floor extended forward to x=0.50 (base_link frame), 4.5 mm behind
+           the intake guide sheet, so the ball spin-walked backward off the
+           wheel top (intake-debug-log #15) lands on floor instead of falling
+           through the old x 0.42-0.50 gap to the court. Floor top is 0.128
+           above ground; the front corner stays 116 mm from the paddle axis
+           (sweep 50 mm). -->
       <collision name="basket_floor_col">
-        <origin xyz="0.15 0 0.073" rpy="0 0 0"/>
-        <geometry><box size="0.54 0.34 0.020"/></geometry>
+        <origin xyz="0.19 0 0.073" rpy="0 0 0"/>
+        <geometry><box size="0.62 0.34 0.020"/></geometry>
       </collision>
       <visual name="basket_floor_vis">
-        <origin xyz="0.15 0 0.073" rpy="0 0 0"/>
-        <geometry><box size="0.54 0.34 0.020"/></geometry>
+        <origin xyz="0.19 0 0.073" rpy="0 0 0"/>
+        <geometry><box size="0.62 0.34 0.020"/></geometry>
         <material name="basket_gray"/>
       </visual>

File: ros2_ws/src/tennis_robot/urdf/components/funnel.urdf.xacro (robot description, xacro)
@@ -56,17 +56,21 @@
         <material name="intake_orange"/>
       </visual>
-      <!-- Deflector plate above/behind the roller: catches the ball flung up
-           the rear wall (rising at x~0.48) and deflects it backward onto the
-           basket floor (top at 0.128 above ground, extended to x=0.42 —
-           basket.urdf.xacro). Ground-frame edges: front-high (0.49, 0.266),
-           rear-low (0.36, 0.204) — 76 mm above the basket floor so a 66 mm
-           ball can't jam under it; clears the roller envelope top (0.15). -->
+      <!-- Spin-walk ceiling over the paddle-wheel top: the paddles carry the
+           ball around the guide and juggle it at the wheel top (ground z
+           ~162-171 centre) with BACKSPIN. This front-LOW / rear-HIGH plate
+           sits just inside the juggle band so the spinning ball presses its
+           top against the underside and friction walks it BACKWARD over the
+           guide edge onto the (forward-extended) basket floor. Ground-frame
+           edges: front-low (0.593, 0.172) — 15.8 mm from the paddle tips so
+           the ball cannot escape forward — rear-high (0.447, 0.238). The old
+           front-high plate assumed a ballistic fling to z 204+ that the
+           paddle transport never reaches (intake-debug-log #15). -->
       <collision name="intake_deflector_col">
-        <origin xyz="0.425 0 0.197" rpy="0 -0.43 0"/>
-        <geometry><box size="0.15 0.20 0.006"/></geometry>
+        <origin xyz="0.52 0 0.167" rpy="0 0.43 0"/>
+        <geometry><box size="0.16 0.20 0.006"/></geometry>
       </collision>
       <visual name="intake_deflector_vis">
-        <origin xyz="0.425 0 0.197" rpy="0 -0.43 0"/>
-        <geometry><box size="0.15 0.20 0.006"/></geometry>
+        <origin xyz="0.52 0 0.167" rpy="0 0.43 0"/>
+        <geometry><box size="0.16 0.20 0.006"/></geometry>
         <material name="intake_orange"/>
       </visual>

Commit message: Live integration: winning defaults, low-hopper sensing, Jazzy motion chain
Make the Phase 1-4 bench-proven intake geometry the default everywhere
(generator, mesh script, xacro args, sweep harness, analyzer, run_ubuntu.sh
fallbacks) and add full dual-wheel env passthrough to docker-compose (it
previously forwarded only roller-era vars).

Adapt collection sensing to the low hopper: basket IR beam pair drops from
the scoop-era 0.158 to 0.085 ground (rolling-ball equator), and the
controller's basket zone becomes x -0.12..0.42 with min ball z 0.075.

Fix the live motion chain, dead twice over on native Jazzy (debug-log #43):
the motor adapter published to bare /cmd_vel, which the gz bridge fed to the
removed Gazebo diff-drive plugin - it now enters twist_mux as
/cmd_vel_collection (priority 70). And Jazzy's twist_mux/diff_drive are
TwistStamped-only, so sim.launch.py wires distro-aware: a new
cmd_vel_stamp_relay node restamps the Twist producers ahead of the mux and
the mux output goes straight to ~/cmd_vel; Humble keeps the old unstamped
chain. sim.launch.py also respects ROBOT_*_FILE env overrides now.

Live collect_one (full stack with YOLO perception): the robot drives and
runs the complete FSM cycle for the first time on native Jazzy. Collection
still fails upstream of the intake: ground truth shows closest approach to
any ball is 0.73 m - the camera loses balls in the near field and the blind
final leg misses. That approach-accuracy campaign is logged as next work.

Co-Authored-By: Claude Fable 5 <noreply@anthropic.com>

File: ros2_ws/src/tennis_robot/urdf/components/basket.urdf.xacro (robot description, xacro)
@@ -62,6 +62,8 @@
         <material name="basket_gray"/>
       </visual>
+      <!-- Matches basket_ir_z in tennis_robot.urdf.xacro: beam at rolling
+           ball equator height in the low hopper (0.085 ground). -->
       <visual name="basket_ir_beam_line_vis">
-        <origin xyz="0.28 0 0.113" rpy="1.5708 0 0"/>
+        <origin xyz="0.28 0 0.040" rpy="1.5708 0 0"/>
         <geometry><cylinder radius="0.003" length="0.21"/></geometry>
         <material name="ir_beam_red"/>

File: ros2_ws/src/tennis_robot/urdf/tennis_robot.urdf.xacro (robot description, xacro)
@@ -21,7 +21,7 @@
        Injected from INTAKE_WHEEL_* envs by scripts/generate_robot_urdf.py. -->
   <xacro:arg name="intake_wheel_radius" default="0.060"/>
-  <xacro:arg name="intake_wheel_gap" default="0.060"/>
-  <xacro:arg name="intake_nip_x" default="0.590"/>
-  <xacro:arg name="intake_wheel_tilt_deg" default="0.0"/>
+  <xacro:arg name="intake_wheel_gap" default="0.056"/>
+  <xacro:arg name="intake_nip_x" default="0.540"/>
+  <xacro:arg name="intake_wheel_tilt_deg" default="35.0"/>
   <xacro:arg name="intake_wheel_max_vel" default="26.3"/>
   <xacro:arg name="intake_wheel_effort" default="1.77"/>
@@ -41,6 +41,6 @@
        the scoop-era launch design; the dual-wheel bench lowers these to make
        the basket a low hopper behind the intake wheels (debug-log #41). -->
-  <xacro:arg name="basket_floor_front_x" default="0.50"/>
-  <xacro:arg name="basket_floor_top_z" default="0.128"/>
+  <xacro:arg name="basket_floor_front_x" default="0.42"/>
+  <xacro:arg name="basket_floor_top_z" default="0.052"/>
   <xacro:property name="chassis_x" value="0.92"/>
   <xacro:property name="chassis_y" value="0.58"/>
@@ -124,5 +124,5 @@
   <xacro:property name="basket_ir_x" value="0.28"/>
   <xacro:property name="basket_ir_y" value="0.105"/>
-  <xacro:property name="basket_ir_z" value="0.113"/>
+  <xacro:property name="basket_ir_z" value="0.040"/>
   <xacro:property name="max_linear_acceleration" value="2.0"/>
   <xacro:property name="max_angular_acceleration" value="4.0"/>
