Commit message: Full-basket 45-ball collection: entry hood + launch profile defaults
The 45-ball loaded basket failed two ways: stored balls escaped during
entry, and the incoming ball bounced off the pile back out of the bin.
Fixes (debug log #54-56):

- Entry hood (roof + side cheeks, rear overhang 40mm, rear clearance
  120mm): stored retention 45/45 in every run since.
- Controlled-launch ramp profile clears the pile where wheel-only
  rolling entry is marginal: 5x repeatability gate at load 45 gave
  launch 5/5 PASS vs rolling 2/5 FAIL; unloaded regression 5/5.
- Launch profile + hood are now the defaults across the whole fallback
  chain (generator, scoop mesh, xacro, sweep harness, docker-compose,
  run_ubuntu). Clean-env load-45 verification run passed transport 6/6
  and basket evidence 8/8 straight from defaults.
- Sweep harness: 45-ball preload with readiness gate, probe duration
  default 35s (25s truncated dwell/settle measurements), launch probe
  window from 0.70m, bench_config echo fallbacks synced (fixes floor
  display bug 0.50/0.128 -> real 0.42/0.025).
- run_ubuntu center lip aligned to the bench-validated 0.010 (live was
  silently running 0.020).
- New analyze_launch_ballistics.py: fits release vector on airborne
  samples (adaptive window until first landing) and reports predicted
  apex/range/landing vs the inverse-ballistic contract, with tests.

Co-Authored-By: Claude Fable 5 <noreply@anthropic.com>

File: ros2_ws/src/tennis_robot/urdf/components/ros2_control.urdf.xacro (robot description, xacro)
@@ -18,5 +18,5 @@
   <!-- intake_max_vel = GB37Y3530-12V-251R no-load speed (251 RPM = 26.3 rad/s). -->
   <xacro:macro name="tennis_robot_ros2_control"
-               params="sim_mode:=true controllers_config wheel_max_vel:=20.0 intake_max_vel:=26.3 enable_assist:=false enable_conveyor:=false">
+               params="sim_mode:=true controllers_config wheel_max_vel:=20.0 intake_max_vel:=26.3 expose_intake_carriage_state:=false enable_assist:=false enable_conveyor:=false">
     <ros2_control name="TennisRobotSystem" type="system">
       <!-- Hardware backend (the only sim/real difference) -->
@@ -98,4 +98,19 @@
         <state_interface name="velocity"/>
       </joint>
+      <!-- Gazebo-only observability for the passive spring carriages. The
+           physical prototype has no carriage encoder, so these state-only
+           interfaces must not become part of the real hardware contract. -->
+      <xacro:if value="${sim_mode}">
+        <xacro:if value="${expose_intake_carriage_state}">
+          <joint name="intake_wheel_left_carriage_joint">
+            <state_interface name="position"/>
+            <state_interface name="velocity"/>
+          </joint>
+          <joint name="intake_wheel_right_carriage_joint">
+            <state_interface name="position"/>
+            <state_interface name="velocity"/>
+          </joint>
+        </xacro:if>
+      </xacro:if>
       <!-- Optional Phase 3 second-stage assist roller. -->
       <xacro:if value="${enable_assist}">

File: ros2_ws/src/tennis_robot/urdf/tennis_robot.urdf.xacro (robot description, xacro)
@@ -19,4 +19,5 @@
   <xacro:arg name="sim_mode" default="true"/>
   <xacro:arg name="controllers_config" default="config/controllers.yaml"/>
+  <xacro:arg name="expose_intake_carriage_state" default="false"/>
   <!-- Dual-wheel intake tuning (docs/dual-wheel-intake-design-el.md).
        Injected from INTAKE_WHEEL_* envs by scripts/generate_robot_urdf.py. -->
@@ -46,4 +47,12 @@
   <xacro:arg name="basket_half_width" default="0.14"/>
   <xacro:arg name="basket_wall_top_z" default="0.25"/>
+  <xacro:arg name="basket_center_lip_height" default="0.010"/>
+  <xacro:arg name="basket_management_run" default="0.14"/>
+  <xacro:arg name="basket_management_rise" default="0.010"/>
+  <xacro:arg name="basket_receiver_run" default="0.050"/>
+  <xacro:arg name="basket_receiver_rise" default="0.005"/>
+  <xacro:arg name="basket_hood_rear_overhang" default="0.040"/>
+  <xacro:arg name="basket_hood_rear_clearance_z" default="0.120"/>
+  <xacro:arg name="basket_hood_front_clearance_z" default="0.135"/>
   <xacro:property name="chassis_x" value="0.92"/>
   <xacro:property name="chassis_y" value="0.58"/>
@@ -125,7 +134,9 @@
   <xacro:property name="ir_y" value="0.105"/>
   <xacro:property name="ir_z" value="-0.005"/>
-  <xacro:property name="basket_ir_x" value="0.40"/>
+  <!-- Basket confirmation beam crosses the midpoint of the inclined receiver
+       at the rolling ball's equator. Sensor coordinates are base_link-frame. -->
+  <xacro:property name="basket_ir_x" value="${float($(arg basket_floor_front_x)) + float($(arg basket_receiver_run)) / 2.0}"/>
   <xacro:property name="basket_ir_y" value="0.105"/>
-  <xacro:property name="basket_ir_z" value="0.040"/>
+  <xacro:property name="basket_ir_z" value="${float($(arg basket_floor_top_z)) + float($(arg basket_management_rise)) + float($(arg basket_receiver_rise)) / 2.0 + 0.033 - base_link_height}"/>
   <xacro:property name="max_linear_acceleration" value="2.0"/>
   <xacro:property name="max_angular_acceleration" value="4.0"/>
@@ -249,5 +260,13 @@
       rear_x="${float($(arg basket_rear_x))}"
       half_width="${float($(arg basket_half_width))}"
-      wall_top_z_ground="${float($(arg basket_wall_top_z))}"/>
+      wall_top_z_ground="${float($(arg basket_wall_top_z))}"
+      center_lip_height="${float($(arg basket_center_lip_height))}"
+      management_run="${float($(arg basket_management_run))}"
+      management_rise="${float($(arg basket_management_rise))}"
+      receiver_run="${float($(arg basket_receiver_run))}"
+      receiver_rise="${float($(arg basket_receiver_rise))}"
+      hood_rear_overhang="${float($(arg basket_hood_rear_overhang))}"
+      hood_rear_clearance_z_ground="${float($(arg basket_hood_rear_clearance_z))}"
+      hood_front_clearance_z_ground="${float($(arg basket_hood_front_clearance_z))}"/>
   <xacro:battery_pack parent="base_link"/>
   <xacro:rplidar_c1_mount
@@ -316,4 +335,5 @@
       sim_mode="$(arg sim_mode)"
       controllers_config="$(arg controllers_config)"
+      expose_intake_carriage_state="$(arg expose_intake_carriage_state)"
       intake_max_vel="${intake_wheel_max_vel}"
       enable_assist="$(arg enable_assist)"
