Commit message: feat(throwing): Throwing Mode slice + COLLECT/LAUNCH mechanical variants
Checkpoint. The Throwing Mode vertical slice (domain model, console service,
HTTP API, UI view) reaches COMPLETED end-to-end in live Gazebo; the mechanical
configuration it needs, and several defects the live runs exposed, are fixed
alongside it.

Mechanical variants
  The intake assembly (x 446..884, z 0..281 mm) and the flywheel launcher
  (wheels x 459..661, z 162..268 mm) claim the same front volume, so no
  configuration may carry both. option-a-launch fits the launcher and omits the
  intake; baseline/option-a-collect keep the intake and default the launcher
  OFF, so a plain run_native.sh can no longer put a collision plate across the
  intake mouth. Measured: same sweep case gave 0 contact samples with the
  launcher fitted vs 90 (45/45 bilateral) without. Conditional Xacro only — no
  forked geometry, and no deployment mechanism invented for a transition that
  has not been designed.

Datums
  Basket lift travel 450 -> 100 mm (the CAD baseline); 450 mm put the raised rim
  above the LiDAR scan plane. LiDAR: the CAD 498 mm was written as a LOCAL z, so
  base_link_height was added twice AND the sim-only +35 mm gpu_lidar offset was
  overlooked — the scan plane actually sat at 578 mm. Now derived from the
  ground datum, verified live at 0.498 m.

Defects found by running it
  * Nav2 delivers position but not heading (shared goal checker uses
    yaw_goal_tolerance 3.14 so collection lanes do not spin; RPP does no final
    rotation; Spin aborts COLLISION_AHEAD against a costmap measured clear).
    Added a bounded closed-loop heading_aligner; the readiness gate still
    decides, and a failed correction faults rather than arming.
  * Feed requests: 15 events for 3 throws, then losses. The repeat-burst
    publisher suits idempotent setpoints, not discrete events -> single-shot
    reliable publish + de-duplication on throw_id at the consumer.
  * basket_joint froze whenever it REACHED a hard stop under command, not only
    when parked on one. Lower stop moved below the parked position and the mover
    bounded by distance and feedback freshness.
  * SIM_BENCH_MINIMAL dropped sim_clock_relay, leaving controller_manager with
    no clock: every ROS timestamp froze at 0 while physics kept running.
  * `self.position or start` turned the lowered endpoint (0.0) into the start.

Not validated
  Feed events are accepted requests, not launched balls
  (BALL_LAUNCH_PHYSICS_NOT_VALIDATED). Basket tilt stays
  MECHANICAL_VALIDATION_PENDING. Stop-during-session and the throw interval
  (measured 7.9/8.6 s for 4.0 s configured) are still open, so
  ORCHESTRATION_VALIDATED_IN_SIM is NOT claimed. Nothing here says anything
  about physical hardware.

Tests: 762 passed, 2 skipped.

Co-Authored-By: Claude Opus 5 <noreply@anthropic.com>

File: ros2_ws/src/tennis_robot/urdf/components/basket.urdf.xacro (robot description, xacro)
@@ -23,5 +23,5 @@
        base_link's origin (base_link_height above ground). -->
   <xacro:macro name="ball_basket"
-      params="parent floor_front_x floor_top_z_ground rear_x half_width wall_top_z_ground center_lip_height management_run management_rise receiver_run receiver_rise hood_rear_overhang hood_rear_clearance_z_ground hood_front_clearance_z_ground x_shift:=0.0 empty_mass:=0.01 payload_mass:=0.0">
+      params="parent floor_front_x floor_top_z_ground rear_x half_width wall_top_z_ground center_lip_height management_run management_rise receiver_run receiver_rise hood_rear_overhang hood_rear_clearance_z_ground hood_front_clearance_z_ground x_shift:=0.0 lift_travel:=0.100 lift_overtravel:=0.010 empty_mass:=0.01 payload_mass:=0.0">
     <xacro:property name="floor_top" value="${floor_top_z_ground - base_link_height}"/>
     <xacro:property name="wall_top" value="${wall_top_z_ground - base_link_height}"/>
@@ -85,8 +85,28 @@
     <xacro:property name="basket_com_x" value="${(floor_front_x + rear_x) / 2.0}"/>
     <xacro:property name="basket_com_z" value="${floor_top + 0.45 * wall_height}"/>
-    <joint name="basket_joint" type="fixed">
+    <!-- The basket carriage is a real actuator boundary.  Collection/transport
+         uses position 0; Throwing Mode raises the complete basket assembly.
+         The same joint/controller contract is reserved for physical hardware,
+         whose driver and limit switches are intentionally still pending.
+         lift_overtravel moves the modelled LOWER hard stop below the parked
+         position. It is not a mechanical dimension: the commanded travel is
+         still exactly 0...lift_travel. A prismatic joint parked exactly ON its
+         lower limit sits on a permanently active DART limit constraint, and
+         gz-sim then cannot drive it with a velocity command — the joint stays
+         frozen even with hold_joints=false and even under gravity. The upper
+         stop needs no margin: the carriage only touches it briefly and gravity
+         immediately pulls it back inside the range, releasing the constraint.
+         lift_travel is the CAD baseline LIFT ONLY (100 mm). The mechanical
+         launch pose is 100 mm lift PLUS ~12 deg tilt; the tilt mechanism is not
+         mechanically validated, so no tilt joint is modelled and reaching this
+         joint's upper limit is NOT the complete physical throwing pose.
+         See docs/mechanism/flywheel-launcher-exploration-el.md. -->
+    <joint name="basket_joint" type="prismatic">
       <parent link="${parent}"/>
       <child link="basket_link"/>
       <origin xyz="${x_shift} 0 0" rpy="0 0 0"/>
+      <axis xyz="0 0 1"/>
+      <limit lower="${-lift_overtravel}" upper="${lift_travel}" effort="120.0" velocity="0.12"/>
+      <dynamics damping="1.0" friction="0.0"/>
     </joint>
     <link name="basket_link">

File: ros2_ws/src/tennis_robot/urdf/components/ros2_control.urdf.xacro (robot description, xacro)
@@ -19,5 +19,5 @@
   <!-- intake_max_vel = GB37Y3530-12V-251R no-load speed (251 RPM = 26.3 rad/s). -->
   <xacro:macro name="tennis_robot_ros2_control"
-               params="sim_mode:=true controllers_config wheel_max_vel:=20.0 intake_max_vel:=26.3 flywheel_max_vel:=320.0 expose_intake_carriage_state:=false enable_flywheel:=false enable_assist:=false enable_conveyor:=false">
+               params="sim_mode:=true controllers_config wheel_max_vel:=20.0 intake_max_vel:=26.3 flywheel_max_vel:=320.0 basket_lift_travel:=0.100 expose_intake_carriage_state:=false enable_intake:=true enable_flywheel:=false enable_assist:=false enable_conveyor:=false">
     <ros2_control name="TennisRobotSystem" type="system">
       <!-- Hardware backend (the only sim/real difference) -->
@@ -40,5 +40,7 @@
           <param name="right_wheel_names">rear_right_wheel_joint,front_right_wheel_joint</param>
           <!-- Two identical GB37 motors, one driver channel each. -->
-          <param name="intake_wheel_names">intake_wheel_left_joint,intake_wheel_right_joint</param>
+          <xacro:if value="${enable_intake}">
+            <param name="intake_wheel_names">intake_wheel_left_joint,intake_wheel_right_joint</param>
+          </xacro:if>
           <xacro:if value="${enable_flywheel}">
             <param name="flywheel_names">flywheel_left_joint,flywheel_right_joint</param>
@@ -85,17 +87,36 @@
         <state_interface name="velocity"/>
       </joint>
-      <!-- Dual-wheel intake (one motor per wheel, opposite spin) -->
-      <joint name="intake_wheel_left_joint">
-        <command_interface name="velocity">
-          <param name="min">-${intake_max_vel}</param>
-          <param name="max">${intake_max_vel}</param>
-        </command_interface>
-        <state_interface name="position"/>
-        <state_interface name="velocity"/>
-      </joint>
-      <joint name="intake_wheel_right_joint">
-        <command_interface name="velocity">
-          <param name="min">-${intake_max_vel}</param>
-          <param name="max">${intake_max_vel}</param>
+      <!-- Dual-wheel intake (one motor per wheel, opposite spin). Absent in
+           the launch configuration, whose intake assembly is not fitted. -->
+      <xacro:if value="${enable_intake}">
+        <joint name="intake_wheel_left_joint">
+          <command_interface name="velocity">
+            <param name="min">-${intake_max_vel}</param>
+            <param name="max">${intake_max_vel}</param>
+          </command_interface>
+          <state_interface name="position"/>
+          <state_interface name="velocity"/>
+        </joint>
+        <joint name="intake_wheel_right_joint">
+          <command_interface name="velocity">
+            <param name="min">-${intake_max_vel}</param>
+            <param name="max">${intake_max_vel}</param>
+          </command_interface>
+          <state_interface name="position"/>
+          <state_interface name="velocity"/>
+        </joint>
+      </xacro:if>
+      <!-- Basket lift carriage.  The actuator primitive is a rated-speed drive,
+           matching both the Gazebo joint and the future physical carriage; the
+           position target is closed by the supervisor above from the `position`
+           state interface (plus limit switches on real hardware).  gz_ros2_control
+           emulates a `position` command interface with an unsaturated
+           proportional controller, so it would ignore this joint's rated speed.
+           Keep min/max equal to the basket_joint velocity limit in
+           components/basket.urdf.xacro. -->
+      <joint name="basket_joint">
+        <command_interface name="velocity">
+          <param name="min">-0.12</param>
+          <param name="max">0.12</param>
         </command_interface>
         <state_interface name="position"/>
@@ -126,5 +147,5 @@
            interfaces must not become part of the real hardware contract. -->
       <xacro:if value="${sim_mode}">
-        <xacro:if value="${expose_intake_carriage_state}">
+        <xacro:if value="${enable_intake and expose_intake_carriage_state}">
           <joint name="intake_wheel_left_carriage_joint">
             <state_interface name="position"/>

File: ros2_ws/src/tennis_robot/urdf/tennis_robot.urdf.xacro (robot description, xacro)
@@ -29,8 +29,16 @@
   <xacro:arg name="battery_center_x" default="-0.143"/>
   <xacro:arg name="enable_compact_electronics" default="false"/>
+  <!-- Mechanical operating configuration. The physical concept has separate
+       COLLECT and LAUNCH configurations; the intake assembly and the flywheel
+       launcher claim the same front volume and are never fitted together.
+       Selected through the packaging variant, see scripts/generate_robot_urdf.py. -->
+  <xacro:arg name="enable_intake" default="true"/>
   <xacro:arg name="enable_flywheel" default="false"/>
   <xacro:arg name="flywheel_max_vel" default="320.0"/>
+  <xacro:arg name="flywheel_nip_gap" default="0.058"/>
   <xacro:arg name="basket_empty_mass" default="0.01"/>
   <xacro:arg name="basket_payload_mass" default="0.0"/>
+  <xacro:arg name="basket_lift_travel" default="0.100"/>
+  <xacro:arg name="basket_lift_overtravel" default="0.010"/>
   <!-- Dual-wheel intake tuning (docs/dual-wheel-intake-design-el.md).
        Injected from INTAKE_WHEEL_* envs by scripts/generate_robot_urdf.py. -->
@@ -125,5 +133,15 @@
   <xacro:property name="intake_conveyor_length" value="0.200"/>
   <xacro:property name="scooper_pitch" value="0.1745"/>  <!-- 10 degrees; funnel-cheek tilt -->
-  <xacro:property name="lidar_xyz" value="-0.42 0 0.498"/>
+  <!-- LiDAR height datum. The CAD/mechanical source of truth is the SCAN PLANE
+       at 498 mm above ground, NOT the link origin: the gpu_lidar sensor sits
+       lidar_sensor_scan_offset above lidar_link (see components/lidar.urdf.xacro),
+       and lidar_link itself sits base_link_height above ground. Deriving the
+       mount height keeps all three terms in one place — hardcoding 0.498 here
+       silently placed the scan plane at 0.578 m. -->
+  <xacro:property name="lidar_scan_plane_z_ground" value="0.498"/>
+  <xacro:property name="lidar_sensor_scan_offset" value="0.035"/>
+  <xacro:property name="lidar_mount_z"
+      value="${lidar_scan_plane_z_ground - base_link_height - lidar_sensor_scan_offset}"/>
+  <xacro:property name="lidar_xyz" value="-0.42 0 ${lidar_mount_z}"/>
   <xacro:property name="lidar_rpy" value="0 0 0"/>  <!-- level chassis: horizontal scan plane -->
   <xacro:property name="camera_xyz" value="${0.535 + functional_shift_x} 0 0.443"/>
@@ -212,36 +230,45 @@
       width="${wheel_width}"
       mass="${wheel_mass}"/>
-  <!-- Left wheel drives ω<0 / right ω>0 (opposite signs, commanded by
-       intake_wheel_velocity_controller) so both inner faces move rearward. -->
-  <xacro:intake_side_wheel
-      side="left"
-      y="${intake_wheel_y}"
-      nip_x="${intake_nip_x}"
-      wheel_z="${intake_wheel_z}"
-      tilt_rad="${intake_wheel_tilt_rad}"
-      radius="${intake_wheel_radius}"
-      height="${intake_wheel_height}"
-      carriage_travel="${intake_carriage_travel}"
-      max_vel="${intake_wheel_max_vel}"
-      effort="${intake_wheel_effort}"
-      mass="0.20"
-      sensor_index="0"/>
-  <xacro:intake_side_wheel
-      side="right"
-      y="${-intake_wheel_y}"
-      nip_x="${intake_nip_x}"
-      wheel_z="${intake_wheel_z}"
-      tilt_rad="${intake_wheel_tilt_rad}"
-      radius="${intake_wheel_radius}"
-      height="${intake_wheel_height}"
-      carriage_travel="${intake_carriage_travel}"
-      max_vel="${intake_wheel_max_vel}"
-      effort="${intake_wheel_effort}"
-      mass="0.20"
-      sensor_index="1"/>
-  <xacro:intake_funnel parent="base_link" chassis_z="${chassis_z}" pitch="${scooper_pitch}"
-      x_shift="${functional_shift_x}"
-      cheek_x_bias="${intake_cad_alignment_x}"
-      enable_cheeks="$(arg enable_funnel)" enable_ramp="$(arg enable_ramp)"/>
+  <!-- INTAKE ASSEMBLY — fitted only in the COLLECT configuration.
+       Its wheels, funnel cheeks, elevation ramp and safety deflector occupy
+       x 446…884 mm / z 0…281 mm, the same volume the flywheel launcher needs
+       (wheels x 459…661, z 162…268). The two are alternative mechanical
+       configurations of one robot, so the launch configuration simply does not
+       carry this assembly — no deployment mechanism is modelled, because none
+       has been selected yet. -->
+  <xacro:if value="$(arg enable_intake)">
+    <!-- Left wheel drives ω<0 / right ω>0 (opposite signs, commanded by
+         intake_wheel_velocity_controller) so both inner faces move rearward. -->
+    <xacro:intake_side_wheel
+        side="left"
+        y="${intake_wheel_y}"
+        nip_x="${intake_nip_x}"
+        wheel_z="${intake_wheel_z}"
+        tilt_rad="${intake_wheel_tilt_rad}"
+        radius="${intake_wheel_radius}"
+        height="${intake_wheel_height}"
+        carriage_travel="${intake_carriage_travel}"
+        max_vel="${intake_wheel_max_vel}"
+        effort="${intake_wheel_effort}"
+        mass="0.20"
+        sensor_index="0"/>
+    <xacro:intake_side_wheel
+        side="right"
+        y="${-intake_wheel_y}"
+        nip_x="${intake_nip_x}"
+        wheel_z="${intake_wheel_z}"
+        tilt_rad="${intake_wheel_tilt_rad}"
+        radius="${intake_wheel_radius}"
+        height="${intake_wheel_height}"
+        carriage_travel="${intake_carriage_travel}"
+        max_vel="${intake_wheel_max_vel}"
+        effort="${intake_wheel_effort}"
+        mass="0.20"
+        sensor_index="1"/>
+    <xacro:intake_funnel parent="base_link" chassis_z="${chassis_z}" pitch="${scooper_pitch}"
+        x_shift="${functional_shift_x}"
+        cheek_x_bias="${intake_cad_alignment_x}"
+        enable_cheeks="$(arg enable_funnel)" enable_ramp="$(arg enable_ramp)"/>
+  </xacro:if>
   <xacro:if value="$(arg enable_assist)">
     <xacro:intake_assist_roller
@@ -295,4 +322,6 @@
       hood_front_clearance_z_ground="${float($(arg basket_hood_front_clearance_z))}"
       x_shift="${functional_shift_x}"
+      lift_travel="${float($(arg basket_lift_travel))}"
+      lift_overtravel="${float($(arg basket_lift_overtravel))}"
       empty_mass="${float($(arg basket_empty_mass))}"
       payload_mass="${float($(arg basket_payload_mass))}"/>
@@ -310,4 +339,5 @@
         base_link_height="${base_link_height}"
         pitch_rad="0.349066"
+        nip_gap="${float($(arg flywheel_nip_gap))}"
         max_vel="${float($(arg flywheel_max_vel))}"/>
   </xacro:if>
@@ -317,4 +347,6 @@
       xyz="${lidar_xyz}"
       rpy="${lidar_rpy}"
+      mount_z="${lidar_mount_z}"
+      scan_offset_z="${lidar_sensor_scan_offset}"
       update_rate="${sensor_update_rate}"/>
   <xacro:oak_d_lite_mount
@@ -379,6 +411,8 @@
       expose_intake_carriage_state="$(arg expose_intake_carriage_state)"
       intake_max_vel="${intake_wheel_max_vel}"
+      enable_intake="$(arg enable_intake)"
       enable_flywheel="$(arg enable_flywheel)"
       flywheel_max_vel="${float($(arg flywheel_max_vel))}"
+      basket_lift_travel="${float($(arg basket_lift_travel))}"
       enable_assist="$(arg enable_assist)"
       enable_conveyor="$(arg enable_conveyor)"/>
