Commit message: Refine collection route behavior and delivery docs

File: ros2_ws/src/tennis_robot/urdf/components/basket.urdf.xacro (robot description, xacro)
@@ -63,5 +63,8 @@
     <xacro:property name="receiver_centre_z" value="${receiver_top_mid_z - cos(receiver_pitch) * floor_thickness / 2.0}"/>
     <xacro:property name="receiver_half_width" value="${entry_half_width}"/>
-    <xacro:property name="confirmation_beam_z" value="${receiver_top_mid_z + 0.033}"/>
+    <xacro:property name="confirmation_beam_x" value="${management_top_mid_x}"/>
+    <!-- Matches basket_ir_z in tennis_robot.urdf.xacro: above court-ball top
+         (0.066) so the beam cannot see ground balls through the mesh. -->
+    <xacro:property name="confirmation_beam_z" value="${management_top_mid_z + 0.045}"/>
     <!-- Optional mesh entry tunnel. Its roof rises toward the wheels, so balls
          from upper basket layers roll rearward instead of spilling into the
@@ -250,10 +253,10 @@
         </visual>
       </xacro:if>
-      <xacro:if value="${receiver_run > 0.0}">
+      <xacro:if value="${management_run > 0.0}">
         <!-- Sensor bodies remain on the chassis. This line only visualises the
              transverse confirmation beam through the removable mesh. -->
         <visual name="basket_ir_beam_line_vis">
-          <origin xyz="${receiver_top_mid_x} 0 ${confirmation_beam_z}" rpy="1.5708 0 0"/>
-          <geometry><cylinder radius="0.003" length="${2.0 * receiver_half_width + 0.03}"/></geometry>
+          <origin xyz="${confirmation_beam_x} 0 ${confirmation_beam_z}" rpy="1.5708 0 0"/>
+          <geometry><cylinder radius="0.003" length="${2.0 * half_width + 0.03}"/></geometry>
           <material name="ir_beam_red"/>
         </visual>

File: ros2_ws/src/tennis_robot/urdf/components/funnel.urdf.xacro (robot description, xacro)
@@ -19,31 +19,33 @@
       </inertial>
       <xacro:if value="${enable_cheeks}">
-        <!-- Cheeks guide the ball INTO the wheel nip, not just near it
-             (intake debug-log #59): front tips unchanged at ~(0.876, ±0.205)
-             (mouth 410 mm), rear tips pulled in to ~(0.680, ±0.104) so the
-             exit corridor caps the ball centre at |y| ≤ ~0.066 — inside the
-             bench-validated ±0.08 envelope. The old rear tips at ±0.146 let
-             the ball exit at |y| ≤ 0.108 and meet the wheel's OUTER front
-             quadrant (surface sweeping outward), deflecting it sideways
-             (collection-route-debug-log-el #3). Rear tips clear the wheel
-             centres (0.590, ±0.090) by 91 mm — rule is ≥65 mm (cylinder
-             r=0.060 + carriage travel). -->
+        <!-- Cheeks guide the ball INTO the wheel nip, not just near it.
+             Iteration 2 (sweep-mode observation: exit corridor still let the
+             ball wander before the wheels): front tips unchanged at
+             ~(0.876, ±0.205) (mouth 410 mm), rear tips pulled in AND closer
+             to the wheels — (0.680, ±0.104) → (0.655, ±0.083) — so the exit
+             caps the ball centre at |y| ≤ ~0.045: ball SURFACE stays ≤0.078,
+             inside the wheel centreline (±0.090), touching only the INNER
+             front quadrant which sweeps it into the nip. The old cap (0.066)
+             let the surface reach 0.099 > 0.090 — outer-quadrant contact
+             deflected balls sideways. Rear tips clear the wheel centres
+             (0.590, ±0.090) by 65.4 mm — rule is ≥65 mm (cylinder r=0.060
+             + carriage travel). -->
         <visual name="funnel_left_cheek_vis">
-          <origin xyz="0.778 0.1545 0.052" rpy="0 ${pitch} 0.476"/>
-          <geometry><box size="0.2205 0.01 0.10"/></geometry>
+          <origin xyz="0.7655 0.144 0.052" rpy="0 ${pitch} 0.504"/>
+          <geometry><box size="0.2524 0.01 0.10"/></geometry>
           <material name="intake_orange"/>
         </visual>
         <collision name="funnel_left_cheek_col">
-          <origin xyz="0.778 0.1545 0.052" rpy="0 ${pitch} 0.476"/>
-          <geometry><box size="0.2205 0.01 0.10"/></geometry>
+          <origin xyz="0.7655 0.144 0.052" rpy="0 ${pitch} 0.504"/>
+          <geometry><box size="0.2524 0.01 0.10"/></geometry>
         </collision>
         <visual name="funnel_right_cheek_vis">
-          <origin xyz="0.778 -0.1545 0.052" rpy="0 ${pitch} -0.476"/>
-          <geometry><box size="0.2205 0.01 0.10"/></geometry>
+          <origin xyz="0.7655 -0.144 0.052" rpy="0 ${pitch} -0.504"/>
+          <geometry><box size="0.2524 0.01 0.10"/></geometry>
           <material name="intake_orange"/>
         </visual>
         <collision name="funnel_right_cheek_col">
-          <origin xyz="0.778 -0.1545 0.052" rpy="0 ${pitch} -0.476"/>
-          <geometry><box size="0.2205 0.01 0.10"/></geometry>
+          <origin xyz="0.7655 -0.144 0.052" rpy="0 ${pitch} -0.504"/>
+          <geometry><box size="0.2524 0.01 0.10"/></geometry>
         </collision>
       </xacro:if>

File: ros2_ws/src/tennis_robot/urdf/tennis_robot.urdf.xacro (robot description, xacro)
@@ -134,9 +134,14 @@
   <xacro:property name="ir_y" value="0.105"/>
   <xacro:property name="ir_z" value="-0.005"/>
-  <!-- Basket confirmation beam crosses the midpoint of the inclined receiver
-       at the rolling ball's equator. Sensor coordinates are base_link-frame. -->
-  <xacro:property name="basket_ir_x" value="${float($(arg basket_floor_front_x)) + float($(arg basket_receiver_run)) / 2.0}"/>
+  <!-- Basket confirmation beam is behind the retention lip, halfway down the
+       internal management tray. A ball on the external receiver is not yet
+       collected and must keep the intake running until it crosses this beam. -->
+  <xacro:property name="basket_ir_x" value="${float($(arg basket_floor_front_x)) - float($(arg basket_management_run)) / 2.0}"/>
   <xacro:property name="basket_ir_y" value="0.105"/>
-  <xacro:property name="basket_ir_z" value="${float($(arg basket_floor_top_z)) + float($(arg basket_management_rise)) + float($(arg basket_receiver_rise)) / 2.0 + 0.033 - base_link_height}"/>
+  <!-- Beam height 0.075 above court: ABOVE a court ball's top (0.066) so the
+       ray cannot clip balls standing beside the robot through the open wire
+       mesh (run 11: 4 false credits, one-sided ir hits 2-11 cm from one
+       sensor), yet still well below a tray-rolling ball's top (0.096). -->
+  <xacro:property name="basket_ir_z" value="${float($(arg basket_floor_top_z)) + float($(arg basket_management_rise)) / 2.0 + 0.045 - base_link_height}"/>
   <xacro:property name="max_linear_acceleration" value="2.0"/>
   <xacro:property name="max_angular_acceleration" value="4.0"/>

Commit message: feat: add compact flywheel Gazebo packaging

File: ros2_ws/src/tennis_robot/urdf/components/basket.urdf.xacro (robot description, xacro)
@@ -23,5 +23,5 @@
        base_link's origin (base_link_height above ground). -->
   <xacro:macro name="ball_basket"
-      params="parent floor_front_x floor_top_z_ground rear_x half_width wall_top_z_ground center_lip_height management_run management_rise receiver_run receiver_rise hood_rear_overhang hood_rear_clearance_z_ground hood_front_clearance_z_ground">
+      params="parent floor_front_x floor_top_z_ground rear_x half_width wall_top_z_ground center_lip_height management_run management_rise receiver_run receiver_rise hood_rear_overhang hood_rear_clearance_z_ground hood_front_clearance_z_ground x_shift:=0.0 empty_mass:=0.01 payload_mass:=0.0">
     <xacro:property name="floor_top" value="${floor_top_z_ground - base_link_height}"/>
     <xacro:property name="wall_top" value="${wall_top_z_ground - base_link_height}"/>
@@ -82,13 +82,22 @@
     <xacro:property name="hood_side_mid_z" value="${(receiver_top_mid_z + hood_side_top_z) / 2.0}"/>
     <xacro:property name="hood_side_height" value="${hood_side_top_z - receiver_top_mid_z}"/>
+    <xacro:property name="basket_mass" value="${empty_mass + payload_mass}"/>
+    <xacro:property name="basket_com_x" value="${(floor_front_x + rear_x) / 2.0}"/>
+    <xacro:property name="basket_com_z" value="${floor_top + 0.45 * wall_height}"/>
     <joint name="basket_joint" type="fixed">
       <parent link="${parent}"/>
       <child link="basket_link"/>
-      <origin xyz="0 0 0" rpy="0 0 0"/>
+      <origin xyz="${x_shift} 0 0" rpy="0 0 0"/>
     </joint>
     <link name="basket_link">
       <inertial>
-        <mass value="0.01"/>
-        <inertia ixx="0.0001" ixy="0" ixz="0" iyy="0.0001" iyz="0" izz="0.0001"/>
+        <origin xyz="${basket_com_x} 0 ${basket_com_z}" rpy="0 0 0"/>
+        <mass value="${basket_mass}"/>
+        <inertia
+            ixx="${basket_mass * ((2.0 * half_width) * (2.0 * half_width) + wall_height * wall_height) / 12.0}"
+            ixy="0" ixz="0"
+            iyy="${basket_mass * (bin_length * bin_length + wall_height * wall_height) / 12.0}"
+            iyz="0"
+            izz="${basket_mass * (bin_length * bin_length + (2.0 * half_width) * (2.0 * half_width)) / 12.0}"/>
       </inertial>
       <collision name="basket_floor_col">

File: ros2_ws/src/tennis_robot/urdf/components/funnel.urdf.xacro (robot description, xacro)
@@ -7,9 +7,9 @@
        enable_cheeks / enable_ramp implement the Concept Validation Plan
        gates (Phase 1 = throat only runs with both disabled). -->
-  <xacro:macro name="intake_funnel" params="parent chassis_z pitch enable_cheeks:=true enable_ramp:=true">
+  <xacro:macro name="intake_funnel" params="parent chassis_z pitch x_shift:=0.0 cheek_x_bias:=0.0 enable_cheeks:=true enable_ramp:=true">
     <joint name="funnel_joint" type="fixed">
       <parent link="${parent}"/>
       <child link="funnel_link"/>
-      <origin xyz="0 0 ${-chassis_z / 2}" rpy="0 0 0"/>
+      <origin xyz="${x_shift} 0 ${-chassis_z / 2}" rpy="0 0 0"/>
     </joint>
     <link name="funnel_link">
@@ -32,19 +32,19 @@
              + carriage travel). -->
         <visual name="funnel_left_cheek_vis">
-          <origin xyz="0.7655 0.144 0.052" rpy="0 ${pitch} 0.504"/>
+          <origin xyz="${0.7655 + cheek_x_bias} 0.144 0.052" rpy="0 ${pitch} 0.504"/>
           <geometry><box size="0.2524 0.01 0.10"/></geometry>
           <material name="intake_orange"/>
         </visual>
         <collision name="funnel_left_cheek_col">
-          <origin xyz="0.7655 0.144 0.052" rpy="0 ${pitch} 0.504"/>
+          <origin xyz="${0.7655 + cheek_x_bias} 0.144 0.052" rpy="0 ${pitch} 0.504"/>
           <geometry><box size="0.2524 0.01 0.10"/></geometry>
         </collision>
         <visual name="funnel_right_cheek_vis">
-          <origin xyz="0.7655 -0.144 0.052" rpy="0 ${pitch} -0.504"/>
+          <origin xyz="${0.7655 + cheek_x_bias} -0.144 0.052" rpy="0 ${pitch} -0.504"/>
           <geometry><box size="0.2524 0.01 0.10"/></geometry>
           <material name="intake_orange"/>
         </visual>
         <collision name="funnel_right_cheek_col">
-          <origin xyz="0.7655 -0.144 0.052" rpy="0 ${pitch} -0.504"/>
+          <origin xyz="${0.7655 + cheek_x_bias} -0.144 0.052" rpy="0 ${pitch} -0.504"/>
           <geometry><box size="0.2524 0.01 0.10"/></geometry>
         </collision>

File: ros2_ws/src/tennis_robot/urdf/components/ros2_control.urdf.xacro (robot description, xacro)
@@ -14,9 +14,10 @@
     intake_assist_wheel_joint -> optional second-stage ramp assist roller
     intake_conveyor_*_joint -> optional Phase 3B ramp conveyor approximation
+	  flywheel_left_joint / flywheel_right_joint -> optional launcher wheels
 	-->
 <robot xmlns:xacro="http://www.ros.org/wiki/xacro">
   <!-- intake_max_vel = GB37Y3530-12V-251R no-load speed (251 RPM = 26.3 rad/s). -->
   <xacro:macro name="tennis_robot_ros2_control"
-               params="sim_mode:=true controllers_config wheel_max_vel:=20.0 intake_max_vel:=26.3 expose_intake_carriage_state:=false enable_assist:=false enable_conveyor:=false">
+               params="sim_mode:=true controllers_config wheel_max_vel:=20.0 intake_max_vel:=26.3 flywheel_max_vel:=320.0 expose_intake_carriage_state:=false enable_flywheel:=false enable_assist:=false enable_conveyor:=false">
     <ros2_control name="TennisRobotSystem" type="system">
       <!-- Hardware backend (the only sim/real difference) -->
@@ -40,4 +41,7 @@
           <!-- Two identical GB37 motors, one driver channel each. -->
           <param name="intake_wheel_names">intake_wheel_left_joint,intake_wheel_right_joint</param>
+          <xacro:if value="${enable_flywheel}">
+            <param name="flywheel_names">flywheel_left_joint,flywheel_right_joint</param>
+          </xacro:if>
           <xacro:if value="${enable_assist}">
             <param name="assist_wheel_names">intake_assist_wheel_joint</param>
@@ -98,4 +102,24 @@
         <state_interface name="velocity"/>
       </joint>
+      <!-- Optional two-motor side-by-side launcher. Opposite commands make
+           both inner wheel faces drive the ball forward (+X). -->
+      <xacro:if value="${enable_flywheel}">
+        <joint name="flywheel_left_joint">
+          <command_interface name="velocity">
+            <param name="min">-${flywheel_max_vel}</param>
+            <param name="max">${flywheel_max_vel}</param>
+          </command_interface>
+          <state_interface name="position"/>
+          <state_interface name="velocity"/>
+        </joint>
+        <joint name="flywheel_right_joint">
+          <command_interface name="velocity">
+            <param name="min">-${flywheel_max_vel}</param>
+            <param name="max">${flywheel_max_vel}</param>
+          </command_interface>
+          <state_interface name="position"/>
+          <state_interface name="velocity"/>
+        </joint>
+      </xacro:if>
       <!-- Gazebo-only observability for the passive spring carriages. The
            physical prototype has no carriage encoder, so these state-only

File: ros2_ws/src/tennis_robot/urdf/tennis_robot.urdf.xacro (robot description, xacro)
@@ -14,4 +14,6 @@
   <xacro:include filename="components/body_panels.urdf.xacro"/>
   <xacro:include filename="components/intake_debug_camera.urdf.xacro"/>
+  <xacro:include filename="components/electronics_packaging.urdf.xacro"/>
+  <xacro:include filename="components/flywheel_launcher.urdf.xacro"/>
   <!-- ros2_control args. sim_mode swaps the hardware backend (sim vs real).
        controllers_config is the absolute path to controllers.yaml, injected by
@@ -20,4 +22,15 @@
   <xacro:arg name="controllers_config" default="config/controllers.yaml"/>
   <xacro:arg name="expose_intake_carriage_state" default="false"/>
+  <!-- Selectable packaging overlay. Baseline remains the frozen collection
+       model; compact shifts the complete functional chain by -100 mm and
+       enables the new mass-bearing components through the generator. -->
+  <xacro:arg name="functional_shift_x" default="0.0"/>
+  <xacro:arg name="intake_cad_alignment_x" default="0.0"/>
+  <xacro:arg name="battery_center_x" default="-0.143"/>
+  <xacro:arg name="enable_compact_electronics" default="false"/>
+  <xacro:arg name="enable_flywheel" default="false"/>
+  <xacro:arg name="flywheel_max_vel" default="320.0"/>
+  <xacro:arg name="basket_empty_mass" default="0.01"/>
+  <xacro:arg name="basket_payload_mass" default="0.0"/>
   <!-- Dual-wheel intake tuning (docs/dual-wheel-intake-design-el.md).
        Injected from INTAKE_WHEEL_* envs by scripts/generate_robot_urdf.py. -->
@@ -62,4 +75,6 @@
        ground, below the 85 mm motor-shaft/wheel-axle centreline. -->
   <xacro:property name="base_link_height" value="0.045"/>
+  <xacro:property name="functional_shift_x" value="${float($(arg functional_shift_x))}"/>
+  <xacro:property name="intake_cad_alignment_x" value="${float($(arg intake_cad_alignment_x))}"/>
   <!-- 4WD skid-steer drivetrain. Four identical 170 mm (radius 0.085) driven
        wheels (HPI Dirt Buster Block, 170x80 mm, Baja 5B), two per side, placed
@@ -84,5 +99,5 @@
   <xacro:property name="intake_wheel_radius" value="${float($(arg intake_wheel_radius))}"/>
   <xacro:property name="intake_wheel_gap" value="${float($(arg intake_wheel_gap))}"/>
-  <xacro:property name="intake_nip_x" value="${float($(arg intake_nip_x))}"/>
+  <xacro:property name="intake_nip_x" value="${float($(arg intake_nip_x)) + functional_shift_x + intake_cad_alignment_x}"/>
   <xacro:property name="intake_wheel_tilt_rad" value="${float($(arg intake_wheel_tilt_deg)) * 0.017453292519943295}"/>
   <xacro:property name="intake_wheel_max_vel" value="${float($(arg intake_wheel_max_vel))}"/>
@@ -112,5 +127,5 @@
   <xacro:property name="lidar_xyz" value="-0.42 0 0.498"/>
   <xacro:property name="lidar_rpy" value="0 0 0"/>  <!-- level chassis: horizontal scan plane -->
-  <xacro:property name="camera_xyz" value="0.535 0 0.443"/>
+  <xacro:property name="camera_xyz" value="${0.535 + functional_shift_x} 0 0.443"/>
   <xacro:property name="camera_rpy" value="0 0.273 0"/>  <!-- forward-down tilt ~15.6deg; preserves the old world aim (0.22 cam + 0.053 chassis pitch) now that the chassis is level -->
   <xacro:property name="sensor_update_rate" value="31.25"/>
@@ -122,5 +137,5 @@
        them, and the ball as it enters the nip. The old side mount
        (0.5, 0.13) is now inside the left wheel's swept volume. -->
-  <xacro:property name="intake_debug_camera_xyz" value="0.78 0 0.06"/>
+  <xacro:property name="intake_debug_camera_xyz" value="${0.78 + functional_shift_x} 0 0.06"/>
   <xacro:property name="intake_debug_camera_rpy" value="0 0.339 3.14159"/>
   <!-- Throat beam crosses the corridor at ball-centre height (40 mm above
@@ -131,5 +146,5 @@
        or maintain the rollers. Collection confirmation is the BASKET beam
        pair below — see gazebo_extras_node.py. -->
-  <xacro:property name="ir_x" value="0.720"/>
+  <xacro:property name="ir_x" value="${0.720 + functional_shift_x}"/>
   <xacro:property name="ir_y" value="0.105"/>
   <xacro:property name="ir_z" value="-0.005"/>
@@ -137,5 +152,5 @@
        internal management tray. A ball on the external receiver is not yet
        collected and must keep the intake running until it crosses this beam. -->
-  <xacro:property name="basket_ir_x" value="${float($(arg basket_floor_front_x)) - float($(arg basket_management_run)) / 2.0}"/>
+  <xacro:property name="basket_ir_x" value="${float($(arg basket_floor_front_x)) - float($(arg basket_management_run)) / 2.0 + functional_shift_x}"/>
   <xacro:property name="basket_ir_y" value="0.105"/>
   <!-- Beam height 0.075 above court: ABOVE a court ball's top (0.066) so the
@@ -226,9 +241,11 @@
       sensor_index="1"/>
   <xacro:intake_funnel parent="base_link" chassis_z="${chassis_z}" pitch="${scooper_pitch}"
+      x_shift="${functional_shift_x}"
+      cheek_x_bias="${intake_cad_alignment_x}"
       enable_cheeks="$(arg enable_funnel)" enable_ramp="$(arg enable_ramp)"/>
   <xacro:if value="$(arg enable_assist)">
     <xacro:intake_assist_roller
         parent="base_link"
-        x="${intake_assist_x}"
+        x="${intake_assist_x + functional_shift_x}"
         z="${intake_assist_z}"
         radius="${intake_assist_radius}"
@@ -240,5 +257,5 @@
         name="intake_conveyor_front"
         parent="base_link"
-        x="${0.525 + intake_conveyor_x_bias}"
+        x="${0.525 + intake_conveyor_x_bias + functional_shift_x}"
         z="${0.051 + intake_conveyor_z_bias}"
         radius="${intake_conveyor_radius}"
@@ -248,5 +265,5 @@
         name="intake_conveyor_mid"
         parent="base_link"
-        x="${0.490 + intake_conveyor_x_bias}"
+        x="${0.490 + intake_conveyor_x_bias + functional_shift_x}"
         z="${0.067 + intake_conveyor_z_bias}"
         radius="${intake_conveyor_radius}"
@@ -256,5 +273,5 @@
         name="intake_conveyor_rear"
         parent="base_link"
-        x="${0.455 + intake_conveyor_x_bias}"
+        x="${0.455 + intake_conveyor_x_bias + functional_shift_x}"
         z="${0.101 + intake_conveyor_z_bias}"
         radius="${intake_conveyor_radius}"
@@ -276,6 +293,23 @@
       hood_rear_overhang="${float($(arg basket_hood_rear_overhang))}"
       hood_rear_clearance_z_ground="${float($(arg basket_hood_rear_clearance_z))}"
-      hood_front_clearance_z_ground="${float($(arg basket_hood_front_clearance_z))}"/>
-  <xacro:battery_pack parent="base_link"/>
+      hood_front_clearance_z_ground="${float($(arg basket_hood_front_clearance_z))}"
+      x_shift="${functional_shift_x}"
+      empty_mass="${float($(arg basket_empty_mass))}"
+      payload_mass="${float($(arg basket_payload_mass))}"/>
+  <xacro:battery_pack parent="base_link"
+      center_x="${float($(arg battery_center_x))}"/>
+  <xacro:if value="$(arg enable_compact_electronics)">
+    <xacro:compact_electronics_packaging
+        parent="base_link" base_link_height="${base_link_height}"/>
+  </xacro:if>
+  <xacro:if value="$(arg enable_flywheel)">
+    <xacro:side_by_side_flywheel_launcher
+        parent="base_link"
+        origin_x="${0.560 + functional_shift_x}"
+        nip_z_ground="0.215"
+        base_link_height="${base_link_height}"
+        pitch_rad="0.349066"
+        max_vel="${float($(arg flywheel_max_vel))}"/>
+  </xacro:if>
   <xacro:rplidar_c1_mount
       parent="base_link"
@@ -345,4 +379,6 @@
       expose_intake_carriage_state="$(arg expose_intake_carriage_state)"
       intake_max_vel="${intake_wheel_max_vel}"
+      enable_flywheel="$(arg enable_flywheel)"
+      flywheel_max_vel="${float($(arg flywheel_max_vel))}"
       enable_assist="$(arg enable_assist)"
       enable_conveyor="$(arg enable_conveyor)"/>
