Commit message: feat: rebuild and validate compact mechanical package

File: ros2_ws/src/tennis_robot/urdf/components/basket.urdf.xacro (robot description, xacro)
@@ -23,10 +23,9 @@
        base_link's origin (base_link_height above ground). -->
   <xacro:macro name="ball_basket"
-      params="parent floor_front_x floor_top_z_ground rear_x half_width wall_top_z_ground center_lip_height management_run management_rise receiver_run receiver_rise hood_rear_overhang hood_rear_clearance_z_ground hood_front_clearance_z_ground x_shift:=0.0 lift_travel:=0.100 lift_overtravel:=0.010 empty_mass:=0.01 payload_mass:=0.0">
+      params="parent floor_front_x floor_top_z_ground rear_x half_width wall_top_z_ground center_lip_height management_run management_rise receiver_run receiver_rise hood_rear_overhang hood_rear_clearance_z_ground hood_front_clearance_z_ground x_shift:=0.0 lift_travel:=0.100 lift_overtravel:=0.010 empty_mass:=0.01 payload_mass:=0.0 launch_tilt_rad:=0.0 launch_pivot_x:=0.470 launch_pivot_z_ground:=0.040 floor_thickness:=0.005 cad_support_details:=false">
     <xacro:property name="floor_top" value="${floor_top_z_ground - base_link_height}"/>
     <xacro:property name="wall_top" value="${wall_top_z_ground - base_link_height}"/>
     <!-- Thin skinned bin: 5 mm floor (exterior bottom = floor_top - 0.005,
          the robot's lowest point), 10 mm wall frames. -->
-    <xacro:property name="floor_thickness" value="0.005"/>
     <xacro:property name="wall_thickness" value="0.010"/>
     <xacro:property name="bin_length" value="${floor_front_x - rear_x}"/>
@@ -83,6 +82,6 @@
     <xacro:property name="hood_side_height" value="${hood_side_top_z - receiver_top_mid_z}"/>
     <xacro:property name="basket_mass" value="${empty_mass + payload_mass}"/>
-    <xacro:property name="basket_com_x" value="${(floor_front_x + rear_x) / 2.0}"/>
-    <xacro:property name="basket_com_z" value="${floor_top + 0.45 * wall_height}"/>
+    <xacro:property name="basket_com_x" value="${0.209460 if cad_support_details else (floor_front_x + rear_x) / 2.0}"/>
+    <xacro:property name="basket_com_z" value="${0.091481 - base_link_height if cad_support_details else floor_top + 0.45 * wall_height}"/>
     <!-- The basket carriage is a real actuator boundary.  Collection/transport
          uses position 0; Throwing Mode raises the complete basket assembly.
@@ -97,16 +96,28 @@
          stop needs no margin: the carriage only touches it briefly and gravity
          immediately pulls it back inside the range, releasing the constraint.
-         lift_travel is the CAD baseline LIFT ONLY (100 mm). The mechanical
-         launch pose is 100 mm lift PLUS ~12 deg tilt; the tilt mechanism is not
-         mechanically validated, so no tilt joint is modelled and reaching this
-         joint's upper limit is NOT the complete physical throwing pose.
-         See docs/mechanism/flywheel-launcher-exploration-el.md. -->
+         lift_travel is the CAD baseline LIFT ONLY (100 mm).  The compact CAD
+         additionally defines a 12 degree mechanical pose about [470,0,40] mm.
+         It is represented by the fixed basket_launch_pose_joint below: a
+         generated configuration, not an invented or controlled actuator. -->
     <joint name="basket_joint" type="prismatic">
       <parent link="${parent}"/>
-      <child link="basket_link"/>
+      <child link="basket_guide_path_link"/>
       <origin xyz="${x_shift} 0 0" rpy="0 0 0"/>
       <axis xyz="0 0 1"/>
       <limit lower="${-lift_overtravel}" upper="${lift_travel}" effort="120.0" velocity="0.12"/>
       <dynamics damping="1.0" friction="0.0"/>
+    </joint>
+    <!-- Kinematic guide-path frame only. It has no fictitious cage geometry or
+         independent mass; the fixed basket child is reduced onto this frame by
+         SDF, leaving basket_joint as the single physical moving coordinate. -->
+    <link name="basket_guide_path_link"/>
+    <joint name="basket_launch_pose_joint" type="fixed">
+      <parent link="basket_guide_path_link"/>
+      <child link="basket_link"/>
+      <!-- T(pivot) * R_y(tilt) * T(-pivot), collapsed into one URDF origin
+           so the entire basket rotates about the CAD pivot without a massless
+           intermediary physical link. -->
+      <origin xyz="${launch_pivot_x - (cos(launch_tilt_rad) * launch_pivot_x + sin(launch_tilt_rad) * (launch_pivot_z_ground - base_link_height))} 0 ${launch_pivot_z_ground - base_link_height - (-sin(launch_tilt_rad) * launch_pivot_x + cos(launch_tilt_rad) * (launch_pivot_z_ground - base_link_height))}"
+              rpy="0 ${launch_tilt_rad} 0"/>
     </joint>
     <link name="basket_link">
@@ -121,4 +132,19 @@
             izz="${basket_mass * (bin_length * bin_length + (2.0 * half_width) * (2.0 * half_width)) / 12.0}"/>
       </inertial>
+      <xacro:if value="${cad_support_details}">
+        <!-- Generated directly from compact_relieved_bin(); this preserves
+             the two 128 x 77 mm tyre pockets and lower chassis relief in both
+             collision and visual geometry.  OpenSCAD STL units are mm. -->
+        <collision name="compact_relieved_bin_col">
+          <origin xyz="0 0 ${-base_link_height}" rpy="0 0 0"/>
+          <geometry><mesh filename="package://tennis_robot/meshes/compact_relieved_bin.stl" scale="0.001 0.001 0.001"/></geometry>
+        </collision>
+        <visual name="compact_relieved_bin_vis">
+          <origin xyz="0 0 ${-base_link_height}" rpy="0 0 0"/>
+          <geometry><mesh filename="package://tennis_robot/meshes/compact_relieved_bin.stl" scale="0.001 0.001 0.001"/></geometry>
+          <material name="basket_gray"/>
+        </visual>
+      </xacro:if>
+      <xacro:unless value="${cad_support_details}">
       <collision name="basket_floor_col">
         <origin xyz="${(floor_front_x + rear_x) / 2.0} 0 ${floor_top - floor_thickness / 2.0}" rpy="0 0 0"/>
@@ -291,5 +317,15 @@
         </visual>
       </xacro:if>
+      </xacro:unless>
     </link>
+    <xacro:if value="${cad_support_details}">
+      <gazebo reference="basket_link">
+        <sensor name="basket_handoff_contact_0" type="contact">
+          <always_on>true</always_on><update_rate>500</update_rate>
+          <topic>/gz/basket_handoff_contact_0</topic>
+          <contact><collision>compact_relieved_bin_col</collision></contact>
+        </sensor>
+      </gazebo>
+    </xacro:if>
   </xacro:macro>
 </robot>

File: ros2_ws/src/tennis_robot/urdf/components/drivetrain.urdf.xacro (robot description, xacro)
@@ -66,5 +66,5 @@
        constant ±y, which one prismatic DOF covers exactly). -->
   <xacro:macro name="intake_side_wheel"
-               params="side y nip_x wheel_z tilt_rad radius height carriage_travel max_vel effort mass sensor_index">
+               params="side y nip_x wheel_z tilt_rad radius height carriage_travel max_vel effort mass sensor_index parent:=base_link">
     <link name="intake_wheel_${side}_carriage_link">
       <inertial>
@@ -83,5 +83,5 @@
          against the SDF-patched spring. -->
     <joint name="intake_wheel_${side}_carriage_joint" type="prismatic">
-      <parent link="base_link"/>
+      <parent link="${parent}"/>
       <child link="intake_wheel_${side}_carriage_link"/>
       <origin xyz="${nip_x} ${y} ${wheel_z}" rpy="0 0 0"/>

File: ros2_ws/src/tennis_robot/urdf/tennis_robot.urdf.xacro (robot description, xacro)
@@ -16,4 +16,5 @@
   <xacro:include filename="components/electronics_packaging.urdf.xacro"/>
   <xacro:include filename="components/flywheel_launcher.urdf.xacro"/>
+  <xacro:include filename="components/compact_mechanics.urdf.xacro"/>
   <!-- ros2_control args. sim_mode swaps the hardware backend (sim vs real).
        controllers_config is the absolute path to controllers.yaml, injected by
@@ -29,8 +30,10 @@
   <xacro:arg name="battery_center_x" default="-0.143"/>
   <xacro:arg name="enable_compact_electronics" default="false"/>
-  <!-- Mechanical operating configuration. The physical concept has separate
-       COLLECT and LAUNCH configurations; the intake assembly and the flywheel
-       launcher claim the same front volume and are never fitted together.
-       Selected through the packaging variant, see scripts/generate_robot_urdf.py. -->
+  <xacro:arg name="enable_compact_mechanics" default="false"/>
+  <xacro:arg name="enable_basket_raised_holders" default="false"/>
+  <xacro:arg name="intake_parent_link" default="base_link"/>
+  <!-- Historical study variants may still select separate collect/launch
+       configurations.  The authoritative compact CAD permanently carries the
+       correctly aligned intake and launcher together. -->
   <xacro:arg name="enable_intake" default="true"/>
   <xacro:arg name="enable_flywheel" default="false"/>
@@ -41,7 +44,11 @@
   <xacro:arg name="basket_lift_travel" default="0.100"/>
   <xacro:arg name="basket_lift_overtravel" default="0.010"/>
+  <xacro:arg name="basket_launch_tilt_rad" default="0.0"/>
+  <xacro:arg name="basket_floor_thickness" default="0.005"/>
+  <xacro:arg name="basket_cad_support_details" default="false"/>
   <!-- Dual-wheel intake tuning (docs/dual-wheel-intake-design-el.md).
        Injected from INTAKE_WHEEL_* envs by scripts/generate_robot_urdf.py. -->
   <xacro:arg name="intake_wheel_radius" default="0.060"/>
+  <xacro:arg name="intake_wheel_width" default="0.080"/>
   <xacro:arg name="intake_wheel_gap" default="0.056"/>
   <xacro:arg name="intake_nip_x" default="0.540"/>
@@ -53,4 +60,6 @@
   <xacro:arg name="enable_funnel" default="true"/>
   <xacro:arg name="enable_ramp" default="true"/>
+  <xacro:arg name="compact_handoff_ramp_mesh"
+      default="package://tennis_robot/meshes/compact_relieved_handoff_ramp.stl"/>
   <xacro:arg name="enable_assist" default="false"/>
   <xacro:arg name="enable_conveyor" default="false"/>
@@ -119,5 +128,5 @@
        x=0.53 — a 0.005 bottom would intersect it). base_link is 45 mm above
        ground, hence wheel_z = 0.025. -->
-  <xacro:property name="intake_wheel_height" value="0.080"/>
+  <xacro:property name="intake_wheel_height" value="${float($(arg intake_wheel_width))}"/>
   <xacro:property name="intake_wheel_z" value="${0.070 - base_link_height}"/>
   <!-- Outward carriage travel: 8 mm absorbs the 3 mm/side nominal
@@ -230,11 +239,19 @@
       width="${wheel_width}"
       mass="${wheel_mass}"/>
-  <!-- INTAKE ASSEMBLY — fitted only in the COLLECT configuration.
-       Its wheels, funnel cheeks, elevation ramp and safety deflector occupy
-       x 446…884 mm / z 0…281 mm, the same volume the flywheel launcher needs
-       (wheels x 459…661, z 162…268). The two are alternative mechanical
-       configurations of one robot, so the launch configuration simply does not
-       carry this assembly — no deployment mechanism is modelled, because none
-       has been selected yet. -->
+  <!-- The compact bridge is the real load path for the intake pods and the
+       launcher cradle.  It must exist before those child joints are emitted. -->
+  <xacro:if value="$(arg enable_compact_mechanics)">
+    <xacro:compact_plywood_bridge parent="base_link" base_link_height="${base_link_height}"/>
+    <xacro:compact_basket_fixed_rails parent="base_link"
+        x_shift="${functional_shift_x}" base_link_height="${base_link_height}"/>
+    <xacro:compact_fixed_entry_hood parent="base_link"
+        x_shift="${functional_shift_x}" base_link_height="${base_link_height}"/>
+    <xacro:if value="$(arg enable_basket_raised_holders)">
+      <xacro:compact_basket_raised_holders parent="base_link"
+          x_shift="${functional_shift_x}" base_link_height="${base_link_height}"/>
+    </xacro:if>
+  </xacro:if>
+  <!-- Intake assembly.  In compact it is bridge-mounted and uses the measured
+       CAD cheeks/ramp; older study variants retain their historical funnel. -->
   <xacro:if value="$(arg enable_intake)">
     <!-- Left wheel drives ω<0 / right ω>0 (opposite signs, commanded by
@@ -252,4 +269,5 @@
         effort="${intake_wheel_effort}"
         mass="0.20"
+        parent="$(arg intake_parent_link)"
         sensor_index="0"/>
     <xacro:intake_side_wheel
@@ -265,9 +283,18 @@
         effort="${intake_wheel_effort}"
         mass="0.20"
+        parent="$(arg intake_parent_link)"
         sensor_index="1"/>
-    <xacro:intake_funnel parent="base_link" chassis_z="${chassis_z}" pitch="${scooper_pitch}"
-        x_shift="${functional_shift_x}"
-        cheek_x_bias="${intake_cad_alignment_x}"
-        enable_cheeks="$(arg enable_funnel)" enable_ramp="$(arg enable_ramp)"/>
+    <xacro:if value="$(arg enable_compact_mechanics)">
+      <xacro:compact_intake_static_structure parent="compact_bridge_link"
+          base_link_height="${base_link_height}"
+          enable_cheeks="$(arg enable_funnel)" enable_ramp="$(arg enable_ramp)"
+          ramp_mesh="$(arg compact_handoff_ramp_mesh)"/>
+    </xacro:if>
+    <xacro:unless value="$(arg enable_compact_mechanics)">
+      <xacro:intake_funnel parent="base_link" chassis_z="${chassis_z}" pitch="${scooper_pitch}"
+          x_shift="${functional_shift_x}"
+          cheek_x_bias="${intake_cad_alignment_x}"
+          enable_cheeks="$(arg enable_funnel)" enable_ramp="$(arg enable_ramp)"/>
+    </xacro:unless>
   </xacro:if>
   <xacro:if value="$(arg enable_assist)">
@@ -325,5 +352,8 @@
       lift_overtravel="${float($(arg basket_lift_overtravel))}"
       empty_mass="${float($(arg basket_empty_mass))}"
-      payload_mass="${float($(arg basket_payload_mass))}"/>
+      payload_mass="${float($(arg basket_payload_mass))}"
+      launch_tilt_rad="${float($(arg basket_launch_tilt_rad))}"
+      floor_thickness="${float($(arg basket_floor_thickness))}"
+      cad_support_details="$(arg basket_cad_support_details)"/>
   <xacro:battery_pack parent="base_link"
       center_x="${float($(arg battery_center_x))}"/>
@@ -333,12 +363,20 @@
   </xacro:if>
   <xacro:if value="$(arg enable_flywheel)">
-    <xacro:side_by_side_flywheel_launcher
-        parent="base_link"
-        origin_x="${0.560 + functional_shift_x}"
-        nip_z_ground="0.215"
-        base_link_height="${base_link_height}"
-        pitch_rad="0.349066"
-        nip_gap="${float($(arg flywheel_nip_gap))}"
-        max_vel="${float($(arg flywheel_max_vel))}"/>
+    <xacro:if value="$(arg enable_compact_mechanics)">
+      <xacro:compact_cad_flywheel_launcher parent="compact_bridge_link"
+          base_link_height="${base_link_height}"
+          nip_gap="${float($(arg flywheel_nip_gap))}"
+          max_vel="${float($(arg flywheel_max_vel))}"/>
+    </xacro:if>
+    <xacro:unless value="$(arg enable_compact_mechanics)">
+      <xacro:side_by_side_flywheel_launcher
+          parent="base_link"
+          origin_x="${0.560 + functional_shift_x}"
+          nip_z_ground="0.215"
+          base_link_height="${base_link_height}"
+          pitch_rad="0.349066"
+          nip_gap="${float($(arg flywheel_nip_gap))}"
+          max_vel="${float($(arg flywheel_max_vel))}"/>
+    </xacro:unless>
   </xacro:if>
   <xacro:rplidar_c1_mount
