Commit message: feat(mechanics): freeze standalone flywheel launcher design

File: ros2_ws/src/tennis_robot/urdf/components/flywheel_launcher_module.urdf.xacro (robot description, xacro)
@@ -12,8 +12,80 @@
     model and contains no feeder, basket or intake geometry.
   -->
+  <xacro:macro name="provisional_candidate_flywheel"
+      params="side parent y radius width rotating_mass spin_inertia transverse_inertia com_z max_vel effort">
+    <link name="flywheel_${side}_link">
+      <inertial>
+        <origin xyz="0 0 ${com_z}" rpy="0 0 0"/>
+        <mass value="${rotating_mass}"/>
+        <inertia ixx="${transverse_inertia}" ixy="0" ixz="0"
+                 iyy="${transverse_inertia}" iyz="0" izz="${spin_inertia}"/>
+      </inertial>
+      <collision name="flywheel_${side}_col">
+        <geometry><cylinder radius="${radius}" length="${width}"/></geometry>
+      </collision>
+      <visual name="flywheel_${side}_vis">
+        <geometry><cylinder radius="${radius}" length="${width}"/></geometry>
+        <material name="safety_orange"/>
+      </visual>
+      <collision name="flywheel_${side}_shaft_col">
+        <origin xyz="0 0 0.032" rpy="0 0 0"/>
+        <geometry><cylinder radius="0.004" length="0.030"/></geometry>
+      </collision>
+      <visual name="flywheel_${side}_shaft_vis">
+        <origin xyz="0 0 0.032" rpy="0 0 0"/>
+        <geometry><cylinder radius="0.004" length="0.030"/></geometry>
+        <material name="mount_gray"/>
+      </visual>
+      <!-- Analysis-only 7075-T6 hub envelope: 22 mm split collar, 10 mm
+           through-wheel pilot, distal M8 washer/nut retention. -->
+      <collision name="flywheel_${side}_hub_collar_col">
+        <origin xyz="0 0 0.03175" rpy="0 0 0"/>
+        <geometry><cylinder radius="0.011" length="0.0135"/></geometry>
+      </collision>
+      <visual name="flywheel_${side}_hub_collar_vis">
+        <origin xyz="0 0 0.03175" rpy="0 0 0"/>
+        <geometry><cylinder radius="0.011" length="0.0135"/></geometry>
+        <material name="electronics_blue"/>
+      </visual>
+      <collision name="flywheel_${side}_hub_pilot_col">
+        <origin xyz="0 0 0" rpy="0 0 0"/>
+        <geometry><cylinder radius="0.005" length="0.050"/></geometry>
+      </collision>
+      <visual name="flywheel_${side}_hub_pilot_vis">
+        <origin xyz="0 0 0" rpy="0 0 0"/>
+        <geometry><cylinder radius="0.005" length="0.050"/></geometry>
+        <material name="electronics_blue"/>
+      </visual>
+      <collision name="flywheel_${side}_retainer_col">
+        <origin xyz="0 0 -0.030" rpy="0 0 0"/>
+        <geometry><cylinder radius="0.011" length="0.008"/></geometry>
+      </collision>
+      <visual name="flywheel_${side}_retainer_vis">
+        <origin xyz="0 0 -0.030" rpy="0 0 0"/>
+        <geometry><cylinder radius="0.011" length="0.008"/></geometry>
+        <material name="electronics_blue"/>
+      </visual>
+    </link>
+    <joint name="flywheel_${side}_joint" type="continuous">
+      <parent link="${parent}"/>
+      <child link="flywheel_${side}_link"/>
+      <origin xyz="0 ${y} 0" rpy="0 0 0"/>
+      <axis xyz="0 0 1"/>
+      <limit effort="${effort}" velocity="${max_vel}"/>
+      <dynamics damping="0.002"/>
+    </joint>
+    <gazebo reference="flywheel_${side}_link">
+      <mu1>2.0</mu1><mu2>2.0</mu2>
+    </gazebo>
+  </xacro:macro>
   <xacro:macro name="authoritative_flywheel_launcher_module"
       params="parent origin_xyz:='0 0 0' pitch_rad:='0.349065850399'
-              wheel_mass:=0.40 fixed_mass:=4.4525888
-              max_vel:=320.0 effort:=6.0">
+              wheel_mass:=0.90 hub_mass:=0.0267636462761
+              spin_inertia:=0.00675116210829 transverse_inertia:=0.00358105785160
+              rotating_com_z:=0.00027153263648 fixed_mass:=4.33478256461
+              fixed_com_x:=-0.00231297294785 fixed_com_z:=0.0185061462201
+              fixed_ixx:=0.0561713265628 fixed_iyy:=0.0294163341856
+              fixed_izz:=0.0630372476838 fixed_ixz:=-0.000350443006278
+              max_vel:=320.0 effort:=0.62">
     <xacro:property name="launcher_ball_d" value="0.066"/>
     <xacro:property name="launcher_wheel_radius" value="0.100"/>
@@ -35,45 +107,65 @@
     </gazebo>
     <link name="flywheel_launcher_frame_link">
-      <!--
-        fixed_mass is a declared simulation estimate, not an authoritative CAD
-        mass: two 256x314x8 mm aluminium plates at 2700 kg/m^3 (3.4725888 kg)
-        plus two documented 0.49 kg D5065 motors. Symmetry places the estimate
-        at the nip origin. The inertia is a conservative box-envelope estimate
-        pending manufactured-part mass properties.
-      -->
+      <!-- fixed_mass = two exit-relieved aluminium plates plus two documented
+           0.49 kg D5065 bodies. Rotor inertia remains a separate sensitivity
+           because the manufacturer value is unavailable. -->
       <inertial>
+        <origin xyz="${fixed_com_x} 0 ${fixed_com_z}" rpy="0 0 0"/>
         <mass value="${fixed_mass}"/>
-        <inertia ixx="${fixed_mass * (launcher_plate_y*launcher_plate_y + 0.094*0.094) / 12.0}"
-                 ixy="0" ixz="0"
-                 iyy="${fixed_mass * (launcher_plate_x*launcher_plate_x + 0.094*0.094) / 12.0}"
+        <inertia ixx="${fixed_ixx}"
+                 ixy="0" ixz="${fixed_ixz}"
+                 iyy="${fixed_iyy}"
                  iyz="0"
-                 izz="${fixed_mass * (launcher_plate_x*launcher_plate_x + launcher_plate_y*launcher_plate_y) / 12.0}"/>
+                 izz="${fixed_izz}"/>
       </inertial>
       <collision name="flywheel_cradle_lower_plate_col">
         <origin xyz="0 0 ${-launcher_plate_offset_z}" rpy="0 0 0"/>
-        <geometry><box size="${launcher_plate_x} ${launcher_plate_y} ${launcher_plate_z}"/></geometry>
+        <geometry><mesh filename="package://tennis_robot/meshes/flywheel_lower_panel_exit_clearance.stl" scale="0.001 0.001 0.001"/></geometry>
       </collision>
       <visual name="flywheel_cradle_lower_plate_vis">
         <origin xyz="0 0 ${-launcher_plate_offset_z}" rpy="0 0 0"/>
-        <geometry><box size="${launcher_plate_x} ${launcher_plate_y} ${launcher_plate_z}"/></geometry>
+        <geometry><mesh filename="package://tennis_robot/meshes/flywheel_lower_panel_exit_clearance.stl" scale="0.001 0.001 0.001"/></geometry>
         <material name="mount_gray"/>
       </visual>
       <collision name="flywheel_cradle_upper_plate_col">
         <origin xyz="0 0 ${launcher_plate_offset_z}" rpy="0 0 0"/>
-        <geometry><box size="${launcher_plate_x} ${launcher_plate_y} ${launcher_plate_z}"/></geometry>
+        <geometry><mesh filename="package://tennis_robot/meshes/flywheel_upper_panel_exit_clearance.stl" scale="0.001 0.001 0.001"/></geometry>
       </collision>
       <visual name="flywheel_cradle_upper_plate_vis">
         <origin xyz="0 0 ${launcher_plate_offset_z}" rpy="0 0 0"/>
-        <geometry><box size="${launcher_plate_x} ${launcher_plate_y} ${launcher_plate_z}"/></geometry>
+        <geometry><mesh filename="package://tennis_robot/meshes/flywheel_upper_panel_exit_clearance.stl" scale="0.001 0.001 0.001"/></geometry>
         <material name="mount_gray"/>
       </visual>
+      <xacro:property name="motor_body_z" value="${launcher_plate_offset_z + launcher_plate_z / 2.0 + 0.065 / 2.0}"/>
+      <collision name="d5065_motor_left_col">
+        <origin xyz="0 ${launcher_wheel_y} ${motor_body_z}" rpy="0 0 0"/>
+        <geometry><cylinder radius="0.025" length="0.065"/></geometry>
+      </collision>
+      <visual name="d5065_motor_left_vis">
+        <origin xyz="0 ${launcher_wheel_y} ${motor_body_z}" rpy="0 0 0"/>
+        <geometry><cylinder radius="0.025" length="0.065"/></geometry>
+        <material name="anthracite"/>
+      </visual>
+      <collision name="d5065_motor_right_col">
+        <origin xyz="0 ${-launcher_wheel_y} ${motor_body_z}" rpy="0 0 0"/>
+        <geometry><cylinder radius="0.025" length="0.065"/></geometry>
+      </collision>
+      <visual name="d5065_motor_right_vis">
+        <origin xyz="0 ${-launcher_wheel_y} ${motor_body_z}" rpy="0 0 0"/>
+        <geometry><cylinder radius="0.025" length="0.065"/></geometry>
+        <material name="anthracite"/>
+      </visual>
     </link>
-    <xacro:flywheel_wheel side="left" parent="flywheel_launcher_frame_link"
+    <xacro:provisional_candidate_flywheel side="left" parent="flywheel_launcher_frame_link"
         y="${launcher_wheel_y}" radius="${launcher_wheel_radius}"
-        width="${launcher_wheel_width}" mass="${wheel_mass}"
+        width="${launcher_wheel_width}" rotating_mass="${wheel_mass + hub_mass}"
+        spin_inertia="${spin_inertia}" transverse_inertia="${transverse_inertia}"
+        com_z="${rotating_com_z}"
         max_vel="${max_vel}" effort="${effort}"/>
-    <xacro:flywheel_wheel side="right" parent="flywheel_launcher_frame_link"
+    <xacro:provisional_candidate_flywheel side="right" parent="flywheel_launcher_frame_link"
         y="${-launcher_wheel_y}" radius="${launcher_wheel_radius}"
-        width="${launcher_wheel_width}" mass="${wheel_mass}"
+        width="${launcher_wheel_width}" rotating_mass="${wheel_mass + hub_mass}"
+        spin_inertia="${spin_inertia}" transverse_inertia="${transverse_inertia}"
+        com_z="${rotating_com_z}"
         max_vel="${max_vel}" effort="${effort}"/>
   </xacro:macro>

File: ros2_ws/src/tennis_robot/urdf/flywheel_launcher_bench.urdf.xacro (robot description, xacro)
@@ -37,9 +37,10 @@
     </hardware>
     <joint name="flywheel_left_joint">
-      <command_interface name="velocity"><param name="min">-320.0</param><param name="max">320.0</param></command_interface>
+      <!-- 20 A provisional D5065 limit: Kt 0.031 N m/A => 0.62 N m. -->
+      <command_interface name="effort"><param name="min">-0.62</param><param name="max">0.62</param></command_interface>
       <state_interface name="position"/><state_interface name="velocity"/>
     </joint>
     <joint name="flywheel_right_joint">
-      <command_interface name="velocity"><param name="min">-320.0</param><param name="max">320.0</param></command_interface>
+      <command_interface name="effort"><param name="min">-0.62</param><param name="max">0.62</param></command_interface>
       <state_interface name="position"/><state_interface name="velocity"/>
     </joint>
