Commit message: feat: update intake hardware and simulation studies

File: ros2_ws/src/tennis_robot/urdf/tennis_robot.urdf.xacro (robot description, xacro)
@@ -3,5 +3,4 @@
   <xacro:include filename="components/materials.urdf.xacro"/>
   <xacro:include filename="components/base.urdf.xacro"/>
-  <xacro:include filename="components/funnel.urdf.xacro"/>
   <xacro:include filename="components/basket.urdf.xacro"/>
   <xacro:include filename="components/battery.urdf.xacro"/>
@@ -20,36 +19,46 @@
        controllers_config is the absolute path to controllers.yaml, injected by
        scripts/generate_robot_urdf.py / the launch file. -->
+  <!-- FALLBACK POLICY (2026-08-27). Every xacro:arg below is ALSO passed by
+       scripts/generate_robot_urdf.py, so these defaults only apply when the
+       xacro is rendered directly. They used to describe the retired baseline
+       robot, so a direct render silently produced a DIFFERENT machine (whole
+       functional chain 170 mm off, intake parented to base_link, 0.01 kg
+       basket). They now describe the ONE robot. If you change a generator
+       value, change the default here in the same edit. -->
   <xacro:arg name="sim_mode" default="true"/>
   <xacro:arg name="controllers_config" default="config/controllers.yaml"/>
-  <xacro:arg name="expose_intake_carriage_state" default="false"/>
-  <!-- Selectable packaging overlay. Baseline remains the frozen collection
-       model; compact shifts the complete functional chain by -100 mm and
-       enables the new mass-bearing components through the generator. -->
-  <xacro:arg name="functional_shift_x" default="0.0"/>
-  <xacro:arg name="intake_cad_alignment_x" default="0.0"/>
+  <!-- Packaging overlay of the ONE robot: the compact CAD machine shifts the
+       complete functional chain by -100 mm. Injected by
+       scripts/generate_robot_urdf.py from scripts/intake_geometry.py. -->
+  <xacro:arg name="functional_shift_x" default="-0.100"/>
+  <xacro:arg name="intake_cad_alignment_x" default="-0.070"/>
   <xacro:arg name="battery_center_x" default="-0.143"/>
-  <xacro:arg name="enable_compact_electronics" default="false"/>
-  <xacro:arg name="enable_compact_mechanics" default="false"/>
+  <xacro:arg name="enable_compact_electronics" default="true"/>
+  <!-- ONE robot: the compact CAD machine. The baseline / option-a-* packaging
+       variants were archived 2026-08-27; components/archive/ keeps their xacro. -->
+  <xacro:arg name="enable_compact_mechanics" default="true"/>
   <xacro:arg name="enable_basket_raised_holders" default="false"/>
-  <xacro:arg name="intake_parent_link" default="base_link"/>
-  <!-- Historical study variants may still select separate collect/launch
-       configurations.  The authoritative compact CAD permanently carries the
-       correctly aligned intake and launcher together. -->
+  <xacro:arg name="intake_parent_link" default="compact_bridge_link"/>
+  <!-- The compact CAD machine permanently carries the correctly aligned
+       intake AND flywheel launcher together, so both default ON: this is the
+       machine we test. Set the env overrides only to isolate one of them. -->
   <xacro:arg name="enable_intake" default="true"/>
-  <xacro:arg name="enable_flywheel" default="false"/>
+  <xacro:arg name="enable_flywheel" default="true"/>
   <xacro:arg name="flywheel_max_vel" default="320.0"/>
   <xacro:arg name="flywheel_nip_gap" default="0.058"/>
-  <xacro:arg name="basket_empty_mass" default="0.01"/>
+  <xacro:arg name="basket_empty_mass" default="1.012"/>
   <xacro:arg name="basket_payload_mass" default="0.0"/>
   <xacro:arg name="basket_lift_travel" default="0.100"/>
   <xacro:arg name="basket_lift_overtravel" default="0.010"/>
   <xacro:arg name="basket_launch_tilt_rad" default="0.0"/>
-  <xacro:arg name="basket_floor_thickness" default="0.005"/>
-  <xacro:arg name="basket_cad_support_details" default="false"/>
-  <!-- NOT_PHYSICAL_INTAKE_ARCHITECTURE surrogate tuning. Physical definition:
-       docs/mechanism/standalone-intake-fixed-motor-compliant-tyre.md.
-       Injected from INTAKE_WHEEL_* envs by scripts/generate_robot_urdf.py. -->
-  <xacro:arg name="intake_wheel_radius" default="0.060"/>
-  <xacro:arg name="intake_wheel_width" default="0.080"/>
+  <xacro:arg name="basket_floor_thickness" default="0.006"/>
+  <xacro:arg name="basket_cad_support_details" default="true"/>
+  <!-- Frozen CAD intake geometry. Single source of truth:
+       scripts/intake_geometry.py (transcribed from the two authoritative SCAD
+       files); injected from INTAKE_WHEEL_* envs by
+       scripts/generate_robot_urdf.py. Wheel radius/width/gap and the derived
+       wheel_y are CAD values, not tuning knobs. -->
+  <xacro:arg name="intake_wheel_radius" default="0.062"/>
+  <xacro:arg name="intake_wheel_width" default="0.073"/>
   <xacro:arg name="intake_wheel_gap" default="0.056"/>
   <xacro:arg name="intake_nip_x" default="0.540"/>
@@ -57,4 +66,7 @@
   <xacro:arg name="intake_wheel_max_vel" default="26.3"/>
   <xacro:arg name="intake_wheel_effort" default="1.77"/>
+  <!-- Physically unmeasured felt/tread friction. SWEPT bound (0.3/0.6/0.9),
+       never a value chosen to make a result pass. -->
+  <xacro:arg name="intake_tread_mu" default="0.6"/>
   <!-- Concept Validation Plan gates: Phase 1 = throat only (both false),
        Phase 2 = +funnel, Phase 3 = wheels+ramp, Phase 4 = full intake. -->
@@ -62,5 +74,5 @@
   <xacro:arg name="enable_ramp" default="true"/>
   <xacro:arg name="compact_handoff_ramp_mesh"
-      default="package://tennis_robot/meshes/compact_relieved_handoff_ramp.stl"/>
+      default="package://tennis_robot/meshes/option_a_handoff_ramp.stl"/>
   <xacro:arg name="enable_assist" default="false"/>
   <xacro:arg name="enable_conveyor" default="false"/>
@@ -124,18 +136,11 @@
   <!-- Wheel centre offset from the corridor centreline. -->
   <xacro:property name="intake_wheel_y" value="${intake_wheel_gap / 2.0 + intake_wheel_radius}"/>
-  <!-- Wheel cylinder spans ground z 0.030..0.110 (centre 0.070): the band
-       still includes the 66 mm ball's equator (rest z=33, and it RISES as
-       the ball is fed onto the ramp), while the wheel undersides clear the
-       ramp sheet where it climbs through their rear span (ramp z≈0.021 at
-       x=0.53 — a 0.005 bottom would intersect it). base_link is 45 mm above
-       ground, hence wheel_z = 0.025. -->
+  <!-- Tilted 124 x 73 mm wheel about the 35 degree axis: its lowest point is
+       4.5 mm above the court and its highest 135.5 mm, centre 70 mm. The band
+       includes the 66 mm ball's equator both at rest on the court (centre 33)
+       and lifted by the handoff ramp (centre 44..64 through the nip stations).
+       base_link is 45 mm above ground, hence wheel_z = 0.025. -->
   <xacro:property name="intake_wheel_height" value="${float($(arg intake_wheel_width))}"/>
   <xacro:property name="intake_wheel_z" value="${0.070 - base_link_height}"/>
-  <!-- NOT_PHYSICAL_INTAKE_ARCHITECTURE:
-       SIMULATION_ONLY_TYRE_COMPLIANCE_SURROGATE, legacy rigid-wheel model.
-       The physical FIT0186 motors and wheel centres are fixed to the bridge;
-       no carriage exists. This 8 mm DOF must not be used as physical-design
-       or validation evidence and must be replaced by calibrated tyre contact. -->
-  <xacro:property name="intake_carriage_travel" value="0.008"/>
   <xacro:property name="intake_assist_x" value="${float($(arg intake_assist_x))}"/>
   <xacro:property name="intake_assist_z" value="${float($(arg intake_assist_z))}"/>
@@ -152,6 +157,27 @@
        and lidar_link itself sits base_link_height above ground. Deriving the
        mount height keeps all three terms in one place — hardcoding 0.498 here
-       silently placed the scan plane at 0.578 m. -->
-  <xacro:property name="lidar_scan_plane_z_ground" value="0.498"/>
+       silently placed the scan plane at 0.578 m.
+       RAISED 0.498 -> 0.5535 (2026-08-27). At 0.498 the lidar_link sat at
+       ground 0.463, so head_vis (r=0.047, length 0.045, CENTRED on the link)
+       spanned ground 0.4405..0.4855 — entirely INSIDE the shell, whose roof
+       panel top is at ground 0.494. The scan plane cleared that roof by only
+       4 mm, against the CAD's own 8 mm scan_clearance rule, and worked purely
+       because the chassis is level.
+       The shell is deliberately tall: its height is set by the basket in its
+       RAISED position, where the basket feeds the flywheel (the lowered
+       position serves the intake). So the roof does not come down to the
+       CAD's older uniform_shell_top_z = 463 — the LiDAR goes up instead.
+       Datum derivation, so it can be re-derived if the roof moves:
+         roof panel top (ground)          0.494
+         + head clearance above the roof  0.002   (CAD sensor_roof_offset = +2)
+         + half of head_vis               0.0225
+         + lidar_sensor_scan_offset       0.035
+         = 0.5535
+       giving lidar_link at ground 0.5185 and the head bottom at 0.496, i.e.
+       resting 2 mm proud of the roof instead of buried 31 mm inside it.
+       NOTE: the CAD lidar-pod-study models a 30 mm sensor whose scan plane is
+       at its top; this URDF uses a 45 mm head with a 35 mm sim-only offset.
+       That 30/45 mm discrepancy is unreconciled and is NOT resolved here. -->
+  <xacro:property name="lidar_scan_plane_z_ground" value="0.5535"/>
   <xacro:property name="lidar_sensor_scan_offset" value="0.035"/>
   <xacro:property name="lidar_mount_z"
@@ -159,5 +185,32 @@
   <xacro:property name="lidar_xyz" value="-0.42 0 ${lidar_mount_z}"/>
   <xacro:property name="lidar_rpy" value="0 0 0"/>  <!-- level chassis: horizontal scan plane -->
-  <xacro:property name="camera_xyz" value="${0.535 + functional_shift_x} 0 0.443"/>
+  <!-- OAK-D. MOVED FORWARD 0.535 -> 0.690 (2026-08-27). The frozen intake
+       extends the robot much further forward than the body panels do: the
+       cheek mouth is at base_link x=0.705 and the CAD nose front
+       (external-panel-study nose_front_x=790, i.e. base_link 0.690) agrees
+       with it. At x=0.535 the camera sat 155-170 mm BEHIND the actual front
+       edge, cantilevered over the flywheel with the cheeks and ramp reaching
+       out past it.
+       Height is unchanged at 0.443 (ground 0.488), which already satisfies
+       "above the flywheel opening" and keeps the calibrated aim:
+         flywheel exit at the nose  ground 0.2987, opening d=116 -> top 0.357
+         camera body bottom          ground 0.463  -> 106 mm above the opening
+         ball centre at the nose     ground 0.2987, ball top 0.332
+                                                   -> 131 mm of launch clearance
+         camera head top             ground 0.5127
+         LiDAR scan plane            ground 0.5535 -> 40.8 mm clear, no occlusion
+       (at the old 0.498 scan plane this camera cut the forward sector by
+       14.7 mm; raising the LiDAR fixed that, see the datum block above.)
+       KNOWN GAP: components/body_panels.urdf.xacro still models the OLD short
+       shell, front face at base_link 0.46 — 230 mm behind the CAD nose. The
+       camera mount therefore still hangs in free air here. Extending the shell
+       to the CAD nose, and cutting the launcher exit opening in it, is a
+       separate task and is NOT done here. -->
+       The literal below is a CAD-frame X: functional_shift_x (-0.100 on the
+       compact variant) converts it to base_link. 0.790 IS the CAD
+       nose_front_x, so compact lands at base_link 0.690, next to the cheek
+       mouth which compact_mechanics hardcodes at base_link 0.705 (CAD 805).
+       Writing 0.690 here would double-shift it to 0.590. -->
+  <xacro:property name="camera_xyz" value="${0.790 + functional_shift_x} 0 0.443"/>
   <xacro:property name="camera_rpy" value="0 0.273 0"/>  <!-- forward-down tilt ~15.6deg; preserves the old world aim (0.22 cam + 0.053 chassis pitch) now that the chassis is level -->
   <xacro:property name="sensor_update_rate" value="31.25"/>
@@ -270,7 +323,7 @@
         radius="${intake_wheel_radius}"
         height="${intake_wheel_height}"
-        carriage_travel="${intake_carriage_travel}"
         max_vel="${intake_wheel_max_vel}"
         effort="${intake_wheel_effort}"
+        tread_mu="${float($(arg intake_tread_mu))}"
         mass="0.20"
         parent="$(arg intake_parent_link)"
@@ -284,7 +337,7 @@
         radius="${intake_wheel_radius}"
         height="${intake_wheel_height}"
-        carriage_travel="${intake_carriage_travel}"
         max_vel="${intake_wheel_max_vel}"
         effort="${intake_wheel_effort}"
+        tread_mu="${float($(arg intake_tread_mu))}"
         mass="0.20"
         parent="$(arg intake_parent_link)"
@@ -296,11 +349,5 @@
           ramp_mesh="$(arg compact_handoff_ramp_mesh)"/>
     </xacro:if>
-    <xacro:unless value="$(arg enable_compact_mechanics)">
-      <xacro:intake_funnel parent="base_link" chassis_z="${chassis_z}" pitch="${scooper_pitch}"
-          x_shift="${functional_shift_x}"
-          cheek_x_bias="${intake_cad_alignment_x}"
-          enable_cheeks="$(arg enable_funnel)" enable_ramp="$(arg enable_ramp)"/>
-    </xacro:unless>
-  </xacro:if>
+</xacro:if>
   <xacro:if value="$(arg enable_assist)">
     <xacro:intake_assist_roller
@@ -374,15 +421,5 @@
           max_vel="${float($(arg flywheel_max_vel))}"/>
     </xacro:if>
-    <xacro:unless value="$(arg enable_compact_mechanics)">
-      <xacro:side_by_side_flywheel_launcher
-          parent="base_link"
-          origin_x="${0.560 + functional_shift_x}"
-          nip_z_ground="0.215"
-          base_link_height="${base_link_height}"
-          pitch_rad="0.349066"
-          nip_gap="${float($(arg flywheel_nip_gap))}"
-          max_vel="${float($(arg flywheel_max_vel))}"/>
-    </xacro:unless>
-  </xacro:if>
+</xacro:if>
   <xacro:rplidar_c1_mount
       parent="base_link"
@@ -452,5 +489,4 @@
       sim_mode="$(arg sim_mode)"
       controllers_config="$(arg controllers_config)"
-      expose_intake_carriage_state="$(arg expose_intake_carriage_state)"
       intake_max_vel="${intake_wheel_max_vel}"
       enable_intake="$(arg enable_intake)"
