Commit message: collect_one live approach: lock refresh, capture profile, wheel gate, odom fusion
Four verified layers between "robot drives" and "ball reaches the wheels",
each measured live against Gazebo ground truth (debug-log #44):

- Perception validated: YOLO+depth world positions match ground truth to
  7.5 cm at 1.1 m; the pipeline was never the problem.
- collect_one locked its target once at first sighting (3-5 m out, max
  error) and drove blind to that stale point. The lock now refreshes on
  every nearer sighting (0.6 m gate against target stealing), shrinking the
  frozen error to the last-visible ~7 cm.
- Capture profile matched to the bench-proven intake: switch to the 0.14 m/s
  creep at 1.0 m (before funnel contact, still inside camera visibility),
  10 s budget instead of 2.8 s (which covered only 0.39 m and timed out
  short of the wheels), clamped steering with a dead-straight commit inside
  0.45 m. Docker capture speeds raised from roller-era 0.07/0.05 to 0.14.
- The intake wheels never spun during live captures: the throat-beam latch
  never fired (0/2336 in 60 s) because the beam at x=0.670 assumed first
  contact at 0.613 while the tilted wheels really touch at 0.645, so a
  plowed ball only grazed it - balls were bulldozed 9.5 m by dead rubber.
  CAPTURE is now ungated (committed ingest; the latch remains for
  APPROACH) and the beam moved to x=0.720, ahead of true first contact.
- Consumers read EKF-fused odometry (/odometry/filtered) instead of raw
  wheel odom, whose yaw is skewed by the wheel_separation SLAM fudge; the
  EKF itself stops fusing accelerometer ax, which double-integrated into a
  25 m off-court drift. Lateral aim during capture creeps is now 0-8 cm,
  inside the funnel envelope.

Remaining (bench campaign next): the ball enters the corridor but arrives
rolling with the robot (near-zero relative speed at the nip), takes a weak
kick to z=0.074 - just under the 0.088 lip - and settles in the jump-base
wedge. The bench-proven capture assumed a static ball.

Co-Authored-By: Claude Fable 5 <noreply@anthropic.com>

File: ros2_ws/src/tennis_robot/urdf/tennis_robot.urdf.xacro (robot description, xacro)
@@ -119,5 +119,5 @@
        contact (ball-centre x≈0.613). Collection confirmation is the BASKET
        beam pair below — see gazebo_extras_node.py. -->
-  <xacro:property name="ir_x" value="0.670"/>
+  <xacro:property name="ir_x" value="0.720"/>
   <xacro:property name="ir_y" value="0.105"/>
   <xacro:property name="ir_z" value="-0.005"/>
